File: AP2100/Power.sch (KiCad schematic (older format))
At the start: 35 parts, among them U4 MPQ8634AGLE-P

Commit message: Add Magjack part
Other:
- note removed: "Is this really correct?\nRemoving the voltage divider\nresistors because Vfb == Vdd"
Changed lines of the file:
@@
 Text Label 5600 1500 0    50   ~ 0
 CPU_VDD
-Text Notes 2900 2400 0    50   ~ 0
-Is this really correct?\nRemoving the voltage divider\nresistors because Vfb == Vdd
 Text Label 1400 1900 0    50   ~ 0
 EN_VDD
@@
 Wire Wire Line
 	3425 5700 3725 5700
+$Comp
+L Scott:GND #PWR?
+U 1 1 5EF7ABF6
+P -475 -500
+F 0 "#PWR?" H -475 -750 50  0001 C CNN
+F 1 "GND" H -470 -673 50  0000 C CNN
+F 2 "" H -475 -500 50  0001 C CNN
+F 3 "" H -475 -500 50  0001 C CNN
+	1    -475 -500
+	1    0    0    -1
+$EndComp
+$Comp
+L Scott:GND #PWR?
+U 1 1 5EF7BF91
+P -50 -500
+F 0 "#PWR?" H -50 -750 50  0001 C CNN
+F 1 "GND" H -45 -673 50  0000 C CNN
+F 2 "" H -50 -500 50  0001 C CNN
+F 3 "" H -50 -500 50  0001 C CNN
+	1    -50  -500
+	1    0    0    -1
+$EndComp
 $EndSCHEMATC

Commit message: Update poe Add cap library
Parts:
- C34: value C_Small -> 500pF; footprint (none) -> Capacitor_SMD:C_0402_1005Metric
- C45: renamed from C?; value .1 -> .1uF
- gave numbers to parts that had none: 15
Connections:
- net EN_VDD: no longer U5.8 (EN)
- net CPU_VDD_PG: now reaches U4.9 (PGOOD)
- net 3V3_PG: now reaches U5.9 (PGOOD)
- net +12V renamed 12V
- new net EN_3V3: U5.8 (EN)
Changed lines of the file:
@@
 P 3725 5200
 F 0 "C34" V 3496 5200 50  0000 C CNN
-F 1 "C_Small" V 3587 5200 50  0000 C CNN
-F 2 "" H 3725 5200 50  0001 C CNN
+F 1 "500pF" V 3587 5200 50  0000 C CNN
+F 2 "Capacitor_SMD:C_0402_1005Metric" H 3725 5200 50  0001 C CNN
 F 3 "~" H 3725 5200 50  0001 C CNN
 	1    3725 5200
@@
 	-1   0    0    1
 $EndComp
-Text Label 650  1500 0    50   ~ 0
-+12V
-Text Label 5600 1500 0    50   ~ 0
-CPU_VDD
-Text Label 1400 1900 0    50   ~ 0
-EN_VDD
-Text Label 3175 2150 0    50   ~ 0
-CPU_VDD_SENSE
-Text Label 3175 2500 0    50   ~ 0
-CPU_GND_SENSE
 Wire Wire Line
 	1700 1650 1700 1500
@@
 	1700 1500 1450 1500
 Wire Wire Line
-	850  1500 650  1500
+	850  1500 800  1500
 Wire Wire Line
 	1150 1500 850  1500
@@
 	3100 2500 3450 2500
 Wire Wire Line
-	3450 2500 4100 2500
-Wire Wire Line
 	3800 2150 3800 1500
 Wire Wire Line
@@
 	3150 3100 3150 3200
 Wire Wire Line
-	1400 1900 1700 1900
+	1650 1900 1700 1900
 Wire Wire Line
 	3650 1500 3800 1500
@@
 	5550 2500 5150 2500
 Wire Wire Line
-	5550 1500 5925 1500
+	5550 1500 5625 1500
 Connection ~ 1700 1500
 Connection ~ 850  1500
@@
 Connection ~ 5550 1500
 $Comp
-L MPQ8634AGLE-P:MPQ8634AGLE-P U?
+L MPQ8634AGLE-P:MPQ8634AGLE-P U5
 U 1 1 5EF244CE
 P 2675 5450
-F 0 "U?" H 2675 6465 50  0000 C CNN
+F 0 "U5" H 2675 6465 50  0000 C CNN
 F 1 "MPQ8634AGLE-P" H 2675 6374 50  0000 C CNN
 F 2 "Scott:QFN45P300X400X100-21N" H 3275 4870 50  0001 L CNN
@@
 $EndComp
 $Comp
-L Device:C_Small C?
+L Device:C_Small C32
 U 1 1 5EF244DD
 P 1125 4800
-F 0 "C?" H 1217 4846 50  0000 L CNN
+F 0 "C32" H 1217 4846 50  0000 L CNN
 F 1 "22uF" H 1217 4755 50  0000 L CNN
 F 2 "Capacitor_SMD:C_0805_2012Metric" H 1125 4800 50  0001 C CNN
@@
 $EndComp
 $Comp
-L Device:C_Small C?
+L Device:C_Small C33
 U 1 1 5EF244EC
 P 1425 4800
-F 0 "C?" H 1517 4846 50  0000 L CNN
+F 0 "C33" H 1517 4846 50  0000 L CNN
 F 1 "22uF" H 1517 4755 50  0000 L CNN
 F 2 "Capacitor_SMD:C_0805_2012Metric" H 1425 4800 50  0001 C CNN
@@
 $EndComp
 $Comp
-L Device:C_Small C?
+L Device:C_Small C35
 U 1 1 5EF244FB
 P 1725 4800
-F 0 "C?" H 1817 4846 50  0000 L CNN
+F 0 "C35" H 1817 4846 50  0000 L CNN
 F 1 "22uF" H 1817 4755 50  0000 L CNN
 F 2 "Capacitor_SMD:C_0805_2012Metric" H 1725 4800 50  0001 C CNN
@@
 $EndComp
 $Comp
-L Device:C_Small C?
+L Device:C_Small C45
 U 1 1 5EF2450A
 P 1325 5550
-F 0 "C?" H 1417 5596 50  0000 L CNN
-F 1 ".1" H 1417 5505 50  0000 L CNN
+F 0 "C45" H 1417 5596 50  0000 L CNN
+F 1 ".1uF" H 1417 5505 50  0000 L CNN
 F 2 "Capacitor_SMD:C_0402_1005Metric" H 1325 5550 50  0001 C CNN
 F 3 "~" H 1325 5550 50  0001 C CNN
@@
 $EndComp
 $Comp
-L power:GNDA #PWR?
+L power:GNDA #PWR0106
 U 1 1 5EF24514
 P 1125 5650
-F 0 "#PWR?" H 1125 5400 50  0001 C CNN
+F 0 "#PWR0106" H 1125 5400 50  0001 C CNN
 F 1 "GNDA" H 1130 5477 50  0000 C CNN
 F 2 "" H 1125 5650 50  0001 C CNN
@@
 $EndComp
 $Comp
-L power:GNDA #PWR?
+L power:GNDA #PWR0107
 U 1 1 5EF2451E
 P 3125 6600
-F 0 "#PWR?" H 3125 6350 50  0001 C CNN
+F 0 "#PWR0107" H 3125 6350 50  0001 C CNN
 F 1 "GNDA" H 3130 6427 50  0000 C CNN
 F 2 "" H 3125 6600 50  0001 C CNN
@@
 $EndComp
 $Comp
-L Scott:GND #PWR?
+L Scott:GND #PWR0108
 U 1 1 5EF24528
 P 2625 6600
-F 0 "#PWR?" H 2625 6350 50  0001 C CNN
+F 0 "#PWR0108" H 2625 6350 50  0001 C CNN
 F 1 "GND" H 2630 6427 50  0000 C CNN
 F 2 "" H 2625 6600 50  0001 C CNN
@@
 $EndComp
 $Comp
-L Device:R_Small_US R?
+L Device:R_Small_US R28
 U 1 1 5EF24537
 P 1475 6150
-F 0 "R?" H 1275 6200 50  0000 L CNN
+F 0 "R28" H 1275 6200 50  0000 L CNN
 F 1 "30.1K" H 1200 6100 50  0000 L CNN
 F 2 "Resistor_SMD:R_0402_1005Metric" H 1475 6150 50  0001 C CNN
@@
 $EndComp
 $Comp
-L Device:R_Small_US R?
+L Device:R_Small_US R29
 U 1 1 5EF24546
 P 1675 6150
-F 0 "R?" H 1475 6100 50  0000 L CNN
+F 0 "R29" H 1475 6100 50  0000 L CNN
 F 1 "6.98K" H 1400 6200 50  0000 L CNN
 F 2 "Resistor_SMD:R_0402_1005Metric" H 1675 6150 50  0001 C CNN
@@
 $EndComp
 $Comp
-L power:GNDA #PWR?
+L power:GNDA #PWR0109
 U 1 1 5EF24550
 P 1475 6300
-F 0 "#PWR?" H 1475 6050 50  0001 C CNN
+F 0 "#PWR0109" H 1475 6050 50  0001 C CNN
 F 1 "GNDA" H 1480 6127 50  0000 C CNN
 F 2 "" H 1475 6300 50  0001 C CNN
@@
 $EndComp
 $Comp
-L Scott:GND #PWR?
+L Scott:GND #PWR0110
 U 1 1 5EF2455A
 P 1325 5650
-F 0 "#PWR?" H 1325 5400 50  0001 C CNN
+F 0 "#PWR0110" H 1325 5400 50  0001 C CNN
 F 1 "GND" H 1330 5477 50  0000 C CNN
 F 2 "" H 1325 5650 50  0001 C CNN
@@
 $EndComp
 $Comp
-L Scott:GND #PWR?
+L Scott:GND #PWR0111
 U 1 1 5EF24564
 P 1675 6300
-F 0 "#PWR?" H 1675 6050 50  0001 C CNN
+F 0 "#PWR0111" H 1675 6050 50  0001 C CNN
 F 1 "GND" H 1680 6127 50  0000 C CNN
 F 2 "" H 1675 6300 50  0001 C CNN
@@
 $EndComp
 $Comp
-L Scott:GND #PWR?
+L Scott:GND #PWR0112
 U 1 1 5EF2456E
 P 1425 4950
-F 0 "#PWR?" H 1425 4700 50  0001 C CNN
+F 0 "#PWR0112" H 1425 4700 50  0001 C CNN
 F 1 "GND" H 1430 4777 50  0000 C CNN
 F 2 "" H 1425 4950 50  0001 C CNN
@@
 $EndComp
 $Comp
-L Device:L L?
+L Device:L L3
 U 1 1 5EF2457D
 P 3775 4700
-F 0 "L?" V 3965 4700 50  0000 C CNN
+F 0 "L3" V 3965 4700 50  0000 C CNN
 F 1 ".56uH" V 3874 4700 50  0000 C CNN
 F 2 "Scott:L_13.5x12.5mm_H6mm" H 3775 4700 50  0001 C CNN
@@
 $EndComp
 $Comp
-L Device:C_Small C?
+L Device:C_Small C36
 U 1 1 5EF2458C
 P 3475 4850
-F 0 "C?" H 3567 4896 50  0000 L CNN
+F 0 "C36" H 3567 4896 50  0000 L CNN
 F 1 ".1uF" H 3567 4805 50  0000 L CNN
 F 2 "Capacitor_SMD:C_0402_1005Metric" H 3475 4850 50  0001 C CNN
@@
 $EndComp
 $Comp
-L Device:C_Small C?
+L Device:C_Small C47
 U 1 1 5EF2459B
 P 3425 6200
-F 0 "C?" H 3333 6154 50  0000 R CNN
+F 0 "C47" H 3333 6154 50  0000 R CNN
 F 1 ".1uF" H 3333 6245 50  0000 R CNN
 F 2 "Capacitor_SMD:C_0402_1005Metric" H 3425 6200 50  0001 C CNN
@@
 $EndComp
 $Comp
-L Device:C_Small C?
+L Device:C_Small C46
 U 1 1 5EF245AA
 P 3575 5900
-F 0 "C?" V 3675 5900 50  0000 C CNN
+F 0 "C46" V 3675 5900 50  0000 C CNN
 F 1 ".1uF" V 3475 5850 50  0000 C CNN
 F 2 "Capacitor_SMD:C_0402_1005Metric" H 3575 5900 50  0001 C CNN
@@
 $EndComp
 $Comp
-L Device:C_Small C?
+L Device:C_Small C37
 U 1 1 5EF245B9
 P 4375 5175
-F 0 "C?" H 4283 5129 50  0000 R CNN
+F 0 "C37" H 4283 5129 50  0000 R CNN
 F 1 ".1uF" H 4283 5220 50  0000 R CNN
 F 2 "Capacitor_SMD:C_0402_1005Metric" H 4375 5175 50  0001 C CNN
@@
 $EndComp
 $Comp
-L power:GNDA #PWR?
+L power:GNDA #PWR0113
 U 1 1 5EF245C3
 P 3425 6400
-F 0 "#PWR?" H 3425 6150 50  0001 C CNN
+F 0 "#PWR0113" H 3425 6150 50  0001 C CNN
 F 1 "GNDA" H 3430 6227 50  0000 C CNN
 F 2 "" H 3425 6400 50  0001 C CNN
@@
 $EndComp
 $Comp
-L Scott:GND #PWR?
+L Scott:GND #PWR0114
 U 1 1 5EF245CD
 P 4375 5900
-F 0 "#PWR?" H 4375 5650 50  0001 C CNN
+F 0 "#PWR0114" H 4375 5650 50  0001 C CNN
 F 1 "GND" H 4380 5727 50  0000 C CNN
 F 2 "" H 4375 5900 50  0001 C CNN
@@
 $EndComp
 $Comp
-L Device:C_Small C?
+L Device:C_Small C38
 U 1 1 5EF245DC
 P 4725 5175
-F 0 "C?" H 4633 5129 50  0000 R CNN
+F 0 "C38" H 4633 5129 50  0000 R CNN
 F 1 "22uF" H 4633 5220 50  0000 R CNN
 F 2 "Capacitor_SMD:C_0805_2012Metric" H 4725 5175 50  0001 C CNN
@@
 $EndComp
 $Comp
-L Device:C_Small C?
+L Device:C_Small C42
 U 1 1 5EF245EB
 P 5075 5175
-F 0 "C?" H 4983 5129 50  0000 R CNN
+F 0 "C42" H 4983 5129 50  0000 R CNN
 F 1 "22uF" H 4983 5220 50  0000 R CNN
 F 2 "Capacitor_SMD:C_0805_2012Metric" H 5075 5175 50  0001 C CNN
@@
 $EndComp
 $Comp
-L Device:C_Small C?
+L Device:C_Small C43
 U 1 1 5EF245FA
 P 5425 5175
-F 0 "C?" H 5333 5129 50  0000 R CNN
+F 0 "C43" H 5333 5129 50  0000 R CNN
 F 1 "100uF" H 5333 5220 50  0000 R CNN
 F 2 "Capacitor_SMD:C_1210_3225Metric" H 5425 5175 50  0001 C CNN
@@
 $EndComp
 $Comp
-L Device:C_Small C?
+L Device:C_Small C44
 U 1 1 5EF24609
 P 5825 5175
-F 0 "C?" H 5733 5129 50  0000 R CNN
+F 0 "C44" H 5733 5129 50  0000 R CNN
 F 1 "100uF" H 5733 5220 50  0000 R CNN
 F 2 "Capacitor_SMD:C_1210_3225Metric" H 5825 5175 50  0001 C CNN
@@
 	-1   0    0    1
 $EndComp
-Text Label 925  4700 0    50   ~ 0
-+12V
-Text Label 5875 4700 0    50   ~ 0
-3V3
-Text Label 1675 5100 0    50   ~ 0
-EN_VDD
 Wire Wire Line
 	1975 4850 1975 4700
@@
 	3425 6300 3425 6400
 Wire Wire Line
-	1675 5100 1975 5100
+	1925 5100 1975 5100
 Wire Wire Line
 	3925 4700 4075 4700
@@
 	3425 5700 3725 5700
 $Comp
-L Scott:GND #PWR?
+L Scott:GND #PWR0115
 U 1 1 5EF7ABF6
 P -475 -500
-F 0 "#PWR?" H -475 -750 50  0001 C CNN
+F 0 "#PWR0115" H -475 -750 50  0001 C CNN
 F 1 "GND" H -470 -673 50  0000 C CNN
 F 2 "" H -475 -500 50  0001 C CNN
@@
 $EndComp
 $Comp
-L Scott:GND #PWR?
+L Scott:GND #PWR0116
 U 1 1 5EF7BF91
 P -50 -500
-F 0 "#PWR?" H -50 -750 50  0001 C CNN
+F 0 "#PWR0116" H -50 -750 50  0001 C CNN
 F 1 "GND" H -45 -673 50  0000 C CNN
 F 2 "" H -50 -500 50  0001 C CNN
@@
 	1    0    0    -1
 $EndComp
+Wire Wire Line
+	1975 5250 1700 5250
+Text GLabel 1700 5250 0    50   Input ~ 0
+3V3_PG
+Text GLabel 6200 4700 2    50   Input ~ 0
+3V3
+Text GLabel 925  4700 0    50   Input ~ 0
+12V
+Text GLabel 1925 5100 0    50   Input ~ 0
+EN_3V3
+Text GLabel 5625 1500 2    50   Input ~ 0
+CPU_VDD
+Text GLabel 800  1500 0    50   Input ~ 0
+12V
+Text GLabel 1650 1900 0    50   Input ~ 0
+EN_VDD
+Text GLabel 1650 2050 0    50   Input ~ 0
+CPU_VDD_PG
+Wire Wire Line
+	1700 2050 1650 2050
+Text GLabel 3800 2275 0    50   Input ~ 0
+CPU_VDD_SENSE
+Text GLabel 3800 2400 0    50   Input ~ 0
+CPU_GND_SENSE
+$Comp
+L Scott:GND #PWR0118
+U 1 1 5F0B155A
+P -625 2400
+F 0 "#PWR0118" H -625 2150 50  0001 C CNN
+F 1 "GND" H -620 2227 50  0000 C CNN
+F 2 "" H -625 2400 50  0001 C CNN
+F 3 "" H -625 2400 50  0001 C CNN
+	1    -625 2400
+	1    0    0    -1
+$EndComp
+Wire Wire Line
+	3450 2500 3800 2500
+Wire Wire Line
+	3800 2150 3800 2275
+Connection ~ 3800 2150
+Wire Wire Line
+	3800 2400 3800 2500
+Connection ~ 3800 2500
+Wire Wire Line
+	3800 2500 4100 2500
 $EndSCHEMATC
