File: AP2100/AP2100.kicad_pcb (KiCad board)
At the start: 6 copper layers, 150 x 150 mm, 231 parts, among them IC1 FDS86242, IC1 PM8805TR, IC2 PM8804TR, IC3 AS4C256M16D4-75BINTR, IC4 AS4C256M16D4-75BINTR, J1 Bus_PCI_Express_Mini, J2 Bus_PCI_Express_Mini, J3 Bus_PCI_Express_Mini, J4 0826-1X1T-GH-F, J5 Barrel_Jack, Q1 HMHA2801AR2, Q1 PBSS4240T, Q2 BSC190N15NS3GATMA1, Q3 PBSS4240T, Q4 FDMC86259P, Q5 FOD817AS, U1 LS1043ASE7KQB, U1 TPS23751PWP, U2 MPQ8634AGLE-P, U2 TL431DBV, U3 MPQ8634AGLE-P, U4 STL90N6F7, U5 STL90N6F7, U6 TS2431-AILT

Commit message: Add + route first 16 memory data lines
Parts:
- added C59: 1uF, Capacitor_SMD:C_0402_1005Metric, F.Cu at (370.9, 98.0)
- added C72: 1uF, Capacitor_SMD:C_0402_1005Metric, F.Cu at (381.1, 91.1)
- added C73: 1uF, Capacitor_SMD:C_0402_1005Metric, F.Cu at (370.9, 94.0)
- added C74: 1uF, Capacitor_SMD:C_0402_1005Metric, F.Cu at (384.0, 91.1)
- added C75: .1uF, Capacitor_SMD:C_0402_1005Metric, F.Cu at (376.7, 97.0)
- added C76: .1uF, Capacitor_SMD:C_0402_1005Metric, F.Cu at (373.8, 96.0)
- added C77: .1uF, Capacitor_SMD:C_0402_1005Metric, F.Cu at (372.3, 100.0)
- added C78: .1uF, Capacitor_SMD:C_0402_1005Metric, F.Cu at (375.2, 100.0)
- added C79: .1uF, Capacitor_SMD:C_0402_1005Metric, F.Cu at (370.9, 96.0)
- added C80: .1uF, Capacitor_SMD:C_0402_1005Metric, F.Cu at (382.5, 93.1)
- added C81: .1uF, Capacitor_SMD:C_0402_1005Metric, F.Cu at (373.8, 94.0)
- added C82: .1uF, Capacitor_SMD:C_0402_1005Metric, F.Cu at (376.7, 95.0)
- added C83: 10uF, Capacitor_SMD:C_0805_2012Metric, F.Cu at (367.2, 97.5)
- added C84: 10uF, Capacitor_SMD:C_0805_2012Metric, F.Cu at (371.6, 91.5)
- added C85: .1uF, Capacitor_SMD:C_0402_1005Metric, F.Cu at (369.4, 100.0)
- added C86: .1uF, Capacitor_SMD:C_0402_1005Metric, F.Cu at (376.7, 93.1)
- added C87: .1uF, Capacitor_SMD:C_0402_1005Metric, F.Cu at (366.5, 99.9)
- added C88: .1uF, Capacitor_SMD:C_0402_1005Metric, F.Cu at (373.8, 98.0)
- added C89: .1uF, Capacitor_SMD:C_0402_1005Metric, F.Cu at (378.2, 91.1)
- added C90: .1uF, Capacitor_SMD:C_0402_1005Metric, F.Cu at (375.3, 91.1)
- added C91: .1uF, Capacitor_SMD:C_0402_1005Metric, F.Cu at (379.6, 93.1)
- added C92: .1uF, Capacitor_SMD:C_0402_1005Metric, F.Cu at (379.6, 95.0)
- added C93: 10uF, Capacitor_SMD:C_0805_2012Metric, F.Cu at (367.2, 91.5)
- added C94: 10uF, Capacitor_SMD:C_0805_2012Metric, F.Cu at (367.2, 94.5)
- added C95: 100pF, Capacitor_SMD:C_0805_2012Metric, F.Cu at (391.0, 98.5)
- added D19: BAS16J, Diode_SMD:D_SOD-323, F.Cu at (403.8, 91.5)
- added D22: BZX84C10, Package_TO_SOT_SMD:SOT-23, F.Cu at (399.4, 92.3)
- added Q3: PBSS4240T, Package_TO_SOT_SMD:SOT-23, F.Cu at (399.4, 96.9)
- added R26: 1K, Resistor_SMD:R_0603_1608Metric, F.Cu at (403.7, 96.8)
- added R27: 22, Resistor_SMD:R_0603_1608Metric, F.Cu at (403.7, 94.3)
- added R33: 10K, Resistor_SMD:R_0603_1608Metric, F.Cu at (395.2, 98.2)
- added U5: STL90N6F7, Scott:TRANS_STL60P4LLF6, F.Cu at (393.4, 93.5)
- IC3, IC4: value AS4C256M16D4-75BINTR -> AS4C256M16D4-75BCN; footprint LIB_AS4C256M16D4-75BINTR:BGA96C80P9X16_750X1350X120 -> Scott:BGA96C80P9X16_750X1350X120
- moved IC3 337.5 mm to (79.8, 100.2)
Connections:
- net Net-(U1-PadA22) renamed /CPU Memory/DDR4_MECC1
- net Net-(U1-PadC22) renamed /CPU Memory/DDR4_MECC0
- net Net-(U1-PadD22) renamed /CPU Memory/DDR4_MECC2
- net Net-(U1-PadD23) renamed /CPU Memory/DDR4_MECC3
- IC2 pad 8: Net-(C44-Pad1) -> GNDPWR
- IC3 pad A1: Net-(IC3-PadA1) -> +GVDD
- IC3 pad A2: Net-(IC3-PadA2) -> CPU_GND_SENSE
- IC3 pad A3: Net-(IC3-PadA3) -> /CPU Memory/DDR4_DQ8
- IC3 pad A8: Net-(IC3-PadA8) -> CPU_GND_SENSE
- IC3 pad A9: Net-(IC3-PadA9) -> +GVDD
- IC3 pad B1: Net-(IC3-PadB1) -> 2V5_VPP
- IC3 pad B2: Net-(IC3-PadB2) -> CPU_GND_SENSE
- IC3 pad B3: Net-(IC3-PadB3) -> +GVDD
- IC3 pad B8: Net-(IC3-PadB8) -> /CPU Memory/DDR4_DQ9
- IC3 pad B9: Net-(IC3-PadB9) -> +GVDD
- IC3 pad C1: Net-(IC3-PadC1) -> +GVDD
- IC3 pad C2: Net-(IC3-PadC2) -> /CPU Memory/DDR4_DQ12
- IC3 pad C3: Net-(IC3-PadC3) -> /CPU Memory/DDR4_DQ10
- IC3 pad C7: Net-(IC3-PadC7) -> /CPU Memory/DDR4_DQ11
- IC3 pad C8: Net-(IC3-PadC8) -> /CPU Memory/DDR4_DQ13
- IC3 pad C9: Net-(IC3-PadC9) -> CPU_GND_SENSE
- IC3 pad D1: Net-(IC3-PadD1) -> +GVDD
- IC3 pad D2: Net-(IC3-PadD2) -> CPU_GND_SENSE
- IC3 pad D3: Net-(IC3-PadD3) -> /CPU Memory/DDR4_DQ14
- IC3 pad D7: Net-(IC3-PadD7) -> /CPU Memory/DDR4_DQ15
- IC3 pad D8: Net-(IC3-PadD8) -> CPU_GND_SENSE
- IC3 pad D9: Net-(IC3-PadD9) -> +GVDD
- IC3 pad E1: Net-(IC3-PadE1) -> CPU_GND_SENSE
- IC3 pad E3: Net-(IC3-PadE3) -> CPU_GND_SENSE
- IC3 pad E8: Net-(IC3-PadE8) -> CPU_GND_SENSE
- IC3 pad E9: Net-(IC3-PadE9) -> CPU_GND_SENSE
- IC3 pad F1: Net-(IC3-PadF1) -> CPU_GND_SENSE
- IC3 pad F2: Net-(IC3-PadF2) -> +GVDD
- IC3 pad F7: Net-(IC3-PadF7) -> /CPU Memory/DDR4_DQ1
- IC3 pad F8: Net-(IC3-PadF8) -> +GVDD
- IC3 pad G1: Net-(IC3-PadG1) -> +GVDD
- IC3 pad G2: Net-(IC3-PadG2) -> /CPU Memory/DDR4_DQ0
- IC3 pad G7: Net-(IC3-PadG7) -> +GVDD
- IC3 pad G8: Net-(IC3-PadG8) -> CPU_GND_SENSE
- IC3 pad G9: Net-(IC3-PadG9) -> +GVDD
- IC3 pad H1: Net-(IC3-PadH1) -> CPU_GND_SENSE
- IC3 pad H2: Net-(IC3-PadH2) -> /CPU Memory/DDR4_DQ4
- IC3 pad H3: Net-(IC3-PadH3) -> /CPU Memory/DDR4_DQ2
- IC3 pad H7: Net-(IC3-PadH7) -> /CPU Memory/DDR4_DQ3
- IC3 pad H8: Net-(IC3-PadH8) -> /CPU Memory/DDR4_DQ5
- IC3 pad H9: Net-(IC3-PadH9) -> CPU_GND_SENSE
- IC3 pad J1: Net-(IC3-PadJ1) -> +GVDD
- IC3 pad J2: Net-(IC3-PadJ2) -> +GVDD
- IC3 pad J3: Net-(IC3-PadJ3) -> /CPU Memory/DDR4_DQ6
- IC3 pad J7: Net-(IC3-PadJ7) -> /CPU Memory/DDR4_DQ7
- IC3 pad J8: Net-(IC3-PadJ8) -> +GVDD
- IC3 pad J9: Net-(IC3-PadJ9) -> +GVDD
- IC3 pad K1: Net-(IC3-PadK1) -> CPU_GND_SENSE
- IC3 pad K9: Net-(IC3-PadK9) -> CPU_GND_SENSE
- IC3 pad L1: Net-(IC3-PadL1) -> +GVDD
- IC3 pad L9: Net-(IC3-PadL9) -> +GVDD
- IC3 pad M9: Net-(IC3-PadM9) -> CPU_GND_SENSE
- IC3 pad N1: Net-(IC3-PadN1) -> CPU_GND_SENSE
- IC3 pad R1: Net-(IC3-PadR1) -> +GVDD
- IC3 pad R9: Net-(IC3-PadR9) -> 2V5_VPP
- IC3 pad T1: Net-(IC3-PadT1) -> CPU_GND_SENSE
- IC3 pad T9: Net-(IC3-PadT9) -> +GVDD
- IC4 pad A1: Net-(IC4-PadA1) -> +GVDD
- IC4 pad A2: Net-(IC4-PadA2) -> CPU_GND_SENSE
- IC4 pad A8: Net-(IC4-PadA8) -> CPU_GND_SENSE
- IC4 pad A9: Net-(IC4-PadA9) -> +GVDD
- IC4 pad B1: Net-(IC4-PadB1) -> 2V5_VPP
- IC4 pad B2: Net-(IC4-PadB2) -> CPU_GND_SENSE
- IC4 pad B3: Net-(IC4-PadB3) -> +GVDD
- IC4 pad B9: Net-(IC4-PadB9) -> +GVDD
- IC4 pad C1: Net-(IC4-PadC1) -> +GVDD
- IC4 pad C9: Net-(IC4-PadC9) -> CPU_GND_SENSE
- IC4 pad D1: Net-(IC4-PadD1) -> +GVDD
- IC4 pad D2: Net-(IC4-PadD2) -> CPU_GND_SENSE
- IC4 pad D8: Net-(IC4-PadD8) -> CPU_GND_SENSE
- IC4 pad D9: Net-(IC4-PadD9) -> +GVDD
- IC4 pad E1: Net-(IC4-PadE1) -> CPU_GND_SENSE
- IC4 pad E3: Net-(IC4-PadE3) -> CPU_GND_SENSE
- IC4 pad E8: Net-(IC4-PadE8) -> CPU_GND_SENSE
- IC4 pad E9: Net-(IC4-PadE9) -> CPU_GND_SENSE
- IC4 pad F1: Net-(IC4-PadF1) -> CPU_GND_SENSE
- IC4 pad F2: Net-(IC4-PadF2) -> +GVDD
- IC4 pad F8: Net-(IC4-PadF8) -> +GVDD
- IC4 pad G1: Net-(IC4-PadG1) -> +GVDD
- IC4 pad G7: Net-(IC4-PadG7) -> +GVDD
- IC4 pad G8: Net-(IC4-PadG8) -> CPU_GND_SENSE
- IC4 pad G9: Net-(IC4-PadG9) -> +GVDD
- IC4 pad H1: Net-(IC4-PadH1) -> CPU_GND_SENSE
- IC4 pad H9: Net-(IC4-PadH9) -> CPU_GND_SENSE
- IC4 pad J1: Net-(IC4-PadJ1) -> +GVDD
- IC4 pad J2: Net-(IC4-PadJ2) -> +GVDD
- IC4 pad J8: Net-(IC4-PadJ8) -> +GVDD
- IC4 pad J9: Net-(IC4-PadJ9) -> +GVDD
- IC4 pad K1: Net-(IC4-PadK1) -> CPU_GND_SENSE
- IC4 pad K9: Net-(IC4-PadK9) -> CPU_GND_SENSE
- IC4 pad L1: Net-(IC4-PadL1) -> +GVDD
- IC4 pad L9: Net-(IC4-PadL9) -> +GVDD
- IC4 pad M9: Net-(IC4-PadM9) -> CPU_GND_SENSE
- IC4 pad N1: Net-(IC4-PadN1) -> CPU_GND_SENSE
- IC4 pad R1: Net-(IC4-PadR1) -> +GVDD
- IC4 pad R9: Net-(IC4-PadR9) -> 2V5_VPP
- IC4 pad T1: Net-(IC4-PadT1) -> CPU_GND_SENSE
- IC4 pad T9: Net-(IC4-PadT9) -> +GVDD
- R25 pad 1: Net-(C44-Pad1) -> GNDPWR
- R38 pad 1: Net-(R38-Pad1) -> 12V0
- R38 pad 2: 12V0 -> Net-(R38-Pad2)
- R41 pad 1: Net-(R38-Pad1) -> Net-(R38-Pad2)
- R44 pad 2: Net-(R38-Pad1) -> Net-(R38-Pad2)
- TR1 pad 6: Net-(TR1-Pad6) -> Net-(C53-Pad1)
- TR1 pad 7: Net-(TR1-Pad6) -> Net-(C53-Pad1)
- U1 pad H24: Net-(U1-PadH24) -> /CPU Memory/DDR4_DQ7
- U1 pad J25: Net-(U1-PadJ25) -> /CPU Memory/DDR4_DQ3
- U1 pad K21: Net-(U1-PadK21) -> /CPU Memory/DDR4_DQ15
- U1 pad K24: Net-(U1-PadK24) -> /CPU Memory/DDR4_DQ1
- U1 pad K25: Net-(U1-PadK25) -> /CPU Memory/DDR4_DQ5
- U1 pad L22: Net-(U1-PadL22) -> /CPU Memory/DDR4_DQ13
- U1 pad L23: Net-(U1-PadL23) -> /CPU Memory/DDR4_DQ11
- U1 pad M21: Net-(U1-PadM21) -> /CPU Memory/DDR4_DQ12
- U1 pad M23: Net-(U1-PadM23) -> /CPU Memory/DDR4_DQ9
- U1 pad N21: Net-(U1-PadN21) -> /CPU Memory/DDR4_DQ8
- U1 pad N24: Net-(U1-PadN24) -> /CPU Memory/DDR4_DQ0
- U1 pad N25: Net-(U1-PadN25) -> /CPU Memory/DDR4_DQ6
- U1 pad P21: Net-(U1-PadP21) -> /CPU Memory/DDR4_DQ10
- U1 pad P23: Net-(U1-PadP23) -> /CPU Memory/DDR4_DQ14
- U1 pad P25: Net-(U1-PadP25) -> /CPU Memory/DDR4_DQ4
- U1 pad R24: Net-(U1-PadR24) -> /CPU Memory/DDR4_DQ2
Routing:
- net /CPU Memory/DDR4_DQ3: track 0.00 -> 24.0 mm, vias 0 -> 2
- net /CPU Memory/DDR4_DQ5: track 0.00 -> 24.0 mm, vias 0 -> 2
- net /CPU Memory/DDR4_DQ7: track 0.00 -> 24.0 mm, vias 0 -> 2
- net /CPU Memory/DDR4_DQ1: track 0.00 -> 18.9 mm, vias 0 -> 2
- net /CPU Memory/DDR4_DQ4: track 0.00 -> 18.5 mm, vias 0 -> 2
- net /CPU Memory/DDR4_DQ0: track 0.00 -> 18.1 mm, vias 0 -> 2
- net /CPU Memory/DDR4_DQ6: track 0.00 -> 16.1 mm, vias 0 -> 2
- net /CPU Memory/DDR4_DQ2: track 0.00 -> 12.9 mm, vias 0 -> 2
- net (no net): track 10.9 -> 8.33 mm
- net Net-(U1-PadR24): track 2.57 -> 0.00 mm
- net Net-(U1-PadN24): track 2.57 -> 0.00 mm
- net Net-(U1-PadN23): track 3.53 -> 2.40 mm, vias 1 -> 0
- net /CPU Memory/DDR4_DQ9: track 0.00 -> 1.12 mm, vias 0 -> 2
- net /CPU Memory/DDR4_DQ8: track 0.00 -> 1.12 mm, vias 0 -> 2
- net /CPU Memory/DDR4_DQ15: track 0.00 -> 1.12 mm, vias 0 -> 2
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
Commit message: Almost finish memory section
Parts:
- moved IC4 346.5 mm to (64.8, 120.9)
- moved IC3 32.9 mm to (54.3, 120.9)
- turned U1 to -90 degrees
Connections:
- IC4 pad A3: Net-(IC4-PadA3) -> /CPU Memory/DDR4_DQ24
- IC4 pad B8: Net-(IC4-PadB8) -> /CPU Memory/DDR4_DQ25
- IC4 pad C2: Net-(IC4-PadC2) -> /CPU Memory/DDR4_DQ28
- IC4 pad C3: Net-(IC4-PadC3) -> /CPU Memory/DDR4_DQ26
- IC4 pad C7: Net-(IC4-PadC7) -> /CPU Memory/DDR4_DQ27
- IC4 pad C8: Net-(IC4-PadC8) -> /CPU Memory/DDR4_DQ29
- IC4 pad D3: Net-(IC4-PadD3) -> /CPU Memory/DDR4_DQ30
- IC4 pad D7: Net-(IC4-PadD7) -> /CPU Memory/DDR4_DQ31
- IC4 pad F7: Net-(IC4-PadF7) -> /CPU Memory/DDR4_DQ17
- IC4 pad G2: Net-(IC4-PadG2) -> /CPU Memory/DDR4_DQ16
- IC4 pad H2: Net-(IC4-PadH2) -> /CPU Memory/DDR4_DQ20
- IC4 pad H3: Net-(IC4-PadH3) -> /CPU Memory/DDR4_DQ18
- IC4 pad H7: Net-(IC4-PadH7) -> /CPU Memory/DDR4_DQ19
- IC4 pad H8: Net-(IC4-PadH8) -> /CPU Memory/DDR4_DQ21
- IC4 pad J3: Net-(IC4-PadJ3) -> /CPU Memory/DDR4_DQ22
- IC4 pad J7: Net-(IC4-PadJ7) -> /CPU Memory/DDR4_DQ23
- U1 pad B24: Net-(U1-PadB24) -> /CPU Memory/DDR4_DQ20
- U1 pad C24: Net-(U1-PadC24) -> /CPU Memory/DDR4_DQ16
- U1 pad C25: Net-(U1-PadC25) -> /CPU Memory/DDR4_DQ17
- U1 pad D24: Net-(U1-PadD24) -> /CPU Memory/DDR4_DQ21
- U1 pad F22: Net-(U1-PadF22) -> /CPU Memory/DDR4_DQ24
- U1 pad F23: Net-(U1-PadF23) -> /CPU Memory/DDR4_DQ29
- U1 pad F24: Net-(U1-PadF24) -> /CPU Memory/DDR4_DQ18
- U1 pad F25: Net-(U1-PadF25) -> /CPU Memory/DDR4_DQ22
- U1 pad G21: Net-(U1-PadG21) -> /CPU Memory/DDR4_DQ28
- U1 pad G25: Net-(U1-PadG25) -> /CPU Memory/DDR4_DQ23
- U1 pad H21: Net-(U1-PadH21) -> /CPU Memory/DDR4_DQ25
- U1 pad H24: /CPU Memory/DDR4_DQ7 -> /CPU Memory/DDR4_DQ4
- U1 pad H25: Net-(U1-PadH25) -> /CPU Memory/DDR4_DQ19
- U1 pad J21: Net-(U1-PadJ21) -> /CPU Memory/DDR4_DQ30
- U1 pad J22: Net-(U1-PadJ22) -> /CPU Memory/DDR4_DQ31
- U1 pad J23: Net-(U1-PadJ23) -> /CPU Memory/DDR4_DQ26
- U1 pad J25: /CPU Memory/DDR4_DQ3 -> /CPU Memory/DDR4_DQ0
- U1 pad K21: /CPU Memory/DDR4_DQ15 -> /CPU Memory/DDR4_DQ12
- U1 pad K23: Net-(U1-PadK23) -> /CPU Memory/DDR4_DQ27
- U1 pad L23: /CPU Memory/DDR4_DQ11 -> /CPU Memory/DDR4_DQ8
- U1 pad M21: /CPU Memory/DDR4_DQ12 -> /CPU Memory/DDR4_DQ14
- U1 pad N21: /CPU Memory/DDR4_DQ8 -> /CPU Memory/DDR4_DQ10
- U1 pad N24: /CPU Memory/DDR4_DQ0 -> /CPU Memory/DDR4_DQ2
- U1 pad P21: /CPU Memory/DDR4_DQ10 -> /CPU Memory/DDR4_DQ11
- U1 pad P23: /CPU Memory/DDR4_DQ14 -> /CPU Memory/DDR4_DQ15
- U1 pad P25: /CPU Memory/DDR4_DQ4 -> /CPU Memory/DDR4_DQ7
- U1 pad R24: /CPU Memory/DDR4_DQ2 -> /CPU Memory/DDR4_DQ3
Routing:
- net /CPU Memory/DDR4_DQ3: track 24.0 -> 0.56 mm, vias 2 -> 1
- net /CPU Memory/DDR4_DQ5: track 24.0 -> 0.56 mm, vias 2 -> 1
- net /CPU Memory/DDR4_DQ7: track 24.0 -> 0.56 mm, vias 2 -> 1
- net /CPU Memory/DDR4_DQ1: track 18.9 -> 0.56 mm, vias 2 -> 1
- net /CPU Memory/DDR4_DQ4: track 18.5 -> 0.56 mm, vias 2 -> 1
- net /CPU Memory/DDR4_DQ0: track 18.1 -> 0.56 mm, vias 2 -> 1
- net /CPU Memory/DDR4_DQ6: track 16.1 -> 0.56 mm, vias 2 -> 1
- net /CPU Memory/DDR4_DQ2: track 12.9 -> 0.56 mm, vias 2 -> 1
- net (no net): track 8.33 -> 3.60 mm, vias 2 -> 0
- net Net-(U1-PadU22): track 4.17 -> 0.00 mm, vias 1 -> 0
- net Net-(U1-PadT23): track 3.37 -> 0.00 mm
- net Net-(U1-PadN23): track 2.40 -> 0.00 mm
- net Net-(U1-PadV25): track 1.60 -> 0.00 mm
- net Net-(U1-PadU25): track 1.60 -> 0.00 mm
- net Net-(U1-PadT25): track 1.60 -> 0.00 mm
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
Commit message: Annotate and update PCB with current design
Parts:
- removed the C1 at (126.4, 111.4)
- removed the C1 at (173.1, 82.8)
- removed the C10 at (132.2, 113.8)
- removed the C10 at (175.0, 87.4)
- removed the C11 at (144.7, 106.2)
- removed the C11 at (183.8, 75.0)
- removed the C12 at (126.5, 106.9)
- removed the C12 at (175.0, 119.0)
- removed the C13 at (183.6, 44.3)
- removed the C13 at (101.8, 93.0)
- removed the C14 at (205.2, 33.4)
- removed the C14 at (184.8, 114.9)
- removed the C15 at (188.0, 44.3)
- removed the C15 at (190.1, 102.0)
- removed the C16 at (191.6, 45.8)
- removed the C16 at (174.8, 121.7)
- removed the C17 at (194.5, 43.8)
- removed the C17 at (195.6, 104.3)
- removed the C18 at (183.6, 47.2)
- removed the C18 at (194.3, 101.8)
- removed the C19 at (188.0, 47.2)
- removed the C19 at (185.7, 109.9)
- removed the C2 at (123.8, 111.5)
- removed the C2 at (182.3, 78.7)
- removed the C20 at (205.8, 29.9)
- removed the C20 at (195.8, 98.6)
- removed the C3 at (140.6, 98.1)
- removed the C3 at (88.0, 84.8)
- removed the C31 at (251.1, 39.1)
- removed the C31 at (198.4, 2.59)
- removed the C4 at (140.6, 101.1)
- removed the C4 at (102.3, 79.5)
- removed the C5 at (130.8, 106.2)
- removed the C5 at (102.3, 82.8)
- removed the C59 at (370.9, 98.0)
- removed the C59 at (-579.3, -446.7)
- removed the C6 at (141.0, 106.7)
- removed the C6 at (102.2, 85.8)
- removed the C7 at (141.0, 109.6)
- removed the C7 at (163.7, 87.2)
- removed the C71 at (-558.2, -465.2)
- removed the C71 at (-544.9, -466.8)
- removed the C8 at (136.0, 107.3)
- removed the C8 at (169.3, 87.4)
- removed the C9 at (136.0, 111.5)
- removed the C9 at (179.4, 82.4)
- removed the D1 at (208.0, -5.93)
- removed the D1 at (166.4, 76.3)
- removed the D19 at (403.8, 91.5)
- removed the D19 at (-562.8, -454.7)
- removed the D2 at (240.9, 30.8)
- removed the D2 at (96.2, 88.0)
- removed the D22 at (399.4, 92.3)
- removed the D22 at (-551.7, -470.2)
- removed the D3 at (236.1, 43.4)
- removed the D3 at (158.7, 120.8)
- removed the D4 at (225.3, 43.4)
- removed the D4 at (181.8, 105.7)
- removed the D5 at (225.3, 51.1)
- removed the D5 at (190.8, 98.8)
- removed the D6 at (251.8, 30.8)
- removed the D6 at (181.3, 109.8)
- removed IC1: PM8805TR, PM8805TR:PM8805TR
- removed IC1: FDS86242, FDS86242:SOIC127P600X175-8N
- removed IC2: PM8804TR, PM8804TR:QFN50P340X340X90-17N
- removed J3: Bus_PCI_Express_Mini, Connector_PCBEdge:BUS_PCI_Express_Mini_Full
- removed the L1 at (194.8, 35.3)
- removed the L1 at (95.0, 76.8)
- removed the Q1 at (-572.7, -448.5)
- removed the Q1 at (159.5, 116.4)
- removed the Q3 at (399.4, 96.9)
- removed the Q3 at (-540.4, -480.8)
- removed the R1 at (144.7, 108.2)
- removed the R1 at (165.3, 82.7)
- removed the R10 at (250.2, 36.2)
- removed the R10 at (182.8, 121.3)
- removed the R11 at (252.2, 49.8)
- removed the R11 at (187.2, 117.4)
- removed the R12 at (266.3, 28.4)
- removed the R12 at (179.2, 118.8)
- removed the R13 at (268.0, 31.2)
- removed the R13 at (195.6, 106.8)
- removed the R14 at (270.5, 28.2)
- removed the R14 at (183.2, 118.4)
- removed the R15 at (258.8, 36.1)
- removed the R15 at (189.7, 109.9)
- removed the R16 at (252.0, 44.8)
- removed the R16 at (185.7, 112.4)
- removed the R17 at (245.2, 41.4)
- removed the R17 at (187.2, 120.0)
- removed the R18 at (243.4, 54.4)
- removed the R18 at (189.7, 112.4)
- removed the R19 at (255.4, 41.9)
- removed the R19 at (193.7, 112.2)
- removed the R2 at (147.6, 106.2)
- removed the R2 at (102.2, 87.8)
- removed the R20 at (268.0, 33.7)
- removed the R20 at (193.7, 109.7)
- removed the R21 at (247.8, 50.6)
- removed the R21 at (198.3, 101.4)
- removed the R26 at (403.7, 96.8)
- removed the R26 at (-563.2, -445.3)
- removed the R26 at (214.9, -8.81)
- removed the R27 at (403.7, 94.3)
- removed the R27 at (-545.1, -464.2)
- removed the R27 at (192.7, 8.29)
- removed the R3 at (443.9, -28.1)
- removed the R3 at (180.6, 115.7)
- removed the R33 at (395.2, 98.2)
- removed the R33 at (-573.4, -437.0)
- removed the R4 at (443.9, -30.6)
- removed the R4 at (192.8, 114.9)
- removed the R5 at (194.5, 45.8)
- removed the R5 at (188.8, 114.9)
- removed the R6 at (197.5, 43.8)
- removed the R6 at (178.8, 121.7)
- removed the R7 at (259.8, 41.1)
- removed the R7 at (175.6, 115.9)
- removed the R8 at (247.8, 53.1)
- removed the R8 at (191.6, 107.2)
- removed the R9 at (256.0, 44.4)
- removed the R9 at (191.6, 104.7)
- removed the TR1 at (-599.6, -449.4)
- removed the TR1 at (116.0, 85.0)
- removed the U1 at (58.7, 100.0)
- removed the U1 at (104.0, 122.4)
- removed the U2 at (130.8, 111.1)
- removed the U2 at (187.1, 106.3)
- removed the U5 at (393.4, 93.5)
- removed the U5 at (-584.4, -454.5)
- added BT1: CR2032, Battery:BatteryHolder_Keystone_3034_1x20mm, F.Cu at (127.0, 27.5)
- added C1: 22uF, Capacitor_SMD:C_1210_3225Metric, F.Cu at (282.0, 85.7)
- added C10: .1uF, Capacitor_SMD:C_0603_1608Metric, F.Cu at (290.1, 87.8)
- added C100: .22uF, Capacitor_SMD:C_0402_1005Metric, F.Cu at (327.6, 56.4)
- added C101: 1uF, Capacitor_SMD:C_0402_1005Metric, F.Cu at (292.0, 92.5)
- added C103: 4.7uF, Capacitor_SMD:C_0805_2012Metric, F.Cu at (325.6, 46.4)
- added C104: 4.7uF, Capacitor_SMD:C_0805_2012Metric, F.Cu at (319.9, 54.9)
- added C106: 4.7uF, Capacitor_SMD:C_0805_2012Metric, F.Cu at (291.5, 85.0)
- added C107: 4.7uF, Capacitor_SMD:C_0805_2012Metric, F.Cu at (330.2, 42.1)
- added C109: 4.7uF, Capacitor_SMD:C_0805_2012Metric, F.Cu at (297.2, 77.7)
- added C11: .1uF, Capacitor_SMD:C_0603_1608Metric, F.Cu at (290.1, 90.3)
- added C110: .1uF, Capacitor_SMD:C_0402_1005Metric, F.Cu at (293.5, 89.7)
- added C111: 4.7uF, Capacitor_SMD:C_0805_2012Metric, F.Cu at (330.2, 39.1)
- added C112: 4.7uF, Capacitor_SMD:C_0805_2012Metric, F.Cu at (303.3, 64.6)
- added C113: 4.7uF, Capacitor_SMD:C_0805_2012Metric, F.Cu at (299.0, 73.6)
- added C114: 4.7uF, Capacitor_SMD:C_0805_2012Metric, F.Cu at (319.9, 51.9)
- added C115: .1uF, Capacitor_SMD:C_0402_1005Metric, F.Cu at (325.2, 59.4)
- added C116: .1uF, Capacitor_SMD:C_0402_1005Metric, F.Cu at (330.5, 54.4)
- added C117: .1uF, Capacitor_SMD:C_0402_1005Metric, F.Cu at (337.9, 45.6)
- added C118: 22uF, Capacitor_SMD:C_0805_2012Metric, F.Cu at (309.0, 63.4)
- added C119: 22uF, Capacitor_SMD:C_0805_2012Metric, F.Cu at (304.3, 70.7)
- added C12: .1uF, Capacitor_SMD:C_0603_1608Metric, F.Cu at (303.2, 73.4)
- added C120: 22uF, Capacitor_SMD:C_0805_2012Metric, F.Cu at (285.9, 89.3)
- added C121: 22uF, Capacitor_SMD:C_0805_2012Metric, F.Cu at (292.7, 77.7)
- added C122: 22uF, Capacitor_SMD:C_0805_2012Metric, F.Cu at (334.6, 39.1)
- added C123: 22uF, Capacitor_SMD:C_0805_2012Metric, F.Cu at (324.5, 43.4)
- added C124: 22uF, Capacitor_SMD:C_0805_2012Metric, F.Cu at (314.6, 56.1)
- added C125: 22uF, Capacitor_SMD:C_0805_2012Metric, F.Cu at (314.6, 59.1)
- added C126: 22uF, Capacitor_SMD:C_0805_2012Metric, F.Cu at (291.5, 82.0)
- added C127: 22uF, Capacitor_SMD:C_0805_2012Metric, F.Cu at (281.4, 89.3)
- added C128: .1uF, Capacitor_SMD:C_0402_1005Metric, F.Cu at (314.9, 69.2)
- added C129: 4.7uF, Capacitor_SMD:C_0805_2012Metric, F.Cu at (325.6, 49.4)
- added C13: 22uF, Capacitor_SMD:C_1210_3225Metric, F.Cu at (294.0, 74.1)
- added C130: 4.7uF, Capacitor_SMD:C_0805_2012Metric, F.Cu at (281.4, 92.3)
- added C131: .1uF, Capacitor_SMD:C_0402_1005Metric, F.Cu at (296.4, 87.8)
- added C132: 2.2uF, Capacitor_SMD:C_1210_3225Metric, F.Cu at (314.9, 48.2)
- added C133: 22uF, Capacitor_SMD:C_0805_2012Metric, F.Cu at (309.0, 60.4)
- added C134: 22uF, Capacitor_SMD:C_0805_2012Metric, F.Cu at (304.3, 67.6)
- added C135: .1uF, Capacitor_SMD:C_0402_1005Metric, F.Cu at (302.1, 83.1)
- added C136: 22uF, Capacitor_SMD:C_0805_2012Metric, F.Cu at (287.1, 82.0)
- added C137: 22uF, Capacitor_SMD:C_0805_2012Metric, F.Cu at (287.1, 85.0)
- added C138: 1uF, Capacitor_SMD:C_0402_1005Metric, F.Cu at (293.5, 87.8)
- added C139: 1uF, Capacitor_SMD:C_0402_1005Metric, F.Cu at (331.6, 51.6)
- added C14: 22uF, Capacitor_SMD:C_1210_3225Metric, F.Cu at (287.7, 78.3)
- added C140: .1uF, Capacitor_SMD:C_0402_1005Metric, F.Cu at (312.0, 71.2)
- added C141: .1uF, Capacitor_SMD:C_0603_1608Metric, F.Cu at (329.8, 44.9)
- added C142: 22uF, Capacitor_SMD:C_1210_3225Metric, F.Cu at (319.5, 44.0)
- added C143: 22uF, Capacitor_SMD:C_1210_3225Metric, F.Cu at (313.8, 39.8)
- added C144: 100uF, Capacitor_SMD:C_1210_3225Metric, F.Cu at (303.6, 49.8)
- added C145: 2.2uF, Capacitor_SMD:C_1210_3225Metric, F.Cu at (303.9, 61.0)
- added C146: 22uF, Capacitor_SMD:C_1210_3225Metric, F.Cu at (288.3, 69.8)
- added C147: 47uF, Capacitor_SMD:C_1210_3225Metric, F.Cu at (298.3, 56.2)
- added C148: 22uF, Capacitor_SMD:C_1210_3225Metric, F.Cu at (282.0, 77.2)
- added C149: 47uF, Capacitor_SMD:C_1210_3225Metric, F.Cu at (320.5, 48.2)
- added C15: 22uF, Capacitor_SMD:C_1210_3225Metric, F.Cu at (325.1, 39.8)
- added C150: 5600pF, Capacitor_SMD:C_0603_1608Metric, F.Cu at (301.4, 76.3)
- added C151: 2.2uF, Capacitor_SMD:C_1210_3225Metric, F.Cu at (294.0, 69.8)
- added C152: 2.2uF, Capacitor_SMD:C_1210_3225Metric, F.Cu at (309.2, 52.5)
- added C153: 1uF, Capacitor_SMD:C_0603_1608Metric, F.Cu at (317.2, 62.7)
- added C154: 1uF, Capacitor_SMD:C_0603_1608Metric, F.Cu at (334.4, 41.9)
- added C155: 3.3nF, Capacitor_SMD:C_0402_1005Metric, F.Cu at (307.8, 75.4)
- added C156: 3.3nF, Capacitor_SMD:C_0402_1005Metric, F.Cu at (304.8, 77.6)
- added C157: 4.4pF, Capacitor_SMD:C_0402_1005Metric, F.Cu at (299.2, 85.1)
- added C158: 2pF, Capacitor_SMD:C_0402_1005Metric, F.Cu at (320.6, 62.4)
- added C159: 1000pF, Capacitor_SMD:C_0402_1005Metric, F.Cu at (299.2, 83.1)
- added C16: .1uF, Capacitor_SMD:C_0603_1608Metric, F.Cu at (295.8, 80.5)
- added C160: 244pF, Capacitor_SMD:C_0402_1005Metric, F.Cu at (309.6, 73.4)
- added C161: EEEFK1C101P, Capacitor_SMD:CP_Elec_6.3x5.9, F.Cu at (224.4, 62.0)
- added C162: EEEFK1C101P, Capacitor_SMD:CP_Elec_6.3x5.9, F.Cu at (213.7, 66.9)
- added C163: 10uF, Capacitor_SMD:C_0805_2012Metric, F.Cu at (404.7, 48.4)
- added C164: .1uF, Capacitor_SMD:C_0402_1005Metric, F.Cu at (404.2, 59.5)
- added C165: .1uF, Capacitor_SMD:C_0402_1005Metric, F.Cu at (417.1, 47.1)
- added C166: .1uF, Capacitor_SMD:C_0402_1005Metric, F.Cu at (423.8, 42.6)
- added C167: .1uF, Capacitor_SMD:C_0402_1005Metric, F.Cu at (414.5, 51.1)
- added C168: 10uF, Capacitor_SMD:C_0805_2012Metric, F.Cu at (408.6, 43.6)
- added C169: .1uF, Capacitor_SMD:C_0402_1005Metric, F.Cu at (404.2, 61.5)
- added C17: .1uF, Capacitor_SMD:C_0603_1608Metric, F.Cu at (313.2, 64.4)
- added C170: 1uF, Capacitor_SMD:C_0402_1005Metric, F.Cu at (422.9, 40.6)
- added C171: .1uF, Capacitor_SMD:C_0402_1005Metric, F.Cu at (425.8, 40.6)
- added C172: 1uF, Capacitor_SMD:C_0402_1005Metric, F.Cu at (407.1, 58.8)
- added C173: .1uF, Capacitor_SMD:C_0402_1005Metric, F.Cu at (417.4, 49.1)
- added C174: 1uF, Capacitor_SMD:C_0402_1005Metric, F.Cu at (407.1, 56.8)
- added C175: .1uF, Capacitor_SMD:C_0402_1005Metric, F.Cu at (411.6, 53.1)
- added C176: 1uF, Capacitor_SMD:C_0402_1005Metric, F.Cu at (401.3, 64.0)
- added C177: .1uF, Capacitor_SMD:C_0402_1005Metric, F.Cu at (401.3, 62.1)
- added C178: 6.8pF, Capacitor_SMD:C_0402_1005Metric, F.Cu at (425.8, 38.6)
- added C179: 6.8pF, Capacitor_SMD:C_0402_1005Metric, F.Cu at (398.4, 68.0)
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Connections:
- net +GVDD renamed /GVDD
- net 2V5_VPP renamed /2V5_VPP
- net ETH0_TD1_N renamed /POE_TD1_N
- net ETH0_TD1_P renamed /POE_TD1_P
- net ETH0_TD2_N renamed /POE_TD2_N
- net ETH0_TD2_P renamed /POE_TD2_P
- net ETH0_TD3_N renamed /POE_TD3_N
- net ETH0_TD3_P renamed /POE_TD3_P
- net ETH0_TD4_N renamed /POE_TD4_N
- net ETH0_TD4_P renamed /POE_TD4_P
- C21 pad 1: CPU_GND_SENSE -> <NO NET>
- C21 pad 2: 3V3 -> VCC
- C22 pad 1: 3V3 -> VCC
- C23 pad 2: CPU_GND_SENSE -> <NO NET>
- C24 pad 2: CPU_GND_SENSE -> <NO NET>
- C25 pad 1: CPU_GND_SENSE -> <NO NET>
- C33 pad 1: CPU_GND_SENSE -> <NO NET>
- C38 pad 2: CPU_GND_SENSE -> <NO NET>
- C47 pad 2: CPU_GND_SENSE -> <NO NET>
- C48 pad 1: CPU_GND_SENSE -> <NO NET>
- C55 pad 1: 12V0 -> /12V
- C55 pad 2: CPU_GND_SENSE -> <NO NET>
- C56 pad 1: 12V0 -> /12V
- C56 pad 2: CPU_GND_SENSE -> <NO NET>
- C57 pad 1: 12V0 -> /CPU_VDD_SENSE
- C57 pad 2: CPU_GND_SENSE -> Net-(C57-Pad2)
- C58 pad 1: 12V0 -> /12V
- C58 pad 2: CPU_GND_SENSE -> <NO NET>
- C60 pad 1: 12V0 -> /12V
- C60 pad 2: CPU_GND_SENSE -> <NO NET>
- C67 pad 1: CPU_GND_SENSE -> <NO NET>
- C70 pad 2: CPU_GND_SENSE -> <NO NET>
- C72 pad 2: CPU_GND_SENSE -> <NO NET>
- C73 pad 2: CPU_GND_SENSE -> <NO NET>
- C74 pad 2: CPU_GND_SENSE -> <NO NET>
- C75 pad 2: CPU_GND_SENSE -> <NO NET>
- C76 pad 2: CPU_GND_SENSE -> <NO NET>
- C77 pad 2: CPU_GND_SENSE -> <NO NET>
- C78 pad 2: CPU_GND_SENSE -> <NO NET>
- C79 pad 2: CPU_GND_SENSE -> <NO NET>
- C80 pad 2: CPU_GND_SENSE -> <NO NET>
- C81 pad 2: CPU_GND_SENSE -> <NO NET>
- C82 pad 2: CPU_GND_SENSE -> <NO NET>
- C83 pad 2: CPU_GND_SENSE -> <NO NET>
- C84 pad 2: CPU_GND_SENSE -> <NO NET>
- C85 pad 2: CPU_GND_SENSE -> <NO NET>
- C86 pad 2: CPU_GND_SENSE -> <NO NET>
- C87 pad 2: CPU_GND_SENSE -> <NO NET>
- C88 pad 2: CPU_GND_SENSE -> <NO NET>
- C89 pad 2: CPU_GND_SENSE -> <NO NET>
- C90 pad 2: CPU_GND_SENSE -> <NO NET>
- C91 pad 2: CPU_GND_SENSE -> <NO NET>
- C92 pad 2: CPU_GND_SENSE -> <NO NET>
- C93 pad 2: CPU_GND_SENSE -> <NO NET>
- C94 pad 2: CPU_GND_SENSE -> <NO NET>
- D17 pad 1: CPU_GND_SENSE -> <NO NET>
- D20 pad 2: CPU_GND_SENSE -> <NO NET>
- D24 pad 1: 12V0 -> /12V
- IC3 pad A2: CPU_GND_SENSE -> <NO NET>
- IC3 pad A7: Net-(IC3-PadA7) -> /CPU Memory/DDR4_DQS1_N
- IC3 pad A8: CPU_GND_SENSE -> <NO NET>
- IC3 pad B2: CPU_GND_SENSE -> <NO NET>
- IC3 pad B7: Net-(IC3-PadB7) -> /CPU Memory/DDR4_DQS1_P
- IC3 pad C9: CPU_GND_SENSE -> <NO NET>
- IC3 pad D2: CPU_GND_SENSE -> <NO NET>
- IC3 pad D8: CPU_GND_SENSE -> <NO NET>
- IC3 pad E1: CPU_GND_SENSE -> <NO NET>
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Routing:
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- removed copper zone on F.Cu, net Net-(C6-Pad2)

Commit message: Review / cleanup footprints, etc
Parts:
- removed C382, C384: 22uF, Capacitor_SMD:C_0805_2012Metric
- removed C383, C385: 10uF, Capacitor_SMD:C_0805_2012Metric
- removed the J1 at (270.6, 153.9)
- removed the J5 at (217.9, 43.0)
- removed the LED4 at (297.2, 123.3)
- removed LED9: LED8, LED_SMD:LED_0805_2012Metric
- removed the R147 at (313.2, 118.0)
- removed the R148 at (309.6, 120.8)
- removed the R150 at (297.4, 130.9)
- removed the R152 at (313.7, 108.1)
- removed the R153 at (301.1, 127.8)
- removed the R154 at (305.5, 125.2)
- removed the R155 at (322.4, 108.1)
- added C102: 4.7uF, Capacitor_SMD:C_1210_3225Metric, F.Cu at (206.2, 44.9)
- added C105: 10nF, Capacitor_SMD:C_0805_2012Metric, F.Cu at (233.0, 24.6)
- added C108: 1nF, Capacitor_SMD:C_0805_2012Metric, F.Cu at (184.9, 72.8)
- added FL3: NFE31PT222Z1E9L, LIB_NFE31PT222Z1E9L:NFE31, F.Cu at (158.6, 146.4)
- added FL4: ACM2012-900-2P-T002, LIB_ACM2012-900-2P-T002:ACM2012_1, F.Cu at (170.2, 149.5)
- added FL5: NFE31PT222Z1E9L, LIB_NFE31PT222Z1E9L:NFE31, F.Cu at (158.6, 141.5)
- added FL6: ACM2012-900-2P-T002, LIB_ACM2012-900-2P-T002:ACM2012_1, F.Cu at (165.7, 153.2)
- added H1: Mounting Hole, MountingHole:MountingHole_2.5mm_Pad_TopBottom, F.Cu at (3.50, 6.00)
- added H2: Mounting Hole, MountingHole:MountingHole_2.5mm_Pad_TopBottom, F.Cu at (146.5, 6.00)
- added H3: Mounting Hole, MountingHole:MountingHole_2.5mm_Pad_TopBottom, F.Cu at (3.50, 149.0)
- added H4: Mounting Hole, MountingHole:MountingHole_2.5mm_Pad_TopBottom, F.Cu at (146.5, 149.0)
- added IC1: MAX17632BATE+, LIB_MAX17632BATE+:QFN50P300X300X80-17N, F.Cu at (64.5, 81.4)
- added IC10: MAX1564ETE+, LIB_MAX1564ETE+:QFN65P400X400X80-17N, F.Cu at (171.5, 142.1)
- added IC2: PM8805TR, LIB_PM8805TR:PM8805TR, F.Cu at (10.0, 25.5)
- added J10: SS-52000-001, LIB_SS-52000-001:SS52000001, F.Cu at (77.4, 52.1)
- added J2: Barrel_Jack, Connector_BarrelJack:BarrelJack_Horizontal, F.Cu at (12.7, 148.3)
- added J3: Conn_ARM_JTAG_SWD_10, Connector_PinHeader_1.27mm:PinHeader_2x05_P1.27mm_Vertical_SMD, F.Cu at (144.3, 102.9)
- added J4: RJ45, Connector_RJ:RJ45_Amphenol_54602-x08_Horizontal, F.Cu at (116.1, 148.2)
- added JP1: SolderJumper_2_Open, Jumper:SolderJumper-2_P1.3mm_Open_TrianglePad1.0x1.5mm, F.Cu at (237.0, 63.0)
- added JP2: SolderJumper_2_Open, Jumper:SolderJumper-2_P1.3mm_Open_TrianglePad1.0x1.5mm, F.Cu at (232.7, 59.5)
- added JP3: SolderJumper_2_Open, Jumper:SolderJumper-2_P1.3mm_Open_TrianglePad1.0x1.5mm, F.Cu at (237.0, 59.5)
- added JP4: SolderJumper_2_Open, Jumper:SolderJumper-2_P1.3mm_Open_TrianglePad1.0x1.5mm, F.Cu at (232.7, 63.0)
- added L10: 10uH, LIB_7443631000:WE-HCF_201322, F.Cu at (14.0, 119.5)
- added L6: 1.5uH, Inductor_SMD:L_Coilcraft_XxL4040, F.Cu at (-21.0, 128.1)
- added L7: 10uH, Inductor_SMD:L_Coilcraft_XAL5030, F.Cu at (-20.4, 116.3)
- added L8: 5.6uH, Inductor_SMD:L_Wuerth_HCI-5040, F.Cu at (199.8, 39.1)
- added L8: 5.6uH, Inductor_SMD:L_Coilcraft_XAL5030, F.Cu at (-8.00, 124.5)
- added L9: 1mH, Inductor_SMD:L_Wuerth_HCI-5040, F.Cu at (199.6, 46.5)
- added LED10: LED8, LED_SMD:LED_0805_2012Metric, F.Cu at (220.9, 136.6)
- added LED4: STATUS LED, LED_SMD:LED_Cree-PLCC4_2x2mm_CW, F.Cu at (216.4, 137.6)
- added LED4: LED3, LED_SMD:LED_0805_2012Metric, F.Cu at (223.2, 127.0)
- added Q6: NTA4151P, Package_TO_SOT_SMD:SOT-416, F.Cu at (242.7, 91.4)
- added Q7: NTA4151P, Package_TO_SOT_SMD:SOT-416, F.Cu at (201.8, 117.0)
- added R147: 330, Resistor_SMD:R_0402_1005Metric, F.Cu at (232.1, 130.4)
- added R147: 220, Resistor_SMD:R_0402_1005Metric, F.Cu at (212.4, 132.9)
- added R148: 330, Resistor_SMD:R_0402_1005Metric, F.Cu at (218.6, 140.5)
- added R148: 220, Resistor_SMD:R_0402_1005Metric, F.Cu at (209.5, 132.9)
- added R150: 330, Resistor_SMD:R_0402_1005Metric, F.Cu at (226.9, 129.5)
- added R150: 220, Resistor_SMD:R_0402_1005Metric, F.Cu at (212.4, 130.9)
- added R152: 220, Resistor_SMD:R_0402_1005Metric, F.Cu at (209.5, 130.9)
- added R152: 330, Resistor_SMD:R_0402_1005Metric, F.Cu at (230.4, 135.4)
- added R153: 330, Resistor_SMD:R_0402_1005Metric, F.Cu at (243.0, 128.4)
- added R153: 220, Resistor_SMD:R_0402_1005Metric, F.Cu at (212.6, 150.5)
- added R154: 330, Resistor_SMD:R_0402_1005Metric, F.Cu at (294.8, 26.4)
- added R154: 330, Resistor_SMD:R_0402_1005Metric, F.Cu at (221.5, 141.1)
- added R155: 330, Resistor_SMD:R_0402_1005Metric, F.Cu at (281.0, 40.9)
- added R155: 330, Resistor_SMD:R_0402_1005Metric, F.Cu at (238.0, 130.4)
- added R231: 0, Resistor_SMD:R_0402_1005Metric, F.Cu at (265.5, 163.9)
- added R232: 0, Resistor_SMD:R_0402_1005Metric, F.Cu at (278.9, 147.5)
- added R233: 0, Resistor_SMD:R_0402_1005Metric, F.Cu at (273.1, 147.5)
- added R234: 2.7K, Resistor_SMD:R_0402_1005Metric, F.Cu at (276.0, 149.5)
- added R235: 2.7K, Resistor_SMD:R_0402_1005Metric, F.Cu at (270.2, 147.5)
- added R236: 10K, Resistor_SMD:R_0402_1005Metric, F.Cu at (276.0, 147.5)
- added R237: 10K, Resistor_SMD:R_0402_1005Metric, F.Cu at (265.5, 161.9)
- added R238: 0, Resistor_SMD:R_0402_1005Metric, F.Cu at (270.2, 151.5)
- added R239: 0, Resistor_SMD:R_0402_1005Metric, F.Cu at (273.1, 149.5)
- added R240: 0, Resistor_SMD:R_0402_1005Metric, F.Cu at (207.4, 118.3)
- added R241: 22, Resistor_SMD:R_0402_1005Metric, F.Cu at (239.0, 109.4)
- added R242: 22, Resistor_SMD:R_0402_1005Metric, F.Cu at (254.7, 90.8)
- added R243: 22, Resistor_SMD:R_0402_1005Metric, F.Cu at (248.3, 94.7)
- added R244: 22, Resistor_SMD:R_0402_1005Metric, F.Cu at (201.6, 121.7)
- added R245: 22, Resistor_SMD:R_0402_1005Metric, F.Cu at (224.9, 118.3)
- added R246: 220, Resistor_SMD:R_0402_1005Metric, F.Cu at (221.9, 118.3)
- added R247: 220, Resistor_SMD:R_0402_1005Metric, F.Cu at (245.4, 96.1)
- added R248: 1K, Resistor_SMD:R_0402_1005Metric, F.Cu at (248.3, 98.7)
- added R249: 22, Resistor_SMD:R_0402_1005Metric, F.Cu at (205.0, 116.3)
- added R250: 10K, Resistor_SMD:R_0402_1005Metric, F.Cu at (210.3, 120.3)
- added R251: 100K, Resistor_SMD:R_0402_1005Metric, F.Cu at (219.0, 118.3)
- added R252: 1K, Resistor_SMD:R_0402_1005Metric, F.Cu at (245.4, 100.1)
- added R253: 10K, Resistor_SMD:R_0402_1005Metric, F.Cu at (216.1, 118.3)
- added R254: 10K, Resistor_SMD:R_0402_1005Metric, F.Cu at (219.0, 120.3)
- added R255: 10K, Resistor_SMD:R_0402_1005Metric, F.Cu at (245.4, 94.1)
- added R256: DNP 10K, Resistor_SMD:R_0402_1005Metric, F.Cu at (201.6, 119.7)
- added R257: DNP 10K, Resistor_SMD:R_0402_1005Metric, F.Cu at (213.2, 118.3)
- added R258: DNP 10K, Resistor_SMD:R_0402_1005Metric, F.Cu at (219.6, 116.3)
- added R259: 10K, Resistor_SMD:R_0402_1005Metric, F.Cu at (251.2, 94.7)
- added R260: 6.04K, Resistor_SMD:R_0402_1005Metric, F.Cu at (216.1, 120.3)
- added R261: DNP 1K, Resistor_SMD:R_0402_1005Metric, F.Cu at (204.5, 119.7)
- added R262: DNP 1K, Resistor_SMD:R_0402_1005Metric, F.Cu at (248.3, 96.7)
- added R263: DNP 1K, Resistor_SMD:R_0402_1005Metric, F.Cu at (227.8, 118.3)
- added R264: 1K, Resistor_SMD:R_0402_1005Metric, F.Cu at (224.9, 120.3)
- added R265: 1K, Resistor_SMD:R_0402_1005Metric, F.Cu at (210.8, 116.3)
- added R266: 1K, Resistor_SMD:R_0402_1005Metric, F.Cu at (242.5, 100.1)
- added R267: DNP 1K, Resistor_SMD:R_0402_1005Metric, F.Cu at (248.3, 92.8)
- added R268: 0, Resistor_SMD:R_0402_1005Metric, F.Cu at (236.1, 111.3)
- added R269: 698, Resistor_SMD:R_0402_1005Metric, F.Cu at (242.5, 102.1)
- added R270: 200, Resistor_SMD:R_0402_1005Metric, F.Cu at (242.5, 96.1)
- added R271: 22, Resistor_SMD:R_0402_1005Metric, F.Cu at (207.4, 120.3)
- added R272: 22, Resistor_SMD:R_0402_1005Metric, F.Cu at (213.8, 116.3)
- added R273: 22, Resistor_SMD:R_0402_1005Metric, F.Cu at (245.4, 102.1)
- added R274: 22, Resistor_SMD:R_0402_1005Metric, F.Cu at (254.1, 92.8)
- added R275: 22, Resistor_SMD:R_0402_1005Metric, F.Cu at (242.5, 104.1)
- added R276: 220, Resistor_SMD:R_0402_1005Metric, F.Cu at (251.2, 92.8)
- added R277: 220, Resistor_SMD:R_0402_1005Metric, F.Cu at (207.9, 116.3)
- added R278: 1K, Resistor_SMD:R_0402_1005Metric, F.Cu at (251.2, 96.7)
- added R279: 22, Resistor_SMD:R_0402_1005Metric, F.Cu at (228.3, 116.3)
- added R280: 10K, Resistor_SMD:R_0402_1005Metric, F.Cu at (245.9, 90.8)
- added R281: 100K, Resistor_SMD:R_0402_1005Metric, F.Cu at (204.5, 121.7)
- added R282: 1K, Resistor_SMD:R_0402_1005Metric, F.Cu at (225.4, 116.3)
- added R283: 6.04K, Resistor_SMD:R_0402_1005Metric, F.Cu at (213.2, 120.3)
- added R284: 10K, Resistor_SMD:R_0402_1005Metric, F.Cu at (221.9, 120.3)
- added R285: 10K, Resistor_SMD:R_0402_1005Metric, F.Cu at (210.3, 118.3)
- added R286: 10K, Resistor_SMD:R_0402_1005Metric, F.Cu at (245.4, 98.1)
- added R287: DNP 10K, Resistor_SMD:R_0402_1005Metric, F.Cu at (242.5, 94.1)
- added R288: DNP 10K, Resistor_SMD:R_0402_1005Metric, F.Cu at (227.8, 120.3)
- added R289: 10K, Resistor_SMD:R_0402_1005Metric, F.Cu at (233.2, 111.3)
- added R290: DNP 10K, Resistor_SMD:R_0402_1005Metric, F.Cu at (251.7, 90.8)
- added R291: DNP 1K, Resistor_SMD:R_0402_1005Metric, F.Cu at (222.5, 116.3)
- added R292: DNP 1K, Resistor_SMD:R_0402_1005Metric, F.Cu at (233.2, 113.3)
- added R293: DNP 1K, Resistor_SMD:R_0402_1005Metric, F.Cu at (236.1, 109.4)
- added R294: 1K, Resistor_SMD:R_0402_1005Metric, F.Cu at (233.2, 109.4)
- added R295: 1K, Resistor_SMD:R_0402_1005Metric, F.Cu at (248.8, 90.8)
- added R296: DNP 1K, Resistor_SMD:R_0402_1005Metric, F.Cu at (216.7, 116.3)
- added R297: 1K, Resistor_SMD:R_0402_1005Metric, F.Cu at (242.5, 98.1)
- added R298: 0, Resistor_SMD:R_0402_1005Metric, F.Cu at (179.0, 143.6)
- added R299: 100K, Resistor_SMD:R_0402_1005Metric, F.Cu at (193.5, 140.0)
- added R300: 100K, Resistor_SMD:R_0402_1005Metric, F.Cu at (181.9, 143.6)
- added R301: 26.1K, Resistor_SMD:R_0402_1005Metric, F.Cu at (187.7, 140.0)
- added R302: 1K, Resistor_SMD:R_0402_1005Metric, F.Cu at (184.8, 140.0)
- added R303: 200, Resistor_SMD:R_0402_1005Metric, F.Cu at (190.6, 140.0)
- added R304: 0, Resistor_SMD:R_0402_1005Metric, F.Cu at (176.1, 145.0)
- added R305: 1K, Resistor_SMD:R_0402_1005Metric, F.Cu at (199.4, 140.0)
- added R306: 200, Resistor_SMD:R_0402_1005Metric, F.Cu at (187.7, 142.0)
- added R307: 0, Resistor_SMD:R_0402_1005Metric, F.Cu at (196.4, 140.0)
- added R308: 1K, Resistor_SMD:R_0402_1005Metric, F.Cu at (184.8, 142.0)
- added R309: 200, Resistor_SMD:R_0402_1005Metric, F.Cu at (176.1, 143.0)
- added SW1: RESET, Button_Switch_SMD:Panasonic_EVQPUJ_EVQPUA, F.Cu at (25.5, 158.0)
- added TP1: TestPoint, TestPoint:TestPoint_Pad_D1.0mm, F.Cu at (241.2, 70.7)
- added TP2: TestPoint, TestPoint:TestPoint_Pad_D1.0mm, F.Cu at (238.1, 70.7)
- added TP3: TestPoint, TestPoint:TestPoint_Pad_D1.0mm, F.Cu at (238.1, 73.7)
- added TP4: TestPoint, TestPoint:TestPoint_Pad_D1.0mm, F.Cu at (250.1, 59.2)
- added U13: 74LVC1G08, Silicon-Standard:SC70, F.Cu at (296.3, 104.9)
- added U14: 74LVC1G07, Silicon-Standard:SC70, F.Cu at (296.3, 108.3)
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- renumbered J4 to J1, J6 to J5, J2 to J6
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Connections:
- BT1 pad 2: <NO NET> -> GND
- C1 pad 2: <NO NET> -> GND
- C10 pad 1: Net-(C10-Pad1) -> /CPU_VDD
- C10 pad 2: <NO NET> -> Net-(C10-Pad2)
- C100 pad 1: <NO NET> -> Net-(C100-Pad1)
- C100 pad 2: Net-(C100-Pad2) -> GNDPWR
- C101 pad 1: <NO NET> -> Net-(C100-Pad1)
- C101 pad 2: Net-(C101-Pad2) -> GNDPWR
- C103 pad 1: <NO NET> -> GND
- C103 pad 2: /PWR_X1VDD -> GNDPWR
- C104 pad 1: <NO NET> -> GNDPWR
- C104 pad 2: /Power/EN_VDD -> Net-(C104-Pad2)
- C106 pad 1: <NO NET> -> Net-(C106-Pad1)
- C106 pad 2: /2V5_VPP -> GNDPWR
- C107 pad 1: <NO NET> -> Net-(C106-Pad1)
- C107 pad 2: /Power/BAKUP1 -> GNDPWR
- C109 pad 1: <NO NET> -> Net-(C109-Pad1)
- C109 pad 2: /Power/BAKUP2 -> Net-(C109-Pad2)
- C11 pad 1: Net-(C11-Pad1) -> GND
- C11 pad 2: <NO NET> -> /3V3
- C110 pad 1: <NO NET> -> Net-(C110-Pad1)
- C110 pad 2: VCC -> Net-(C110-Pad2)
- C111 pad 1: <NO NET> -> /12V
- C111 pad 2: VCC -> GND
- C112 pad 1: <NO NET> -> /12V
- C112 pad 2: VCC -> GND
- C113 pad 1: <NO NET> -> /12V
- C113 pad 2: VCC -> GND
- C114 pad 1: <NO NET> -> /12V
- C114 pad 2: VCC -> GND
- C115 pad 1: <NO NET> -> Net-(C110-Pad1)
- C115 pad 2: VCC -> Net-(C115-Pad2)
- C116 pad 1: <NO NET> -> /12V
- C116 pad 2: VCC -> GND
- C117 pad 1: <NO NET> -> /12V
- C117 pad 2: VCC -> GND
- C118 pad 1: <NO NET> -> GNDA
- C118 pad 2: /GVDD -> Net-(C118-Pad2)
- C119 pad 1: <NO NET> -> Net-(C106-Pad1)
- C119 pad 2: /GVDD -> GNDPWR
- C12 pad 1: <NO NET> -> Net-(C12-Pad1)
- C12 pad 2: Net-(C11-Pad1) -> GND
- C120 pad 1: <NO NET> -> Net-(C120-Pad1)
- C120 pad 2: /GVDD -> Net-(C120-Pad2)
- C121 pad 1: <NO NET> -> Net-(C121-Pad1)
- C121 pad 2: /GVDD -> Net-(C121-Pad2)
- C122 pad 1: <NO NET> -> GND
- C122 pad 2: /1V5 -> Net-(C122-Pad2)
- C123 pad 1: <NO NET> -> Net-(C123-Pad1)
- C123 pad 2: /1V5 -> Net-(C123-Pad2)
- C124 pad 1: <NO NET> -> GNDA
- C124 pad 2: /1V5 -> Net-(C124-Pad2)
- C125 pad 1: <NO NET> -> Net-(C125-Pad1)
- C125 pad 2: /1V5 -> Net-(C123-Pad2)
- C126 pad 1: <NO NET> -> GNDA
- C126 pad 2: /1V5 -> Net-(C126-Pad2)
- C127 pad 1: <NO NET> -> Net-(C127-Pad1)
- C127 pad 2: /1V5 -> GND
- C128 pad 1: <NO NET> -> GND
- C128 pad 2: VCC -> Net-(C128-Pad2)
- C129 pad 1: <NO NET> -> Net-(C128-Pad2)
- C129 pad 2: VCC -> GND
- C13 pad 1: /12V -> Net-(C13-Pad1)
- C13 pad 2: <NO NET> -> GND
- C130 pad 1: <NO NET> -> Net-(C128-Pad2)
- C130 pad 2: VCC -> GND
- C131 pad 1: <NO NET> -> Net-(C128-Pad2)
- C131 pad 2: VCC -> GND
- C132 pad 1: /12V -> Net-(C128-Pad2)
- C132 pad 2: <NO NET> -> GND
- C133 pad 1: <NO NET> -> GND
- C133 pad 2: /DDR_VTT -> Net-(C128-Pad2)
- C134 pad 1: <NO NET> -> /3V3
- C134 pad 2: /DDR_VTT -> GND
- C135 pad 1: /GVDD -> Net-(C135-Pad1)
- C135 pad 2: Net-(C135-Pad2) -> GND
- C136 pad 1: <NO NET> -> Net-(C135-Pad1)
- C136 pad 2: VCC -> GND
- C137 pad 1: <NO NET> -> Net-(C137-Pad1)
- C137 pad 2: VCC -> GND
- C138 pad 1: <NO NET> -> Net-(C137-Pad1)
- C138 pad 2: /DDR_VREF -> GND
- C139 pad 1: <NO NET> -> Net-(C139-Pad1)
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Routing:
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Other:
- board size 150 x 150 mm -> 150 x 160 mm
