File: AP2100/AP2100v4.kicad_pcb (KiCad board)
At the start: 4 copper layers, 160 x 90 mm, 151 parts, among them J1 Conn_01x03, J10 690-019-298-412, J11 USB_OTG, J12 10018783-11200TLF, J13 690-008-221-904, J14 Conn_02x05_Odd_Even, J15 Conn_01x22_Female, J16 Conn_01x22_Female, J17 Molex 470531000, J19 Barrel_Jack, J2 Conn_02x07_Odd_Even, J20 AMP171826-4, J22 690-019-298-412, J3 Conn_01x03, J4 Conn_01x22_Female, J5 Conn_01x22_Female, J6 THD-02-R, J7 Micro_SD_Card_Det, J8 THD-20-R, J9 THD-02-R, Q1 DMP3013SFV-7, U1 TPD4EUSB30, U11 EMC2301-1-ACZL-TR, U12 RT9742SNGV, U13 FSUSB42MUX, U14 74LVC1G07SE-7, U15 AP64501SP-13, U16 AP64501SP-13, U18 RT9742GGJ5, U2 TPD4EUSB30, U3 MagJack-A70-112-331N126, U4 TPD4EUSB30, U5 74LVC1G07SE-7, U6 USB2514B-I/M2, U7 AP22653W6, U8 PCF85063AT/AAZ, U9 74LVC1G07SE-7, Y1 24MHz, Y2 X32K768S301

Commit message: Finish PoE section Rename CM4IO library as AP2100
Parts:
- J10, J22: footprint CM4IO:EDAC 690-019-298-412 -> AP2100:EDAC 690-019-298-412
- J11: footprint CM4IO:USB_Micro-B_EDAC_UCON00686 -> AP2100:USB_Micro-B_EDAC_UCON00686
- J12: footprint CM4IO:PCIex1-36 -> AP2100:PCIex1-36
- J13: footprint CM4IO:MOLEX_USB_67298-4090 -> AP2100:MOLEX_USB_67298-4090
- J15, J16, J4, J5: footprint CM4IO:Hirose_FH12-22S-0.5SH_1x22-1MP_P0.50mm_Horizontal -> AP2100:Hirose_FH12-22S-0.5SH_1x22-1MP_P0.50mm_Horizontal
- J19: footprint CM4IO:BarrelJack_Horizontal -> AP2100:BarrelJack_Horizontal
- J7: footprint CM4IO:SDCARD_MOLEX_503398-1892 -> AP2100:SDCARD_MOLEX_503398-1892
- Module1: footprint CM4IO:Raspberry-Pi-4-Compute-Module -> AP2100:Raspberry-Pi-4-Compute-Module
- U15: footprint CM4IO:SOIC-8-1EP_3.9x4.9mm_P1.27mm_EP2.95x4.9mm_Mask2.71x3.4mm_ThermalVias -> AP2100:SOIC-8-1EP_3.9x4.9mm_P1.27mm_EP2.95x4.9mm_Mask2.71x3.4mm_ThermalVias
- U3: footprint CM4IO:TRJG0926HENL -> AP2100:TRJG0926HENL
Changed lines of the file:
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@@
     )
   )
-  (module "CM4IO:Hirose_FH12-22S-0.5SH_1x22-1MP_P0.50mm_Horizontal" (layer "F.Cu")
+  (module "AP2100:Hirose_FH12-22S-0.5SH_1x22-1MP_P0.50mm_Horizontal" (layer "F.Cu")
     (at 90.5 75 180)
     (descr "Molex FH12, FFC/FPC connector, FH12-22S-0.5SH, 22 Pins per row (https://www.hirose.com/product/en/products/FH12/FH12-24S-0.5SH(55)/), generated with kicad-footprint-generator")
@@
     (pad "MP" smd rect (at 7.15 1.4 180) (size 1.8 2.2) (layers "F.Cu" "F.Paste" "F.Mask"))
     (pad "MP" smd rect (at -7.15 1.4 180) (size 1.8 2.2) (layers "F.Cu" "F.Paste" "F.Mask"))
-    (model "./CM4IO.3dshapes/FH12-22S-0.5SHa.stp"
+    (model "./AP2100.3dshapes/FH12-22S-0.5SHa.stp"
       (offset (xyz 16.5 -10.6 2))
       (scale (xyz 1 1 1))
@@
     )
   )
-  (module "CM4IO:Hirose_FH12-22S-0.5SH_1x22-1MP_P0.50mm_Horizontal" (layer "F.Cu")
+  (module "AP2100:Hirose_FH12-22S-0.5SH_1x22-1MP_P0.50mm_Horizontal" (layer "F.Cu")
     (at 126.5 75 180)
     (descr "Molex FH12, FFC/FPC connector, FH12-22S-0.5SH, 22 Pins per row (https://www.hirose.com/product/en/products/FH12/FH12-24S-0.5SH(55)/), generated with kicad-footprint-generator")
@@
     (pad "MP" smd rect (at 7.15 1.4 180) (size 1.8 2.2) (layers "F.Cu" "F.Paste" "F.Mask"))
     (pad "MP" smd rect (at -7.15 1.4 180) (size 1.8 2.2) (layers "F.Cu" "F.Paste" "F.Mask"))
-    (model "./CM4IO.3dshapes/FH12-22S-0.5SHa.stp"
+    (model "./AP2100.3dshapes/FH12-22S-0.5SHa.stp"
       (offset (xyz 16.5 -10.6 2))
       (scale (xyz 1 1 1))
@@
     )
   )
-  (module "CM4IO:USB_Micro-B_EDAC_UCON00686" locked (layer "F.Cu")
+  (module "AP2100:USB_Micro-B_EDAC_UCON00686" locked (layer "F.Cu")
     (at 187 158.3)
     (descr "Micro USB Type B 10103594-0001LF, http://cdn.amphenol-icc.com/media/wysiwyg/files/drawing/10103594.pdf")
@@
     (pad "6" smd rect (at 2.9875 -1.7) (size 1.825 0.7) (layers "F.Cu" "F.Paste" "F.Mask")
       (net 1 "GND") (pinfunction "Shield"))
-    (model "./CM4IO.3dshapes/10103594.stp"
+    (model "./AP2100.3dshapes/10103594.stp"
       (offset (xyz 0 1.35 2.2))
       (scale (xyz 1 1 1))
@@
     )
   )
-  (module "CM4IO:BarrelJack_Horizontal" (layer "F.Cu")
+  (module "AP2100:BarrelJack_Horizontal" (layer "F.Cu")
     (at 232.25 147.7 90)
     (descr "DC Barrel Jack")
@@
     (pad "3" thru_hole roundrect (at -3 4.8 90) (size 5 2.8) (drill oval 3 0.8) (layers *.Cu *.Mask) (roundrect_rratio 0.25)
       (net 1 "GND"))
-    (model "./CM4IO.3dshapes/CUI_DEVICES_PJ-102AH.step"
+    (model "./AP2100.3dshapes/CUI_DEVICES_PJ-102AH.step"
       (offset (xyz -13.7 0 6.5))
       (scale (xyz 1 1 1))
@@
     )
   )
-  (module "CM4IO:TRJG0926HENL" locked (layer "F.Cu")
+  (module "AP2100:TRJG0926HENL" locked (layer "F.Cu")
     (at 153 150.5)
     (descr "https://p.globalsources.com/IMAGES/PDT/SPEC/690/K1160305690.pdf")
@@
     (pad "20" thru_hole circle (at 7.875 -3.05) (size 2.5 2.5) (drill 1.7) (layers *.Cu *.Mask)
       (net 1 "GND") (pinfunction "SHIELD"))
-    (model "./CM4IO.3dshapes/TRJG0926HENL .stp"
+    (model "./AP2100.3dshapes/TRJG0926HENL .stp"
       (offset (xyz 0 10.45 6.8))
       (scale (xyz 1 1 1))
@@
     )
   )
-  (module "CM4IO:EDAC 690-019-298-412" locked (layer "F.Cu")
+  (module "AP2100:EDAC 690-019-298-412" locked (layer "F.Cu")
     (at 127 150.45)
     (property "Field4" "Farnell")
@@
     (pad "SH4" thru_hole oval (at 7.25 5.96) (size 1.5 2.3) (drill oval 0.9 1.7) (layers *.Cu *.Mask)
       (net 1 "GND") (pinfunction "SH"))
-    (model "./CM4IO.3dshapes/471511051.stp"
+    (model "./AP2100.3dshapes/471511051.stp"
       (offset (xyz 0 -10.5 3.5))
       (scale (xyz 1 1 1))
@@
     )
   )
-  (module "CM4IO:EDAC 690-019-298-412" (layer "F.Cu")
+  (module "AP2100:EDAC 690-019-298-412" (layer "F.Cu")
     (at 102 150.45)
     (property "Field4" "Farnell")
@@
     (pad "SH4" thru_hole oval (at 7.25 5.96) (size 1.5 2.3) (drill oval 0.9 1.7) (layers *.Cu *.Mask)
       (net 1 "GND") (pinfunction "SH"))
-    (model "./CM4IO.3dshapes/471511051.stp"
+    (model "./AP2100.3dshapes/471511051.stp"
       (offset (xyz 0 -10.5 3.5))
       (scale (xyz 1 1 1))
@@
     )
   )
-  (module "CM4IO:MOLEX_USB_67298-4090" (layer "F.Cu")
+  (module "AP2100:MOLEX_USB_67298-4090" (layer "F.Cu")
     (at 172 150.7)
     (property "Field4" "Farnell")
@@
     (pad "MT4" thru_hole circle (at 6.57 -5.68) (size 3.45 3.45) (drill 2.3) (layers *.Cu *.Mask)
       (net 1 "GND") (pinfunction "MT4"))
-    (model "./CM4IO.3dshapes/672984090.stp"
+    (model "./AP2100.3dshapes/672984090.stp"
       (offset (xyz 0 -9.800000000000001 8))
       (scale (xyz 1 1 1))
@@
     (pad "4" thru_hole circle (at 3.75 -4.55 180) (size 1.408 1.408) (drill 0.9) (layers *.Cu *.Mask)
       (net 227 "/+5v") (pinfunction "Pin_4"))
-    (model "./CM4IO.3dshapes/c-171826-4-y3-3d.stp"
+    (model "./AP2100.3dshapes/c-171826-4-y3-3d.stp"
       (offset (xyz 0 0.75 0))
       (scale (xyz 1 1 1))
@@
       (rotate (xyz 0 0 0))
     )
-    (model "./CM4IO.3dshapes/ECS-.327-12.5-12QS-TR.stp"
+    (model "./AP2100.3dshapes/ECS-.327-12.5-12QS-TR.stp"
       (offset (xyz 0 0 0))
       (scale (xyz 1 1 1))
@@
     )
   )
-  (module "CM4IO:SDCARD_MOLEX_503398-1892" locked (layer "F.Cu")
+  (module "AP2100:SDCARD_MOLEX_503398-1892" locked (layer "F.Cu")
     (at 201.08 152.45 180)
     (property "Field4" "Farnell")
@@
     (pad "11" smd rect (at -6.48 5.64 180) (size 0.7 3.33) (layers "F.Cu" "F.Paste" "F.Mask")
       (net 1 "GND") (pinfunction "SHIELD"))
-    (model "./CM4IO.3dshapes/5033981892.stp"
+    (model "./AP2100.3dshapes/5033981892.stp"
       (offset (xyz -135.9 -16.4 154.4))
       (scale (xyz 1 1 1))
@@
     )
   )
-  (module "CM4IO:Hirose_FH12-22S-0.5SH_1x22-1MP_P0.50mm_Horizontal" (layer "F.Cu")
+  (module "AP2100:Hirose_FH12-22S-0.5SH_1x22-1MP_P0.50mm_Horizontal" (layer "F.Cu")
     (at 108.5 75 180)
     (descr "Molex FH12, FFC/FPC connector, FH12-22S-0.5SH, 22 Pins per row (https://www.hirose.com/product/en/products/FH12/FH12-24S-0.5SH(55)/), generated with kicad-footprint-generator")
@@
     (pad "MP" smd rect (at 7.15 1.4 180) (size 1.8 2.2) (layers "F.Cu" "F.Paste" "F.Mask"))
     (pad "MP" smd rect (at -7.15 1.4 180) (size 1.8 2.2) (layers "F.Cu" "F.Paste" "F.Mask"))
-    (model "./CM4IO.3dshapes/FH12-22S-0.5SHa.stp"
+    (model "./AP2100.3dshapes/FH12-22S-0.5SHa.stp"
       (offset (xyz 16.5 -10.6 2))
       (scale (xyz 1 1 1))
@@
     )
   )
-  (module "CM4IO:Hirose_FH12-22S-0.5SH_1x22-1MP_P0.50mm_Horizontal" (layer "F.Cu")
+  (module "AP2100:Hirose_FH12-22S-0.5SH_1x22-1MP_P0.50mm_Horizontal" (layer "F.Cu")
     (at 84 93.5 -90)
     (descr "Molex FH12, FFC/FPC connector, FH12-22S-0.5SH, 22 Pins per row (https://www.hirose.com/product/en/products/FH12/FH12-24S-0.5SH(55)/), generated with kicad-footprint-generator")
@@
     (pad "MP" smd rect (at 7.15 1.4 270) (size 1.8 2.2) (layers "F.Cu" "F.Paste" "F.Mask"))
     (pad "MP" smd rect (at -7.15 1.4 270) (size 1.8 2.2) (layers "F.Cu" "F.Paste" "F.Mask"))
-    (model "./CM4IO.3dshapes/FH12-22S-0.5SHa.stp"
+    (model "./AP2100.3dshapes/FH12-22S-0.5SHa.stp"
       (offset (xyz 16.5 -10.6 2))
       (scale (xyz 1 1 1))
@@
       (rotate (xyz 0 0 90))
     )
-    (model "./CM4IO.3dshapes/DMP3018SFVQ-13.stp"
+    (model "./AP2100.3dshapes/DMP3018SFVQ-13.stp"
       (offset (xyz 0 0 0))
       (scale (xyz 1 1 1))
@@
     )
   )
-  (module "CM4IO:SOIC-8-1EP_3.9x4.9mm_P1.27mm_EP2.95x4.9mm_Mask2.71x3.4mm_ThermalVias" (layer "F.Cu")
+  (module "AP2100:SOIC-8-1EP_3.9x4.9mm_P1.27mm_EP2.95x4.9mm_Mask2.71x3.4mm_ThermalVias" (layer "F.Cu")
     (at 228.35 126.0625 90)
     (descr "SOIC, 8 Pin (http://www.ti.com/lit/ds/symlink/lm5017.pdf#page=31), generated with kicad-footprint-generator ipc_gullwing_generator.py")
@@
     )
   )
-  (module "CM4IO:PCIex1-36" locked (layer "F.Cu")
+  (module "AP2100:PCIex1-36" locked (layer "F.Cu")
     (at 207.75 114.15 90)
     (property "Field4" "Mouser")
@@
     (pad "B18" thru_hole circle (at 19 4.5) (size 1.3 1.3) (drill 0.7) (layers *.Cu *.Mask)
       (net 1 "GND") (pinfunction "GND"))
-    (model "./CM4IO.3dshapes/PCIe-x1-36.step"
+    (model "./AP2100.3dshapes/PCIe-x1-36.step"
       (offset (xyz 11.5 -1.25 0))
       (scale (xyz 1 1 1))
@@
     )
   )
-  (module "CM4IO:Raspberry-Pi-4-Compute-Module" locked (layer "F.Cu")
+  (module "AP2100:Raspberry-Pi-4-Compute-Module" locked (layer "F.Cu")
     (at 195.5 73.5 180)
     (descr "Raspberry Pi 4 Compute Module")
@@
     (pad "200" smd rect (at 35 -11.7 90) (size 0.2 0.7) (layers "F.Cu" "F.Paste" "F.Mask")
       (net 117 "/CM4_HighSpeed/HDMI0_SCL") (pinfunction "HDMI0_SCL"))
-    (model "./CM4IO.3dshapes/DF40C-100DS.stp"
+    (model "./AP2100.3dshapes/DF40C-100DS.stp"
       (offset (xyz -0.46 15.38 0))
       (scale (xyz 1 1 1))
       (rotate (xyz -90 0 0))
     )
-    (model "./CM4IO.3dshapes/DF40C-100DS.stp"
+    (model "./AP2100.3dshapes/DF40C-100DS.stp"
       (offset (xyz 33.46 15.38 0))
       (scale (xyz 1 1 1))
