File: AP2100/poe.kicad_sch (KiCad schematic)
At the start: 136 parts, among them IC2 PM8805TR, IC3 PM8804TR, J1 0826-1X1T-GH-F, J2 Barrel_Jack, Q1 BSC190N15NS3GATMA1, Q2 PBSS4240T, Q3 PBSS4240T, Q4 FDMC86259P, Q5 FOD817AS, T1 RN102-2-02-1M1, T2 RN102-2-02-1M1, U4 STL90N6F7, U5 STL90N6F7, U6 TS2431-AILT

Commit message: Rename AP2100 as AP2100.ls1043 shelving the Layerscape design and starting a new Raspberry Pi 4 compute module based board
Parts:
- removed C100, C101, C102, C95, C99: 4.7uF, Capacitor_SMD:C_1210_3225Metric, symbol Device:C_Small
- removed C103, C93, C94: 2.2nF, Capacitor_SMD:C_1812_4532Metric, symbol Device:C_Small
- removed C104: 1.5nF, Capacitor_SMD:C_0603_1608Metric, symbol Device:C_Small
- removed C105: 10nF, Capacitor_SMD:C_0805_2012Metric, symbol Device:C_Small
- removed C106, C127: 2.2uF 25V, Capacitor_SMD:C_0805_2012Metric, symbol Device:C_Small
- removed C107, C117, C119, C121, C122, C126: 100nF, Capacitor_SMD:C_0603_1608Metric, symbol Device:C_Small
- removed C108, C109, C112, C79, C83, C97, C98: 1nF, Capacitor_SMD:C_0805_2012Metric, symbol Device:C_Small
- removed C110, C111: 100pF, Capacitor_SMD:C_0805_2012Metric, symbol Device:C_Small
- removed C113, C114, C116: 47uF, Capacitor_SMD:C_1210_3225Metric, symbol Device:C_Small
- removed C115: 100uF, Capacitor_SMD:CP_Elec_6.3x5.9, symbol Device:CP1_Small
- removed C118, C87, C89: 10nF, Capacitor_SMD:C_0603_1608Metric, symbol Device:C_Small
- removed C120: 47nF, Capacitor_SMD:C_1206_3216Metric, symbol Device:C_Small
- removed C123: 220pF, Capacitor_SMD:C_0603_1608Metric, symbol Device:C_Small
- removed C124: 100pF, Capacitor_SMD:C_0603_1608Metric, symbol Device:C_Small
- removed C125: 22nF, Capacitor_SMD:C_0603_1608Metric, symbol Device:C_Small
- removed C78, C80, C84, C85: 33nF, Capacitor_SMD:C_0805_2012Metric, symbol Device:C_Small
- removed C81, C82, C86, C88: .1uF, Capacitor_SMD:C_0402_1005Metric, symbol Device:C_Small
- removed C90: 1nF, Capacitor_SMD:C_0603_1608Metric, symbol Device:C_Small
- removed C91, C92: 33uF, LIB_EEEFK2A330P:CAPAE1030X1050N, symbol AP2100-rescue:EEEFK2A330P-EEEFK2A330P
- removed C96: 100nF, Capacitor_SMD:C_0805_2012Metric, symbol Device:C_Small
- removed D1, D2, D3, D4, D5, D6: SM15T68CA, Diode_SMD:D_SMC, symbol Device:D_TVS_ALT
- removed D10: SMAJ58A, Diode_SMD:D_SMA, symbol Device:D_TVS_ALT
- removed D11, D12, D13, D14, D15: BAS16J, Diode_SMD:D_SOD-323, symbol Device:D_ALT
- removed D16: BZX84C10LT1G, Package_TO_SOT_SMD:SOT-23, symbol Diode:BAS19
- removed D17: BZX84C10, Package_TO_SOT_SMD:SOT-23, symbol Diode:BAS19
- removed D18, D19, D20: BAS70, Diode_SMD:D_SOD-323, symbol Device:D_ALT
- removed D7: STPS4S200S, LIB_STPS4S200S:DIOM8059X265N, symbol AP2100-rescue:STPS4S200S-STPS4S200S
- removed D8: BAV70, Package_TO_SOT_SMD:SOT-23, symbol Diode:BAV70
- removed D9: SMAJ58A, Diode_SMD:D_SMA, symbol Device:D_Schottky_ALT
- removed FB1, FB2, FB3, FB4: 220 OHM, Inductor_SMD:L_0805_2012Metric, symbol Device:L
- removed IC2: PM8805TR, LIB_PM8805TR:PM8805TR, symbol AP2100-rescue:PM8805TR-PM8805TR
- removed IC3: PM8804TR, LIB_PM8804TR:QFN50P340X340X90-17N, symbol AP2100-rescue:PM8804TR-PM8804TR
- removed J1: 0826-1X1T-GH-F, 0826-1X1T-GH-F:BEL_0826-1X1T-GH-F, symbol AP2100-rescue:0826-1X1T-GH-F-0826-1X1T-GH-F
- removed J2: Barrel_Jack, Connector_BarrelJack:BarrelJack_Horizontal, symbol Connector:Barrel_Jack
- removed L10: 10uH, LIB_7443631000:WE-HCF_201322, symbol 7443631000:7443631000
- removed L8: 5.6uH, Inductor_SMD:L_Coilcraft_XAL5030, symbol Device:L
- removed L9: 1mH, Inductor_SMD:L_Coilcraft_LPS4018, symbol Device:L
- removed LED1: T2, LED_SMD:LED_0603_1608Metric, symbol Device:LED_ALT
- removed LED2: T1, LED_SMD:LED_0603_1608Metric, symbol Device:LED_ALT
- removed LED3: T0, LED_SMD:LED_0603_1608Metric, symbol Device:LED_ALT
- removed LED4: AUX, LED_SMD:LED_0603_1608Metric, symbol Device:LED_ALT
- removed LED5: +12V, LED_SMD:LED_0603_1608Metric, symbol Device:LED_ALT
- removed Q1: BSC190N15NS3GATMA1, Scott:TRANS_BSC100N06LS3GATMA1, symbol BSC190N15NS3GATMA1:BSC190N15NS3GATMA1
- removed Q2, Q3: PBSS4240T, Package_TO_SOT_SMD:SOT-23, symbol Device:Q_NPN_BEC
- removed Q4: FDMC86259P, LIB_FDMC86259P:FDMC86160, symbol FDMC86259P:FDMC86259P
- removed Q5: FOD817AS, LIB_FOD817AS:SOP254P1016X385-4N, symbol FOD817AS:FOD817AS
- removed R17: 36.5, Resistor_SMD:R_0805_2012Metric, symbol Device:R_Small_US
- removed R18: 150, Resistor_SMD:R_0805_2012Metric, symbol Device:R_Small_US
- removed R19: 26.1K, Resistor_SMD:R_0603_1608Metric, symbol Device:R_Small_US
- removed R20, R22, R23: 3.9K, Resistor_SMD:R_0603_1608Metric, symbol Device:R_Small_US
- removed R21: 0, Resistor_SMD:R_2010_5025Metric, symbol Device:R_Small_US
- removed R24, R36: 10, Resistor_SMD:R_0805_2012Metric, symbol Device:R_Small_US
- removed R25: 100K, Resistor_SMD:R_0603_1608Metric, symbol Device:R_Small_US
- removed R26, R53: 4.7K, Resistor_SMD:R_0603_1608Metric, symbol Device:R_Small_US
- removed R27, R28, R33, R39, R40, R44: 10K, Resistor_SMD:R_0603_1608Metric, symbol Device:R_Small_US
- removed R29, R31, R311: 1K, Resistor_SMD:R_0603_1608Metric, symbol Device:R_Small_US
- removed R30, R32: 22, Resistor_SMD:R_0603_1608Metric, symbol Device:R_Small_US
- removed R34: 18, Resistor_SMD:R_0805_2012Metric, symbol Device:R_Small_US
- removed R35: 88.7K, Resistor_SMD:R_0603_1608Metric, symbol Device:R_Small_US
- removed R37: 330K, Resistor_SMD:R_0603_1608Metric, symbol Device:R_Small_US
- removed R38: 10K, Resistor_SMD:R_0805_2012Metric, symbol Device:R_Small_US
- removed R41: 0R05, Resistor_SMD:R_1210_3225Metric, symbol Device:R_Small_US
- removed R42: R100, Resistor_SMD:R_1210_3225Metric, symbol Device:R_Small_US
- removed R43: 0, Resistor_SMD:R_1206_3216Metric, symbol Device:R_Small_US
- removed R45, R46: 0, Resistor_SMD:R_0603_1608Metric, symbol Device:R_Small_US
- removed R47: 20K, Resistor_SMD:R_0603_1608Metric, symbol Device:R_Small_US
- removed R48, R50: 2K, Resistor_SMD:R_0603_1608Metric, symbol Device:R_Small_US
- removed R49: 47K, Resistor_SMD:R_0603_1608Metric, symbol Device:R_Small_US
- removed R51: 390, Resistor_SMD:R_0603_1608Metric, symbol Device:R_Small_US
- removed R52: 130K, Resistor_SMD:R_0603_1608Metric, symbol Device:R_Small_US
- removed R54: 5.23K, Resistor_SMD:R_0603_1608Metric, symbol Device:R_Small_US
- removed T1, T2: RN102-2-02-1M1, Inductor_THT:Choke_Schaffner_RN102-04-14.0x14.0mm, symbol Filter:Choke_Schaffner_RN102-2-02-1M1
- removed TR1: POE120PL-12L, Scott:Transformer_Coilcraft_POE120PL, symbol Scott:Transformer_POE120PL-12L
- removed U4, U5: STL90N6F7, Scott:TRANS_STL60P4LLF6, symbol STL90N6F7:STL90N6F7
- removed U6: TS2431-AILT, digikey-footprints:SOT-23-3, symbol dk_PMIC-Voltage-Reference:TL431AIDBZR
- added C? (x7): 1nF, Capacitor_SMD:C_0805_2012Metric, symbol Device:C_Small
- added C? (x3): 2.2nF, Capacitor_SMD:C_1812_4532Metric, symbol Device:C_Small
- added C? (x4): .1uF, Capacitor_SMD:C_0402_1005Metric, symbol Device:C_Small
- added C?: 100pF, Capacitor_SMD:C_0603_1608Metric, symbol Device:C_Small
- added C? (x2): 100u 6.3v, Capacitor_SMD:C_1206_3216Metric, symbol Device:C
- added C?: 100uF, Capacitor_SMD:CP_Elec_6.3x5.9, symbol Device:CP1_Small
- added C? (x2): 100pF, Capacitor_SMD:C_0805_2012Metric, symbol Device:C_Small
- added C?: 100n 16v, Capacitor_SMD:C_0402_1005Metric, symbol Device:C
- added C? (x5): 4.7uF, Capacitor_SMD:C_1210_3225Metric, symbol Device:C_Small
- added C?: 330p 50v, Capacitor_SMD:C_0603_1608Metric, symbol Device:C
- added C? (x3): 47uF, Capacitor_SMD:C_1210_3225Metric, symbol Device:C_Small
- added C? (x3): 10nF, Capacitor_SMD:C_0603_1608Metric, symbol Device:C_Small
- added C? (x4): 33nF, Capacitor_SMD:C_0805_2012Metric, symbol Device:C_Small
- added C? (x2): 1000p 100v, Capacitor_SMD:C_0805_2012Metric, symbol Device:C
- added C? (x3): .1u 100v, Capacitor_SMD:C_0603_1608Metric, symbol Device:C
- added C?: 10n 100v, Capacitor_SMD:C_0603_1608Metric, symbol Device:C
- added C? (x2): 1u 100v, Capacitor_SMD:C_1206_3216Metric, symbol Device:C
- added C? (x6): 100nF, Capacitor_SMD:C_0603_1608Metric, symbol Device:C_Small
- added C?: 47nF, Capacitor_SMD:C_1206_3216Metric, symbol Device:C_Small
- added C?: .47u 16V, Capacitor_SMD:C_0603_1608Metric, symbol Device:C
- added C?: 10u 10v, Capacitor_SMD:C_0805_2012Metric, symbol Device:C
- added C?: 100n 50v, Capacitor_SMD:C_0603_1608Metric, symbol Device:C
- added C?: 10u 35v, Capacitor_SMD:C_0805_2012Metric, symbol Device:C
- added C?: 22nF, Capacitor_SMD:C_0603_1608Metric, symbol Device:C_Small
- added C?: 1u 35v, Capacitor_SMD:C_0402_1005Metric, symbol Device:C
- added C?: 10nF, Capacitor_SMD:C_0805_2012Metric, symbol Device:C_Small
- added C?: 13p 50v, Capacitor_SMD:C_0402_1005Metric, symbol Device:C
- added C? (x2): 2.2uF 25V, Capacitor_SMD:C_0805_2012Metric, symbol Device:C_Small
- added C?: 100n 100v, Capacitor_SMD:C_0402_1005Metric, symbol Device:C
- added C?: 1nF, Capacitor_SMD:C_0603_1608Metric, symbol Device:C_Small
- added C?: 220pF, Capacitor_SMD:C_0603_1608Metric, symbol Device:C_Small
- added C? (x2): 33uF, LIB_EEEFK2A330P:CAPAE1030X1050N, symbol AP2100-rescue:EEEFK2A330P-EEEFK2A330P
- added C?: 100n, Capacitor_SMD:C_0402_1005Metric, symbol Device:C
- added C?: 100nF, Capacitor_SMD:C_0805_2012Metric, symbol Device:C_Small
- added C?: 47u 63v, Capacitor_SMD:CP_Elec_8x10.5, symbol AP2100-rescue:EEEFK2A330P-EEEFK2A330P
- added C?: 1u 35v, Capacitor_SMD:C_0603_1608Metric, symbol Device:C
- added C?: 1.5nF, Capacitor_SMD:C_0603_1608Metric, symbol Device:C_Small
- added C?: 1.8n 50v, Capacitor_SMD:C_0603_1608Metric, symbol Device:C
- added D? (x9): B2100, Diode_SMD:D_SMA, symbol Device:D_Schottky_ALT
- added D?: BZX84C10LT1G, Package_TO_SOT_SMD:SOT-23, symbol Diode:BAS19
- added D? (x5): BAS16J, Diode_SMD:D_SOD-323, symbol Device:D_ALT
- added D?: STPS4S200S, LIB_STPS4S200S:DIOM8059X265N, symbol AP2100-rescue:STPS4S200S-STPS4S200S
- added D? (x6): SM15T68CA, Diode_SMD:D_SMC, symbol Device:D_TVS_ALT
- added D?: BZX84C10, Package_TO_SOT_SMD:SOT-23, symbol Diode:BAS19
- added D? (x3): BAS70, Diode_SMD:D_SOD-323, symbol Device:D_ALT
- added D?: BAV70, Package_TO_SOT_SMD:SOT-23, symbol Diode:BAV70
- added D?: MMBZ5242BLT3G, Diode_SMD:D_SOT-23_ANK, symbol Diode:BZX84Cxx
- added D? (x2): SMAJ58A, Diode_SMD:D_SMA, symbol Device:D_Schottky_ALT
- added D?: SMAJ58A, Diode_SMD:D_SMA, symbol Device:D_TVS_ALT
- added FB? (x4): 500 OHM, Inductor_SMD:L_1206_3216Metric, symbol Device:L
- added FB? (x4): 220 OHM, Inductor_SMD:L_0805_2012Metric, symbol Device:L
- added IC?: PM8805TR, LIB_PM8805TR:PM8805TR, symbol AP2100-rescue:PM8805TR-PM8805TR
- added IC?: PM8804TR, LIB_PM8804TR:QFN50P340X340X90-17N, symbol AP2100-rescue:PM8804TR-PM8804TR
- added IC?: TPS23751PWPR, SOP65P640X120-17N, symbol CM4IO:TPS23751PWPR
- added J? (x2): Barrel_Jack, Connector_BarrelJack:BarrelJack_Horizontal, symbol Connector:Barrel_Jack
- added J?: Barrel_Jack, Connector_BarrelJack:BarrelJack_Horizontal, symbol CM4IO:Barrel_Jack
- added J?: 0826-1X1T-GH-F, 0826-1X1T-GH-F:BEL_0826-1X1T-GH-F, symbol AP2100-rescue:0826-1X1T-GH-F-0826-1X1T-GH-F
- added L?: 10uH, LIB_7443631000:WE-HCF_201322, symbol 7443631000:7443631000
- added L?: 5.6uH, Inductor_SMD:L_Coilcraft_XAL5030, symbol Device:L
- added L?: LPS4018-332MRB, Inductor_SMD:L_Coilcraft_LPS4018, symbol pspice:INDUCTOR
- added L?: 1mH, Inductor_SMD:L_Coilcraft_LPS4018, symbol Device:L
- added L?: XAL4020-601MEB, Inductor_SMD:L_Coilcraft_XxL4020, symbol pspice:INDUCTOR
- added LED?: AUX, LED_SMD:LED_0603_1608Metric, symbol Device:LED_ALT
- added LED?: T0, LED_SMD:LED_0603_1608Metric, symbol Device:LED_ALT
- added LED?: T1, LED_SMD:LED_0603_1608Metric, symbol Device:LED_ALT
- added LED?: T2, LED_SMD:LED_0603_1608Metric, symbol Device:LED_ALT
- added LED?: +12V, LED_SMD:LED_0603_1608Metric, symbol Device:LED_ALT
- added Q?: FDMC86259P, LIB_FDMC86259P:FDMC86160, symbol FDMC86259P:FDMC86259P
- added Q?: DMP3013SFV-7, Package_SON:Diodes_PowerDI3333-8, symbol Transistor_FET:DMP3013SFV
- added Q?: BSC190N15NS3GATMA1, Scott:TRANS_BSC100N06LS3GATMA1, symbol BSC190N15NS3GATMA1:BSC190N15NS3GATMA1
- added Q? (x2): PBSS4240T, Package_TO_SOT_SMD:SOT-23, symbol Device:Q_NPN_BEC
- added Q?: FOD817AS, LIB_FOD817AS:SOP254P1016X385-4N, symbol FOD817AS:FOD817AS
- added R? (x2): 2K, Resistor_SMD:R_0603_1608Metric, symbol Device:R_Small_US
- added R? (x3): 3.9K, Resistor_SMD:R_0603_1608Metric, symbol Device:R_Small_US
- added R? (x6): 10K, Resistor_SMD:R_0603_1608Metric, symbol Device:R_Small_US
- added R? (x2): 10, Resistor_SMD:R_0805_2012Metric, symbol Device:R_Small_US
- added R?: 47K, Resistor_SMD:R_0603_1608Metric, symbol Device:R_Small_US
- added R?: 36.5, Resistor_SMD:R_0805_2012Metric, symbol Device:R_Small_US
- added R? (x2): 22, Resistor_SMD:R_0603_1608Metric, symbol Device:R_Small_US
- added R?: 88.7K, Resistor_SMD:R_0603_1608Metric, symbol Device:R_Small_US
- added R?: 34K 1%, Resistor_SMD:R_0402_1005Metric, symbol Device:R
- added R? (x2): 4.7K, Resistor_SMD:R_0603_1608Metric, symbol Device:R_Small_US
- added R?: 390, Resistor_SMD:R_0603_1608Metric, symbol Device:R_Small_US
- added R?: 100K, Resistor_SMD:R_0603_1608Metric, symbol Device:R_Small_US
- added R? (x2): 100K 1%, Resistor_SMD:R_0402_1005Metric, symbol Device:R
- added R?: 20K, Resistor_SMD:R_0603_1608Metric, symbol Device:R_Small_US
- added R? (x3): 1K, Resistor_SMD:R_0603_1608Metric, symbol Device:R_Small_US
- added R?: 26.1K, Resistor_SMD:R_0603_1608Metric, symbol Device:R_Small_US
- added R?: 750K 1%, Resistor_SMD:R_0402_1005Metric, symbol Device:R
- added R?: 10K 1%, Resistor_SMD:R_0402_1005Metric, symbol Device:R
- added R? (x2): 0, Resistor_SMD:R_0603_1608Metric, symbol Device:R_Small_US
- added R?: 12K 1%, Resistor_SMD:R_0402_1005Metric, symbol Device:R
- added R?: 18, Resistor_SMD:R_0805_2012Metric, symbol Device:R_Small_US
- added R?: 330K, Resistor_SMD:R_0603_1608Metric, symbol Device:R_Small_US
- added R?: 150, Resistor_SMD:R_0805_2012Metric, symbol Device:R_Small_US
- added R?: 63.4 1%, Resistor_SMD:R_0402_1005Metric, symbol Device:R
- added R?: 0, Resistor_SMD:R_2010_5025Metric, symbol Device:R_Small_US
- added R?: R100, Resistor_SMD:R_1210_3225Metric, symbol Device:R_Small_US
- added R?: 27.1K .1%, Resistor_SMD:R_0805_2012Metric, symbol Device:R
- added R?: 8.87K 1%, Resistor_SMD:R_0402_1005Metric, symbol Device:R
- added R?: 5.23K, Resistor_SMD:R_0603_1608Metric, symbol Device:R_Small_US
- added R?: 10K, Resistor_SMD:R_0805_2012Metric, symbol Device:R_Small_US
- added R?: 48.7K 1%, Resistor_SMD:R_0402_1005Metric, symbol Device:R
- added R?: 24.9K 1%, Resistor_SMD:R_0603_1608Metric, symbol Device:R
- added R?: 130K, Resistor_SMD:R_0603_1608Metric, symbol Device:R_Small_US
- added R?: 0R05, Resistor_SMD:R_1210_3225Metric, symbol Device:R_Small_US
- added R?: 6.04K 1%, Resistor_SMD:R_0402_1005Metric, symbol Device:R
- added R?: 0, Resistor_SMD:R_1206_3216Metric, symbol Device:R_Small_US
- added T? (x2): RN102-2-02-1M1, Inductor_THT:Choke_Schaffner_RN102-04-14.0x14.0mm, symbol Filter:Choke_Schaffner_RN102-2-02-1M1
- added TP? (x6): TestPoint, TestPoint:TestPoint_Pad_2.0x2.0mm, symbol Connector:TestPoint
- added TR?: POE120PL-12L, Scott:Transformer_Coilcraft_POE120PL, symbol Scott:Transformer_POE120PL-12L
- added U?: TPS54A24RTWR, QFN50P400X400X80-25N, symbol CM4IO:TPS54A24RTWR
- added U?: TS2431-AILT, digikey-footprints:SOT-23-3, symbol dk_PMIC-Voltage-Reference:TL431AIDBZR
- added U? (x2): STL90N6F7, Scott:TRANS_STL60P4LLF6, symbol STL90N6F7:STL90N6F7
Connections:
- net 12V: now also C?.1, C?.1, C?.1, C?.1, C?.1, D?.1 (K), L?.2, R?.1, R?.2, R?.2
- net Earth: now also C?.1, C?.1, C?.1, C?.1, C?.1, C?.2, D?.1 (A1), D?.1 (A1), D?.2 (A2), D?.2 (A2), J?.21 (SHIELD), J?.22 (SHIELD), R?.2
- net GND: now also C?.1, C?.1, C?.2, C?.2, C?.2, C?.2, C?.2, C?.2, C?.2, C?.2, C?.2, C?.2, C?.2, C?.2, C?.2, C?.2, C?.2, C?.2, D?.1 (A), D?.1 (A), J?.2, J?.3, LED?.1 (K), R?.1, R?.1, R?.2, R?.2, R?.2, R?.2, R?.2, TP?.1, U?.1 (AGND), U?.1 (S_1), U?.1 (S_1), U?.12 (PGND-4), U?.13 (PGND-1), U?.14 (PGND-2), U?.15 (PGND-7), U?.2 (S_2), U?.2 (S_2), U?.3 (A), U?.3 (S_3), U?.3 (S_3), U?.4 (PGND), U?.5 (PGND-5), U?.6 (PGND-6), U?.7 (PGND-3)
- net GNDA: now also C?.1, C?.1, C?.1, C?.2, IC?.1 (AGND), IC?.17 (EP), Q?.3, R?.1, R?.1, R?.1, R?.2
- net GNDPWR: now also C?.1, C?.1, C?.2, C?.2, C?.2, C?.2, C?.2, C?.2, C?.2, C?.2, C?.2, C?.2, C?.2, C?.2, C?.2, C?.2, C?.2, C?.2, C?.2, C?.2, C?.2, C?.2, C?.2, C?.2, C?.2, C?.2, C?.2, C?.2, D?.1 (K), D?.2 (A), D?.2 (A), D?.2 (A2), FB?.2, IC?.10 (FAUX), IC?.10 (PGND), IC?.13 (GND12_1), IC?.14 (ARTN), IC?.14 (GND12_2), IC?.15 (RTN), IC?.21 (GND36_1), IC?.22 (GND36_2), IC?.3 (STBY), IC?.34 (GND45_1), IC?.35 (GND45_2), IC?.42 (GND78_1), IC?.43 (GND78_2), IC?.6 (AGND), IC?.9 (SRT), J?.2, Q?.1 (S_1), Q?.2 (S_2), Q?.3 (S_3), R?.1, R?.1, R?.1, R?.1, R?.1, R?.1, R?.2, R?.2, R?.2, R?.2, R?.2, R?.2, TR?.1
- net IN_12: now also C?.1, FB?.2, IC?.12 (IN12_1), IC?.15 (IN12_2), IC?.16 (IN12_3), IC?.EP4
- net IN_36: now also C?.2, FB?.2, IC?.19 (IN36_1), IC?.20 (IN36_2), IC?.23 (IN36_3), IC?.EP3
- net IN_45: now also C?.1, FB?.2, IC?.33 (IN45_1), IC?.36 (IN45_2), IC?.37 (IN45_3), IC?.EP2
- net IN_78: now also C?.2, FB?.2, IC?.1 (IN78_1), IC?.40 (IN78_2), IC?.41 (IN78_3), IC?.EP1
- net PGD: now also C?.1, IC?.25 (PGD), IC?.6 (PGD), R?.2
- net POE_LEDG+O-: now also J?.20 (LEDG+_O-)
- net POE_LEDG-O+: now also J?.19 (LEDG-_O+)
- net POE_LEDY+: now also J?.18 (LEDY+)
- net POE_LEDY-: now also J?.17 (LEDY-)
- net POE_TD1_N: now also J?.10 (TRD1-)
- net POE_TD1_P: now also J?.11 (TRD1+)
- net POE_TD2_N: now also J?.5 (TRD2-)
- net POE_TD2_P: now also J?.4 (TRD2+)
- net POE_TD3_N: now also J?.2 (TRD3-)
- net POE_TD3_P: now also J?.3 (TRD3+)
- net POE_TD4_N: now also J?.9 (TRD4-)
- net POE_TD4_P: now also J?.8 (TRD4+)
- net VB: now also C?.1, IC?.2 (VB), LED?.2 (A), LED?.2 (A), LED?.2 (A), R?.1
- net VDC: now also C?.1, C?.1, C?.1, C?.1, C?.1, C?.1, C?.1, C?.1, D?.1, D?.1 (K), D?.2 (A), IC?.27 (VOUT_1), IC?.28 (VOUT_2), L?.1
- net VOB: now also C?.1, C?.2, D?.1 (A), D?.1 (A1), IC?.17 (VOB_1), IC?.18 (VOB_2), IC?.29 (VOB_3), IC?.30 (VDD), IC?.38 (VOB_4), IC?.39 (VOB_5), IC?.EP5, IC?.EP6, R?.1
- new net: C?.2, D?.2 (A), D?.2 (A), D?.2 (A), D?.2 (A), FB?.1
- new net: C?.2, C?.2, D?.2 (A), R?.1, U?.1 (K)
- new net: Q?.2, R?.2
- new net: C?.1, C?.1, D?.1 (K), L?.1, R?.1, R?.1, TR?.10, U?.5 (D_1), U?.6 (D_2), U?.7 (D_3), U?.8 (D_4)
- new net: C?.1, D?.2 (A), FB?.2, R?.1
- new net: IC?.8 (T1), R?.1
- new net: LED?.1 (K), R?.2 (x3)
- new net: C?.1, IC?.11 (RAUX), R?.1, R?.1
- new net: C?.1, D?.1 (K), D?.1 (K), D?.1 (K), D?.1 (K), FB?.1
- new net: C?.1, IC?.8 (VIN), R?.1
- new net: C?.1, C?.1, C?.1, L?.2, R?.2, TR?.5
- new net: C?.2, J?.6 (TRCT2)
- new net: C?.1, D?.1 (K), D?.2 (A), R?.1
- new net: C?.2, Q?.5 (D_1), Q?.6 (D_2), Q?.7 (D_3), Q?.8 (D_4), TR?.2
- new net: D?.2 (A), TR?.6
- new net: C?.1, D?.1 (K), R?.1, R?.1, TR?.8, U?.5 (D_1), U?.6 (D_2), U?.7 (D_3), U?.8 (D_4)
- new net: C?.1, D?.1 (A1), D?.2 (A2), J?.13 (VC1), T?.1
- new net: C?.1, FB?.1, T?.2 (x2)
- new net: C?.2, D?.2 (A2), D?.2 (A2), J?.14 (VC2), T?.3
- new net: C?.2, FB?.1, T?.4 (x2)
- new net: IC?.4 (CLS1), R?.1
- new net: C?.2, D?.3 (K), Q?.1 (B), R?.2 (x2)
- new net: C?.2, IC?.14 (CS), R?.2
- new net: D?.2 (A), Q?.2 (E), R?.2, U?.4 (G) (x2)
- new net: Q?.1 (S_1), Q?.2 (S_2), Q?.3 (S_3), R?.1, R?.2, R?.2
- new net: C?.1, U?.18 (BOOT)
- new net: C?.2, L?.1, U?.10 (SW-2), U?.11 (SW-1), U?.8 (SW), U?.9 (SW-3)
- new net: C?.1, FB?.1, J?.1
- new net: Q?.3 (C), R?.2 (x2)
- new net: C?.2, FB?.1, J?.2
- new net: D?.2, J?.1, LED?.2 (A), R?.2
- new net: C?.1, IC?.11 (CS), R?.2
- new net: C?.1, D?.2 (A), Q?.4 (G), R?.2
- new net: C?.1, Q?.5 (D_1), Q?.6 (D_2), Q?.7 (D_3), Q?.8 (D_4)
- new net: C?.2, IC?.2 (SS)
- new net: C?.1, D?.1 (A1), D?.1 (A1), J?.15 (VC3), T?.1
- new net: C?.2, D?.1 (A1), D?.2 (A2), J?.16 (VC4), T?.3
- new net: C?.2, R?.1
- new net: R?.1, R?.2
- new net: IC?.4 (FSW), R?.2
- new net: C?.1, D?.3 (K), IC?.32 (VCP)
- new net: D?.1 (K), D?.1 (K), L?.2
- new net: IC?.5 (RT), R?.1
- new net: LED?.1 (K), R?.1
- new net: C?.1, R?.1, R?.1, R?.1, U?.2 (REF)
- new net: C?.1, R?.2 (x2)
- new net: IC?.15 (CTL), Q?.4, R?.1
- new net: C?.2, R?.2
- new net: C?.2, D?.2 (A), Q?.4 (G), R?.1
- new net: C?.1, J?.1, Q?.5 (D)
- new net: C?.1, C?.1, L?.2
- new net: C?.1, C?.1, C?.1, IC?.12 (VC), L?.1
- new net: C?.2, IC?.24 (CTRL)
- new net: IC?.31 (DET), R?.2
- new net: IC?.5 (CLS2), R?.1
- new net: IC?.7 (T0), R?.1
- new net: IC?.9 (T2), R?.1
- new net: R?.1, R?.2, R?.2
- new net: C?.1, IC?.10 (VB)
- new net: C?.2, IC?.11 (GAT2)
- new net: C?.1, R?.1, U?.22 (COMP)
- new net: IC?.16 (BLK), R?.2
- new net: IC?.3 (DT), R?.2
- new net: D?.1 (K), IC?.9 (GAT1), R?.1
- new net: C?.2, J?.12 (TRCT1)
- new net: C?.2, U?.21 (SS/TRK)
- new net: IC?.2 (DEN), R?.2
- new net: IC?.3 (CLS), R?.1
- new net: C?.2, J?.1 (TRCT3)
- new net: D?.2 (A), Q?.4 (G), R?.2, R?.2
- new net: R?.1, U?.19 (PGOOD)
- new net: R?.1, R?.2, U?.23 (FB)
- new net: R?.1, U?.24 (RT/CLK)
- new net: LED?.2 (A), R?.1
- new net: C?.2, Q?.1, R?.2
- new net: C?.2, J?.7 (TRCT4)
- new net +12v: C?.1, C?.1, D?.1 (K), Q?.1 (S), Q?.2 (S), Q?.3 (S), TP?.1
- new net +3.3v: C?.1, C?.1, L?.2, R?.1, R?.2, TP?.1
- new net +5v: C?.1, C?.1, C?.1, U?.16 (VIN-1), U?.17 (VIN-2), U?.2 (VIN), U?.3 (VIN-3)
- new net APD: C?.1, IC?.4 (APD), R?.1, R?.2
- new net T2P: IC?.6 (T2P), TP?.1
- new net TR0_TAP: D?.1 (K), D?.2 (A)
- new net TR1_TAP: D?.1 (K), D?.2 (A)
- new net TR2_TAP: D?.1 (K), D?.2 (A)
- new net TR3_TAP: D?.1 (K), D?.2 (A)
- new net VDD: C?.1, C?.1, C?.1, D?.1 (K), D?.1 (K), FB?.2, IC?.1 (VDD), L?.1, R?.1, R?.1, TP?.1
- new net VSS: C?.2, D?.2 (A), FB?.2, IC?.16 (VSS), IC?.17 (EP), R?.2, TP?.1
- no-connect marks 4 -> 6
Other:
- note added: "+12v Input"
- note added: "+3.3v @6A PSU ( 5v Input )"
- note added: "2.1mm Tip +ve"
- note added: "2.5mm Tip +ve"
- note added: "21.6v - 57v Input"
- note added: "Ideal diode to prevent reverse polarity at the input"
- company: ISis ImageStream Internet Solutions, Inc. -> (none)
- title: AP2100 -> (none)

Commit message: Finish PoE section Rename CM4IO library as AP2100
Parts:
- removed C? (x7): 1nF, Capacitor_SMD:C_0805_2012Metric, symbol Device:C_Small
- removed C? (x3): 2.2nF, Capacitor_SMD:C_1812_4532Metric, symbol Device:C_Small
- removed C? (x4): .1uF, Capacitor_SMD:C_0402_1005Metric, symbol Device:C_Small
- removed C?: 100pF, Capacitor_SMD:C_0603_1608Metric, symbol Device:C_Small
- removed C? (x2): 100u 6.3v, Capacitor_SMD:C_1206_3216Metric, symbol Device:C
- removed C?: 100uF, Capacitor_SMD:CP_Elec_6.3x5.9, symbol Device:CP1_Small
- removed C? (x2): 100pF, Capacitor_SMD:C_0805_2012Metric, symbol Device:C_Small
- removed C?: 100n 16v, Capacitor_SMD:C_0402_1005Metric, symbol Device:C
- removed C? (x5): 4.7uF, Capacitor_SMD:C_1210_3225Metric, symbol Device:C_Small
- removed C? (x3): 47uF, Capacitor_SMD:C_1210_3225Metric, symbol Device:C_Small
- removed C? (x3): 10nF, Capacitor_SMD:C_0603_1608Metric, symbol Device:C_Small
- removed C? (x4): 33nF, Capacitor_SMD:C_0805_2012Metric, symbol Device:C_Small
- removed C? (x6): 100nF, Capacitor_SMD:C_0603_1608Metric, symbol Device:C_Small
- removed C?: 47nF, Capacitor_SMD:C_1206_3216Metric, symbol Device:C_Small
- removed C?: 10u 10v, Capacitor_SMD:C_0805_2012Metric, symbol Device:C
- removed C?: 100n 50v, Capacitor_SMD:C_0603_1608Metric, symbol Device:C
- removed C?: 10u 35v, Capacitor_SMD:C_0805_2012Metric, symbol Device:C
- removed C?: 22nF, Capacitor_SMD:C_0603_1608Metric, symbol Device:C_Small
- removed C?: 1u 35v, Capacitor_SMD:C_0402_1005Metric, symbol Device:C
- removed C?: 10nF, Capacitor_SMD:C_0805_2012Metric, symbol Device:C_Small
- removed C?: 13p 50v, Capacitor_SMD:C_0402_1005Metric, symbol Device:C
- removed C? (x2): 2.2uF 25V, Capacitor_SMD:C_0805_2012Metric, symbol Device:C_Small
- removed C?: 100n 100v, Capacitor_SMD:C_0402_1005Metric, symbol Device:C
- removed C?: 1nF, Capacitor_SMD:C_0603_1608Metric, symbol Device:C_Small
- removed C?: 220pF, Capacitor_SMD:C_0603_1608Metric, symbol Device:C_Small
- removed C? (x2): 33uF, LIB_EEEFK2A330P:CAPAE1030X1050N, symbol AP2100-rescue:EEEFK2A330P-EEEFK2A330P
- removed C?: 100n, Capacitor_SMD:C_0402_1005Metric, symbol Device:C
- removed C?: 100nF, Capacitor_SMD:C_0805_2012Metric, symbol Device:C_Small
- removed C?: 1u 35v, Capacitor_SMD:C_0603_1608Metric, symbol Device:C
- removed C?: 1.5nF, Capacitor_SMD:C_0603_1608Metric, symbol Device:C_Small
- removed C?: 1.8n 50v, Capacitor_SMD:C_0603_1608Metric, symbol Device:C
- removed D?: BZX84C10LT1G, Package_TO_SOT_SMD:SOT-23, symbol Diode:BAS19
- removed D? (x5): BAS16J, Diode_SMD:D_SOD-323, symbol Device:D_ALT
- removed D?: STPS4S200S, LIB_STPS4S200S:DIOM8059X265N, symbol AP2100-rescue:STPS4S200S-STPS4S200S
- removed D? (x6): SM15T68CA, Diode_SMD:D_SMC, symbol Device:D_TVS_ALT
- removed D?: BZX84C10, Package_TO_SOT_SMD:SOT-23, symbol Diode:BAS19
- removed D? (x3): BAS70, Diode_SMD:D_SOD-323, symbol Device:D_ALT
- removed D?: BAV70, Package_TO_SOT_SMD:SOT-23, symbol Diode:BAV70
- removed D?: MMBZ5242BLT3G, Diode_SMD:D_SOT-23_ANK, symbol Diode:BZX84Cxx
- removed D?: SMAJ58A, Diode_SMD:D_SMA, symbol Device:D_Schottky_ALT
- removed D?: SMAJ58A, Diode_SMD:D_SMA, symbol Device:D_TVS_ALT
- removed FB? (x4): 220 OHM, Inductor_SMD:L_0805_2012Metric, symbol Device:L
- removed IC?: PM8805TR, LIB_PM8805TR:PM8805TR, symbol AP2100-rescue:PM8805TR-PM8805TR
- removed IC?: PM8804TR, LIB_PM8804TR:QFN50P340X340X90-17N, symbol AP2100-rescue:PM8804TR-PM8804TR
- removed J?: Barrel_Jack, Connector_BarrelJack:BarrelJack_Horizontal, symbol Connector:Barrel_Jack
- removed J?: Barrel_Jack, Connector_BarrelJack:BarrelJack_Horizontal, symbol CM4IO:Barrel_Jack
- removed J?: 0826-1X1T-GH-F, 0826-1X1T-GH-F:BEL_0826-1X1T-GH-F, symbol AP2100-rescue:0826-1X1T-GH-F-0826-1X1T-GH-F
- removed L?: 10uH, LIB_7443631000:WE-HCF_201322, symbol 7443631000:7443631000
- removed L?: 5.6uH, Inductor_SMD:L_Coilcraft_XAL5030, symbol Device:L
- removed L?: 1mH, Inductor_SMD:L_Coilcraft_LPS4018, symbol Device:L
- removed L?: XAL4020-601MEB, Inductor_SMD:L_Coilcraft_XxL4020, symbol pspice:INDUCTOR
- removed LED?: AUX, LED_SMD:LED_0603_1608Metric, symbol Device:LED_ALT
- removed LED?: T0, LED_SMD:LED_0603_1608Metric, symbol Device:LED_ALT
- removed LED?: T1, LED_SMD:LED_0603_1608Metric, symbol Device:LED_ALT
- removed LED?: T2, LED_SMD:LED_0603_1608Metric, symbol Device:LED_ALT
- removed LED?: +12V, LED_SMD:LED_0603_1608Metric, symbol Device:LED_ALT
- removed Q?: FDMC86259P, LIB_FDMC86259P:FDMC86160, symbol FDMC86259P:FDMC86259P
- removed Q?: DMP3013SFV-7, Package_SON:Diodes_PowerDI3333-8, symbol Transistor_FET:DMP3013SFV
- removed Q?: BSC190N15NS3GATMA1, Scott:TRANS_BSC100N06LS3GATMA1, symbol BSC190N15NS3GATMA1:BSC190N15NS3GATMA1
- removed Q? (x2): PBSS4240T, Package_TO_SOT_SMD:SOT-23, symbol Device:Q_NPN_BEC
- removed Q?: FOD817AS, LIB_FOD817AS:SOP254P1016X385-4N, symbol FOD817AS:FOD817AS
- removed R? (x2): 2K, Resistor_SMD:R_0603_1608Metric, symbol Device:R_Small_US
- removed R? (x3): 3.9K, Resistor_SMD:R_0603_1608Metric, symbol Device:R_Small_US
- removed R? (x6): 10K, Resistor_SMD:R_0603_1608Metric, symbol Device:R_Small_US
- removed R? (x2): 10, Resistor_SMD:R_0805_2012Metric, symbol Device:R_Small_US
- removed R?: 47K, Resistor_SMD:R_0603_1608Metric, symbol Device:R_Small_US
- removed R?: 36.5, Resistor_SMD:R_0805_2012Metric, symbol Device:R_Small_US
- removed R? (x2): 22, Resistor_SMD:R_0603_1608Metric, symbol Device:R_Small_US
- removed R?: 88.7K, Resistor_SMD:R_0603_1608Metric, symbol Device:R_Small_US
- removed R? (x2): 4.7K, Resistor_SMD:R_0603_1608Metric, symbol Device:R_Small_US
- removed R?: 390, Resistor_SMD:R_0603_1608Metric, symbol Device:R_Small_US
- removed R?: 100K, Resistor_SMD:R_0603_1608Metric, symbol Device:R_Small_US
- removed R?: 20K, Resistor_SMD:R_0603_1608Metric, symbol Device:R_Small_US
- removed R? (x3): 1K, Resistor_SMD:R_0603_1608Metric, symbol Device:R_Small_US
- removed R?: 26.1K, Resistor_SMD:R_0603_1608Metric, symbol Device:R_Small_US
- removed R?: 10K 1%, Resistor_SMD:R_0402_1005Metric, symbol Device:R
- removed R? (x2): 0, Resistor_SMD:R_0603_1608Metric, symbol Device:R_Small_US
- removed R?: 12K 1%, Resistor_SMD:R_0402_1005Metric, symbol Device:R
- removed R?: 18, Resistor_SMD:R_0805_2012Metric, symbol Device:R_Small_US
- removed R?: 330K, Resistor_SMD:R_0603_1608Metric, symbol Device:R_Small_US
- removed R?: 150, Resistor_SMD:R_0805_2012Metric, symbol Device:R_Small_US
- removed R?: 0, Resistor_SMD:R_2010_5025Metric, symbol Device:R_Small_US
- removed R?: R100, Resistor_SMD:R_1210_3225Metric, symbol Device:R_Small_US
- removed R?: 27.1K .1%, Resistor_SMD:R_0805_2012Metric, symbol Device:R
- removed R?: 5.23K, Resistor_SMD:R_0603_1608Metric, symbol Device:R_Small_US
- removed R?: 10K, Resistor_SMD:R_0805_2012Metric, symbol Device:R_Small_US
- removed R?: 48.7K 1%, Resistor_SMD:R_0402_1005Metric, symbol Device:R
- removed R?: 130K, Resistor_SMD:R_0603_1608Metric, symbol Device:R_Small_US
- removed R?: 0R05, Resistor_SMD:R_1210_3225Metric, symbol Device:R_Small_US
- removed R?: 100K 1%, Resistor_SMD:R_0402_1005Metric, symbol Device:R
- removed R?: 6.04K 1%, Resistor_SMD:R_0402_1005Metric, symbol Device:R
- removed R?: 0, Resistor_SMD:R_1206_3216Metric, symbol Device:R_Small_US
- removed T? (x2): RN102-2-02-1M1, Inductor_THT:Choke_Schaffner_RN102-04-14.0x14.0mm, symbol Filter:Choke_Schaffner_RN102-2-02-1M1
- removed TP? (x3): TestPoint, TestPoint:TestPoint_Pad_2.0x2.0mm, symbol Connector:TestPoint
- removed TR?: POE120PL-12L, Scott:Transformer_Coilcraft_POE120PL, symbol Scott:Transformer_POE120PL-12L
- removed U?: TPS54A24RTWR, QFN50P400X400X80-25N, symbol CM4IO:TPS54A24RTWR
- removed U?: TS2431-AILT, digikey-footprints:SOT-23-3, symbol dk_PMIC-Voltage-Reference:TL431AIDBZR
- removed U? (x2): STL90N6F7, Scott:TRANS_STL60P4LLF6, symbol STL90N6F7:STL90N6F7
- added C? (x3): 47u 10v, Capacitor_SMD:C_1206_3216Metric, symbol Device:C
- added C?: 10n 100v, Capacitor_SMD:C_0603_1608Metric, symbol Device:C
- added C? (x2): 330u 6.3v, Capacitor_SMD:CP_Elec_6.3x7.7, symbol AP2100-rescue:EEEFK2A330P-EEEFK2A330P
- added C? (x2): 1u 16v, Capacitor_SMD:C_0805_2012Metric, symbol Device:C
- added C?: .1u 100v, Capacitor_SMD:C_0603_1608Metric, symbol Device:C
- added C?: 1u 25v, Capacitor_SMD:C_0805_2012Metric, symbol Device:C
- added C?: 22u 25v, Capacitor_SMD:CP_Elec_5x5.8, symbol AP2100-rescue:EEEFK2A330P-EEEFK2A330P
- added C?: .022u 50v, Capacitor_SMD:C_0603_1608Metric, symbol Device:C
- added C? (x2): .47u 16V, Capacitor_SMD:C_0603_1608Metric, symbol Device:C
- added C?: 1000p 100v, Capacitor_SMD:C_0805_2012Metric, symbol Device:C
- added C?: 2.2nF 2KV, Capacitor_SMD:C_1812_4532Metric, symbol Device:C_Small
- added D? (x2): BAT54S, Package_TO_SOT_SMD:SOT-23, symbol Diode:BAT54S
- added D?: MURS120T3G, Diode_SMD:D_SMB, symbol Device:D_ALT
- added D?: 1N4148W, Diode_SMD:D_SOD-123, symbol Device:D_ALT
- added D?: MBR0530T1G, Diode_SMD:D_SOD-123, symbol Device:D_Schottky_ALT
- added L?: XAL5030-331MEB, Inductor_SMD:L_Coilcraft_XAL5030, symbol pspice:INDUCTOR
- added Q?: BSC520N15NS3 G, Scott:TRANS_BSC100N06LS3GATMA1, symbol BSC190N15NS3GATMA1:BSC190N15NS3GATMA1
- added Q?: MMBT2907ALT1G, Package_TO_SOT_SMD:SOT-23, symbol Device:Q_PNP_BEC
- added Q?: MMBT3906LT1G, Package_TO_SOT_SMD:SOT-23, symbol Device:Q_PNP_BEC
- added R?: 10 1W, Resistor_SMD:R_2512_6332Metric, symbol Device:R
- added R?: 1K 1%, Resistor_SMD:R_0402_1005Metric, symbol Device:R
- added R?: 13.7K 1%, Resistor_SMD:R_0402_1005Metric, symbol Device:R
- added R?: 332 1%, Resistor_SMD:R_0402_1005Metric, symbol Device:R
- added R? (x4): 10K 1%, Resistor_SMD:R_0402_1005Metric, symbol Device:R
- added R?: 39K 1%, Resistor_SMD:R_0805_2012Metric, symbol Device:R
- added R?: 604 1%, Resistor_SMD:R_0402_1005Metric, symbol Device:R
- added R?: 3.65K 1%, Resistor_SMD:R_0402_1005Metric, symbol Device:R
- added R?: 10, Resistor_SMD:R_0805_2012Metric, symbol Device:R
- added R?: 49.9 1%, Resistor_SMD:R_0402_1005Metric, symbol Device:R
- added R?: 41.2K 1%, Resistor_SMD:R_0402_1005Metric, symbol Device:R
- added R?: .09 1%, Resistor_SMD:R_0805_2012Metric, symbol Device:R
- added R? (x2): 43.2 1%, Resistor_SMD:R_0402_1005Metric, symbol Device:R
- added TP? (x5): TestPoint, TestPoint:TestPoint_Pad_2.0x2.0mm, symbol Connector:TestPoint
- added TR?: Transformer_JA4456-DLB, AP2100:SOP300P3000X1270-12N, symbol AP2100:Transformer_JA4456-DLB
- added TR?: PH9085.011NLT, symbol AP2100:TRANSF5
- added U?: SIR422DP-T1-GE3, Package_SO:PowerPAK_SO-8_Single, symbol STL90N6F7:STL90N6F7
- added U?: TCMT1107, Package_SO:SOP-4_4.4x2.6mm_P1.27mm, symbol Isolator:TCMT1107
- added U?: TLV431ACDBZR, Package_TO_SOT_SMD:SOT-23, symbol dk_PMIC-Voltage-Reference:TL431AIDBZR
- IC?: symbol CM4IO:TPS23751PWPR -> AP2100:TPS23751PWPR
Connections:
- net +5v: now also C?.1, C?.1, L?.2, R?.2, TP?.1
- net GND: now also C?.2, C?.2, C?.2, C?.2, C?.2, C?.2, C?.2, C?.2, D?.1, Q?.3 (C), R?.1, R?.1, R?.1, R?.1, TP?.1, TR?.3, U?.1 (S_1), U?.2 (S_2), U?.3 (A), U?.3 (S_3)
- net GNDPWR: now also C?.1, C?.2, C?.2, Q?.3 (C), R?.1, R?.1, TR?.5, U?.3
- net VB: now also C?.1, IC?.10 (VB), R?.2, R?.2
- net at C?.1, IC?.11 (CS), R?.2: now also R?.1
- net at C?.1, C?.1, L?.2: now also C?.1, R?.1, TR?.1, TR?.2
- net VC: now reaches IC?.12 (VC)
- net VC: now also C?.1, C?.1, D?.1 (K), TR?.6
- net at IC?.13 (GATE): now also C?.1, R?.1
- net at IC?.8 (CTL): now also C?.2, R?.1, U?.4
- new net: D?.2, Q?.2 (E), R?.2, U?.4 (G)
- new net: C?.1, TP?.1, TR?.7, TR?.8, TR?.9, U?.5 (D_1), U?.6 (D_2), U?.7 (D_3), U?.8 (D_4)
- new net: C?.2, R?.2
- new net: C?.1, C?.1, C?.1, C?.1, L?.1, TR?.10, TR?.11, TR?.12
- new net: C?.1, R?.1
- new net: C?.1, C?.1, D?.1, D?.3, R?.1, U?.1 (K), U?.2
- new net: C?.2, R?.1, R?.2, U?.2 (REF)
- new net: Q?.1 (S_1), Q?.2 (S_2), Q?.3 (S_3), R?.2, R?.2
- new net: D?.1 (K), Q?.2 (E), Q?.4 (G), R?.2
- new net: D?.2 (A), Q?.5 (D_1), Q?.6 (D_2), Q?.7 (D_3), Q?.8 (D_4), TP?.1, TR?.3, TR?.4
- new net: D?.2, R?.1, R?.2, R?.2, R?.2, TP?.1
- new net: R?.1, U?.1
- new net: D?.3, Q?.1 (B), R?.2
- new net: C?.2, D?.1 (K), R?.2
- new net: R?.2, TR?.6
- new net: C?.2, TR?.4
- new net: C?.1, TR?.1
- new net: C?.2, R?.1, R?.2
- new net: D?.2 (A), R?.1
- new net: D?.2 (A), Q?.1 (B), R?.2
- no-connect marks 6 -> 3
Other:
- note added: "5V @ 5A"
- note removed: "+12v Input"
- note removed: "+3.3v @6A PSU ( 5v Input )"
- note removed: "12V 4A"
- note removed: "2.1mm Tip +ve"
- note removed: "Ideal diode to prevent reverse polarity at the input"
- note removed: "NOTE: Class 6 PD device 50W"
- note removed: "Note: DC IN 18V-48V"
- moved on the sheet: C?, D?, FB?, J?, R?, TP?
