File: AP2100/RTC.kicad_sch (KiCad schematic)
At the start: 14 parts, among them J17 Molex 470531000, U11 EMC2301-1-ACZL-TR, U14 74LVC1G07SE-7, U8 PCF85063AT/AAZ, Y2 X32K768S301

Commit message: Finish PoE section Rename CM4IO library as AP2100
Parts:
- U11: symbol CM4IO:EMC2301 -> AP2100:EMC2301
- U14: symbol CM4IO:74LVC1G07_copy -> AP2100:74LVC1G07_copy
Changed lines of the file:
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@@
   (junction (at 213.36 49.53) (diameter 1.016) (color 0 0 0 0))
   (junction (at 213.36 62.23) (diameter 1.016) (color 0 0 0 0))
+  (no_connect (at 138.43 138.43))
   (no_connect (at 138.43 135.89))
-  (no_connect (at 138.43 138.43))
   (wire (pts (xy 38.1 44.45) (xy 46.228 44.45))
     (stroke (width 0) (type solid) (color 0 0 0 0))
@@
     )
   )
-  (symbol (lib_id "CM4IO:74LVC1G07_copy") (at 227.33 62.23 0) (unit 1)
+  (symbol (lib_id "AP2100:74LVC1G07_copy") (at 227.33 62.23 0) (unit 1)
     (in_bom yes) (on_board yes)
     (property "Reference" "U14" (id 0) (at 230.505 55.88 0))
@@
     )
   )
-  (symbol (lib_id "CM4IO:EMC2301") (at 130.81 146.05 0) (unit 1)
+  (symbol (lib_id "AP2100:EMC2301") (at 130.81 146.05 0) (unit 1)
     (in_bom yes) (on_board yes)
     (property "Reference" "U11" (id 0) (at 128.905 129.159 0))
