File: AP2100/AP2100v4.kicad_sch (KiCad schematic)
At the start: 8 parts

Commit message: Finish PoE section Rename CM4IO library as AP2100
Other:
- sheet PoE ports: added +5v, TR0_TAP, TR1_TAP, TR2_TAP, TR3_TAP; removed none
- note added: "Connectors ------- Ethernet 40way RPI Jumpers"
- note removed: "Connectors ------- Ethernet SDCARD 40way RPI Jumpers"

Commit message: Finish PCie routing
Other:
- added sheet Additional Ethernet (eth_add.kicad_sch)
- added sheet PCIe Switch Power and GND (pcie_pwr_gnd.kicad_sch)
- sheet PCIe Routing ports: added +1.5v, +3.3v; removed +12v
- sheet PSUs ports: added +1.5v; removed +12v
