File: AP2100/CM4_HighSpeed.kicad_sch (KiCad schematic)
At the start: 6 parts, among them J4 Conn_01x22_Female, J5 Conn_01x22_Female, J6 THD-02-R

Commit message: Finish PoE section Rename CM4IO library as AP2100
Parts:
- Module1: footprint CM4IO:Raspberry-Pi-4-Compute-Module -> AP2100:Raspberry-Pi-4-Compute-Module; symbol CM4IO:ComputeModule4-CM4 -> AP2100:ComputeModule4-CM4
Changed lines of the file:
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@@
   (junction (at 157.48 133.35) (diameter 1.016) (color 0 0 0 0))
   (junction (at 157.48 140.97) (diameter 1.016) (color 0 0 0 0))
+  (no_connect (at 102.87 39.37))
+  (no_connect (at 160.02 71.12))
+  (no_connect (at 160.02 63.5))
+  (no_connect (at 41.91 29.21))
+  (no_connect (at 102.87 26.67))
+  (no_connect (at 41.91 31.75))
+  (no_connect (at 160.02 60.96))
+  (no_connect (at 160.02 138.43))
+  (no_connect (at 160.02 53.34))
   (no_connect (at 160.02 55.88))
-  (no_connect (at 160.02 53.34))
-  (no_connect (at 160.02 138.43))
-  (no_connect (at 102.87 39.37))
-  (no_connect (at 102.87 26.67))
-  (no_connect (at 41.91 29.21))
-  (no_connect (at 160.02 71.12))
-  (no_connect (at 160.02 60.96))
-  (no_connect (at 41.91 31.75))
-  (no_connect (at 160.02 63.5))
   (wire (pts (xy 25.4 74.93) (xy 41.91 74.93))
     (stroke (width 0) (type solid) (color 0 0 0 0))
@@
     )
   )
-  (symbol (lib_id "CM4IO:ComputeModule4-CM4") (at -67.31 87.63 0) (unit 2)
+  (symbol (lib_id "AP2100:ComputeModule4-CM4") (at -67.31 87.63 0) (unit 2)
     (in_bom yes) (on_board yes)
     (property "Reference" "Module1" (id 0) (at 72.39 15.367 0))
     (property "Value" "ComputeModule4" (id 1) (at 72.39 17.6784 0))
-    (property "Footprint" "CM4IO:Raspberry-Pi-4-Compute-Module" (id 2) (at 74.93 114.3 0)
-      (effects (font (size 1.27 1.27)) hide)
-    )
+    (property "Footprint" "AP2100:Raspberry-Pi-4-Compute-Module" (id 2) (at 74.93 114.3 0)
+      (effects (font (size 1.27 1.27)) hide)
+    )
