File: AP2100/PSUs.kicad_sch (KiCad schematic)
At the start: 25 parts

Commit message: Finish PoE section Rename CM4IO library as AP2100
Parts:
- U?: symbol CM4IO:TPS628640AYCGR -> AP2100:TPS628640AYCGR
- U?: symbol CM4IO:TPS54A24RTWR -> AP2100:TPS54A24RTWR
Changed lines of the file:
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@@
   (symbol (lib_id "power:GND") (at 93.98 86.36 0) (unit 1)
     (in_bom yes) (on_board yes)
-    (property "Reference" "#PWR?" (id 0) (at 93.98 92.71 0)
+    (property "Reference" "#PWR0155" (id 0) (at 93.98 92.71 0)
       (effects (font (size 1.27 1.27)) hide)
     )
@@
   (symbol (lib_id "power:GND") (at 147.32 149.86 0) (unit 1)
     (in_bom yes) (on_board yes)
-    (property "Reference" "#PWR?" (id 0) (at 147.32 156.21 0)
+    (property "Reference" "#PWR0157" (id 0) (at 147.32 156.21 0)
       (effects (font (size 1.27 1.27)) hide)
     )
@@
   (symbol (lib_id "power:GND") (at 157.48 86.36 0) (unit 1)
     (in_bom yes) (on_board yes)
-    (property "Reference" "#PWR?" (id 0) (at 157.48 92.71 0)
+    (property "Reference" "#PWR0156" (id 0) (at 157.48 92.71 0)
       (effects (font (size 1.27 1.27)) hide)
     )
@@
     )
   )
-  (symbol (lib_id "CM4IO:TPS628640AYCGR") (at 143.51 127 0) (unit 1)
+  (symbol (lib_id "AP2100:TPS628640AYCGR") (at 143.51 127 0) (unit 1)
     (in_bom yes) (on_board yes)
     (property "Reference" "U?" (id 0) (at 143.51 111.76 0))
@@
     )
   )
-  (symbol (lib_id "CM4IO:TPS54A24RTWR") (at 139.7 60.96 0) (unit 1)
+  (symbol (lib_id "AP2100:TPS54A24RTWR") (at 139.7 60.96 0) (unit 1)
     (in_bom yes) (on_board yes)
     (property "Reference" "U?" (id 0) (at 139.7 33.02 0))

Commit message: Add AP3000 single radio for security cameras. Add CM4IO Raspi board
Parts:
- U16: renamed from U?; footprint QFN50P400X400X80-25N -> AP2100:QFN50P400X400X80-25N
- gave numbers to parts that had none: 22
Changed lines of the file:
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@@
   (symbol (lib_id "Connector:TestPoint") (at 182.88 149.86 180) (unit 1)
     (in_bom yes) (on_board yes)
-    (property "Reference" "TP?" (id 0) (at 181.4068 154.1272 0)
+    (property "Reference" "TP15" (id 0) (at 181.4068 154.1272 0)
       (effects (font (size 1.27 1.27)) (justify left))
     )
@@
   (symbol (lib_id "Connector:TestPoint") (at 185.42 115.57 0) (unit 1)
     (in_bom yes) (on_board yes)
-    (property "Reference" "TP?" (id 0) (at 187.325 111.633 0)
+    (property "Reference" "TP14" (id 0) (at 187.325 111.633 0)
       (effects (font (size 1.27 1.27)) (justify left))
     )
@@
   (symbol (lib_id "Device:R") (at 121.92 143.51 0) (mirror x) (unit 1)
     (in_bom yes) (on_board yes)
-    (property "Reference" "R?" (id 0) (at 124.46 142.367 0)
+    (property "Reference" "R76" (id 0) (at 124.46 142.367 0)
       (effects (font (size 1.27 1.27)) (justify left))
     )
@@
   (symbol (lib_id "Device:R") (at 162.56 80.01 0) (mirror y) (unit 1)
     (in_bom yes) (on_board yes)
-    (property "Reference" "R?" (id 0) (at 167.64 78.613 0)
+    (property "Reference" "R75" (id 0) (at 167.64 78.613 0)
       (effects (font (size 1.27 1.27)) (justify left))
     )
@@
   (symbol (lib_id "Device:R") (at 170.18 43.18 90) (mirror x) (unit 1)
     (in_bom yes) (on_board yes)
-    (property "Reference" "R?" (id 0) (at 171.323 40.64 90)
+    (property "Reference" "R71" (id 0) (at 171.323 40.64 90)
       (effects (font (size 1.27 1.27)) (justify left))
     )
@@
   (symbol (lib_id "Device:R") (at 185.42 71.12 90) (mirror x) (unit 1)
     (in_bom yes) (on_board yes)
-    (property "Reference" "R?" (id 0) (at 186.563 68.58 90)
+    (property "Reference" "R73" (id 0) (at 186.563 68.58 90)
       (effects (font (size 1.27 1.27)) (justify left))
     )
@@
   (symbol (lib_id "Device:R") (at 200.66 59.69 0) (mirror y) (unit 1)
     (in_bom yes) (on_board yes)
-    (property "Reference" "R?" (id 0) (at 205.74 58.293 0)
+    (property "Reference" "R72" (id 0) (at 205.74 58.293 0)
       (effects (font (size 1.27 1.27)) (justify left))
     )
@@
   (symbol (lib_id "Device:R") (at 200.66 74.93 0) (mirror y) (unit 1)
     (in_bom yes) (on_board yes)
-    (property "Reference" "R?" (id 0) (at 205.74 73.533 0)
+    (property "Reference" "R74" (id 0) (at 205.74 73.533 0)
       (effects (font (size 1.27 1.27)) (justify left))
     )
@@
   (symbol (lib_id "pspice:INDUCTOR") (at 173.99 119.38 0) (unit 1)
     (in_bom yes) (on_board yes)
-    (property "Reference" "L?" (id 0) (at 173.99 113.919 0))
+    (property "Reference" "L4" (id 0) (at 173.99 113.919 0))
     (property "Value" "XAL4020-221MEB" (id 1) (at 173.99 116.2304 0))
     (property "Footprint" "Inductor_SMD:L_Coilcraft_XxL4020" (id 2) (at 173.99 119.38 0)
@@
   (symbol (lib_id "pspice:INDUCTOR") (at 185.42 54.61 0) (unit 1)
     (in_bom yes) (on_board yes)
-    (property "Reference" "L?" (id 0) (at 185.42 49.149 0))
+    (property "Reference" "L3" (id 0) (at 185.42 49.149 0))
     (property "Value" "XAL4020-601MEB" (id 1) (at 185.42 51.4604 0))
     (property "Footprint" "Inductor_SMD:L_Coilcraft_XxL4020" (id 2) (at 185.42 54.61 0)
@@
   (symbol (lib_id "Device:C") (at 78.74 62.23 0) (unit 1)
     (in_bom yes) (on_board yes)
-    (property "Reference" "C?" (id 0) (at 81.661 61.0616 0)
+    (property "Reference" "C111" (id 0) (at 81.661 61.0616 0)
       (effects (font (size 1.27 1.27)) (justify left))
     )
@@
   (symbol (lib_id "Device:C") (at 88.9 62.23 0) (unit 1)
     (in_bom yes) (on_board yes)
-    (property "Reference" "C?" (id 0) (at 91.821 61.0616 0)
+    (property "Reference" "C112" (id 0) (at 91.821 61.0616 0)
       (effects (font (size 1.27 1.27)) (justify left))
     )
@@
   (symbol (lib_id "Device:C") (at 99.06 62.23 0) (unit 1)
     (in_bom yes) (on_board yes)
-    (property "Reference" "C?" (id 0) (at 101.981 61.0616 0)
+    (property "Reference" "C113" (id 0) (at 101.981 61.0616 0)
       (effects (font (size 1.27 1.27)) (justify left))
     )
@@
   (symbol (lib_id "Device:C") (at 106.68 132.08 0) (unit 1)
     (in_bom yes) (on_board yes)
-    (property "Reference" "C?" (id 0) (at 109.601 130.9116 0)
+    (property "Reference" "C119" (id 0) (at 109.601 130.9116 0)
       (effects (font (size 1.27 1.27)) (justify left))
     )
@@
   (symbol (lib_id "Device:C") (at 116.84 81.28 90) (unit 1)
     (in_bom yes) (on_board yes)
-    (property "Reference" "C?" (id 0) (at 118.2116 77.089 90)
+    (property "Reference" "C118" (id 0) (at 118.2116 77.089 90)
       (effects (font (size 1.27 1.27)) (justify left))
     )
@@
   (symbol (lib_id "Device:C") (at 165.1 53.34 0) (unit 1)
     (in_bom yes) (on_board yes)
-    (property "Reference" "C?" (id 0) (at 168.021 52.1716 0)
+    (property "Reference" "C110" (id 0) (at 168.021 52.1716 0)
       (effects (font (size 1.27 1.27)) (justify left))
     )
@@
   (symbol (lib_id "Device:C") (at 180.34 78.74 0) (unit 1)
     (in_bom yes) (on_board yes)
-    (property "Reference" "C?" (id 0) (at 183.261 77.5716 0)
+    (property "Reference" "C116" (id 0) (at 183.261 77.5716 0)
       (effects (font (size 1.27 1.27)) (justify left))
     )
@@
   (symbol (lib_id "Device:C") (at 190.5 78.74 0) (unit 1)
     (in_bom yes) (on_board yes)
-    (property "Reference" "C?" (id 0) (at 193.421 77.5716 0)
+    (property "Reference" "C117" (id 0) (at 193.421 77.5716 0)
       (effects (font (size 1.27 1.27)) (justify left))
     )
@@
   (symbol (lib_id "Device:C") (at 193.04 132.08 0) (unit 1)
     (in_bom yes) (on_board yes)
-    (property "Reference" "C?" (id 0) (at 195.961 130.9116 0)
+    (property "Reference" "C120" (id 0) (at 195.961 130.9116 0)
       (effects (font (size 1.27 1.27)) (justify left))
     )
@@
   (symbol (lib_id "Device:C") (at 220.98 68.58 0) (unit 1)
     (in_bom yes) (on_board yes)
-    (property "Reference" "C?" (id 0) (at 223.901 67.4116 0)
+    (property "Reference" "C114" (id 0) (at 223.901 67.4116 0)
       (effects (font (size 1.27 1.27)) (justify left))
     )
@@
   (symbol (lib_id "Device:C") (at 232.41 68.58 0) (unit 1)
     (in_bom yes) (on_board yes)
-    (property "Reference" "C?" (id 0) (at 235.331 67.4116 0)
+    (property "Reference" "C115" (id 0) (at 235.331 67.4116 0)
       (effects (font (size 1.27 1.27)) (justify left))
     )
@@
   (symbol (lib_id "AP2100:TPS628640AYCGR") (at 143.51 127 0) (unit 1)
     (in_bom yes) (on_board yes)
-    (property "Reference" "U?" (id 0) (at 143.51 111.76 0))
+    (property "Reference" "U17" (id 0) (at 143.51 111.76 0))
     (property "Value" "TPS628640AYCGR" (id 1) (at 143.51 114.3 0))
     (property "Footprint" "BGA15C35P3X5_101X174X50" (id 2) (at 156.21 116.84 0)
@@
   (symbol (lib_id "AP2100:TPS54A24RTWR") (at 139.7 60.96 0) (unit 1)
     (in_bom yes) (on_board yes)
-    (property "Reference" "U?" (id 0) (at 139.7 33.02 0))
+    (property "Reference" "U16" (id 0) (at 139.7 33.02 0))
     (property "Value" "TPS54A24RTWR" (id 1) (at 139.7 35.56 0))
-    (property "Footprint" "QFN50P400X400X80-25N" (id 2) (at 139.7 78.74 0)
+    (property "Footprint" "AP2100:QFN50P400X400X80-25N" (id 2) (at 139.7 78.74 0)
       (effects (font (size 1.27 1.27)) (justify left bottom) hide)
     )
