File: AP2100/eth_add.kicad_sch (KiCad schematic)
At the start: 0 parts

Commit message: Add AP3000 single radio for security cameras. Add CM4IO Raspi board
Parts:
- added IC1: WGI210CS_S_LKKM, AP2100:QFN50P900X900X100-65N, symbol AP2100:WGI210CS_S_LKKM
Changed lines of the file:
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@@
   (page 1 10)
   (paper "A4")
+  (symbol (lib_id "AP2100:WGI210CS_S_LKKM") (at 60.325 73.025 0) (unit 1)
+    (in_bom yes) (on_board yes)
+    (property "Reference" "IC1" (id 0) (at 117.475 86.36 0)
+      (effects (font (size 1.27 1.27)) (justify left))
+    )
+    (property "Value" "WGI210CS_S_LKKM" (id 1) (at 117.475 88.9 0)
+      (effects (font (size 1.27 1.27)) (justify left))
+    )
+    (property "Footprint" "AP2100:QFN50P900X900X100-65N" (id 2) (at 112.395 47.625 0)
+      (effects (font (size 1.27 1.27)) (justify left) hide)
+    )
+    (property "Datasheet" "https://componentsearchengine.com/Datasheets/1/WGI210CS S LKKM.pdf" (id 3) (at 112.395 50.165 0)
+      (effects (font (size 1.27 1.27)) (justify left) hide)
+    )
+    (property "Description" "Ethernet ICs DEVICE CON" (id 4) (at 112.395 52.705 0)
+      (effects (font (size 1.27 1.27)) (justify left) hide)
+    )
+    (property "Height" "1" (id 5) (at 112.395 55.245 0)
+      (effects (font (size 1.27 1.27)) (justify left) hide)
+    )
+    (property "Manufacturer_Name" "Intel" (id 6) (at 112.395 57.785 0)
+      (effects (font (size 1.27 1.27)) (justify left) hide)
+    )
+    (property "Manufacturer_Part_Number" "WGI210CS S LKKM" (id 7) (at 112.395 60.325 0)
+      (effects (font (size 1.27 1.27)) (justify left) hide)
+    )
+    (property "Arrow Part Number" "" (id 8) (at 112.395 62.865 0)
+      (effects (font (size 1.27 1.27)) (justify left) hide)
+    )
+    (property "Arrow Price/Stock" "" (id 9) (at 112.395 65.405 0)
+      (effects (font (size 1.27 1.27)) (justify left) hide)
+    )
+    (property "Mouser Part Number" "607-WGI210CSSLKKM" (id 10) (at 112.395 67.945 0)
+      (effects (font (size 1.27 1.27)) (justify left) hide)
+    )
+    (property "Mouser Price/Stock" "https://www.mouser.co.uk/ProductDetail/Intel/WGI210CS-S-LKKM?qs=d5w0Orft5TqN8mKiqgAr2Q%3D%3D" (id 11) (at 112.395 70.485 0)
+      (effects (font (size 1.27 1.27)) (justify left) hide)
+    )
+  )
 )
