File: AP2100-power-proto/AP2100-power-proto.kicad_pcb (KiCad board)
At the start: 2 copper layers, 150 x 160 mm, 386 parts, among them IC1 MAX17632BATE+, IC2 PM8805TR, IC3 PM8804TR, IC4 MIC2774N-29YM5-TR, J1 0826-1X1T-GH-F, J2 Barrel_Jack, J3 RJ45, Q1 BSC190N15NS3GATMA1, Q2 PBSS4240T, Q3 PBSS4240T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

Commit message: Cleanups per ST Micro's review. Add old and old-old kinda by accident
Parts:
- added T1: RN102-2-02-1M1, Inductor_THT:Choke_Schaffner_RN102-04-14.0x14.0mm, F.Cu at (18.8, 123.0)
- added T2: RN102-2-02-1M1, Inductor_THT:Choke_Schaffner_RN102-04-14.0x14.0mm, F.Cu at (3.89, 123.0)
- C104: value 10nF -> 1.5nF
- C116: value 100uF -> 1nF; footprint Capacitor_SMD:CP_Elec_6.3x5.9 -> Capacitor_SMD:C_0805_2012Metric
- C117: value 100uF -> 47uF; footprint Capacitor_SMD:CP_Elec_6.3x5.9 -> Capacitor_SMD:C_1210_3225Metric
- C78: value 1nF -> 33nF; moved to B.Cu
- C79: value 33nF -> 1nF; moved to B.Cu
- C80, C85, FB1, FB2, R19: moved to B.Cu
- R24: value 10K -> 10; footprint Resistor_SMD:R_0603_1608Metric -> Resistor_SMD:R_0805_2012Metric
- TR1: value POE72PR-12ED -> POE120PL-12L; footprint Scott:Transformer_Coilcraft_POE72PR -> Scott:Transformer_Coilcraft_POE120PL
- moved C108 129.9 mm to (21.0, 93.2)
- moved C87 128.4 mm to (95.1, 164.8)
- moved LED2 128.4 mm to (76.0, 183.5)
- moved LED3 128.4 mm to (82.2, 176.8)
- moved D8 121.8 mm to (12.3, 92.5), turned to -90 degrees
- moved C83 117.6 mm to (-30.2, 84.5)
- moved C84 117.5 mm to (-35.6, 93.3)
- moved FB4 117.4 mm to (-30.2, 81.6), turned to 0 degrees
- moved R19 115.8 mm to (13.1, 96.7)
- moved R28 114.4 mm to (20.9, 91.4), turned to 180 degrees
- moved FB3 112.9 mm to (-24.5, 77.3), turned to 0 degrees
- moved LED1 107.6 mm to (82.4, 155.6)
- moved D9 102.6 mm to (87.7, 137.1)
- moved D10 101.1 mm to (87.8, 143.6)
- moved TR1 97.4 mm to (111.6, 57.3)
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Connections:
- C116 pad 1: /12V -> Net-(C116-Pad1)
- C116 pad 2: GND -> GNDA
- C79 pad 1: Net-(C78-Pad1) -> Net-(C79-Pad1)
- C79 pad 2: Net-(C78-Pad2) -> Net-(C79-Pad2)
- C84 pad 1: Net-(C83-Pad1) -> Net-(C84-Pad1)
- C84 pad 2: Net-(C83-Pad2) -> Net-(C84-Pad2)
- D1 pad 1: Net-(C78-Pad1) -> Net-(C79-Pad1)
- D1 pad 2: Net-(C78-Pad2) -> Net-(C79-Pad2)
- D2 pad 2: Net-(C78-Pad1) -> Net-(C79-Pad1)
- D5 pad 2: Net-(C78-Pad2) -> Net-(C79-Pad2)
- FB3 pad 1: Net-(C83-Pad1) -> Net-(C84-Pad1)
- FB4 pad 1: Net-(C83-Pad2) -> Net-(C84-Pad2)
- IC2 pad 10: Net-(IC2-Pad10) -> GNDPWR
- IC2 pad 3: /PoE Power/STBY -> GNDPWR
- IC3 pad 8: GNDPWR -> Net-(C116-Pad1)
- J1 pad 13: Net-(C78-Pad1) -> Net-(C79-Pad1)
- J1 pad 14: Net-(C78-Pad2) -> Net-(C79-Pad2)
- R24 pad 1: Net-(IC2-Pad10) -> Net-(C116-Pad1)
- R24 pad 2: GNDPWR -> Net-(C100-Pad1)
- R28 pad 1: GNDPWR -> /PoE Power/VB
- TR1 pad 1: Net-(C100-Pad1) -> GNDPWR
- TR1 pad 2: (no net) -> Net-(C120-Pad2)
- TR1 pad 4: Net-(D11-Pad2) -> Net-(TR1-Pad4)
- TR1 pad 5: GNDPWR -> Net-(C100-Pad1)
- TR1 pad 6: Net-(C109-Pad1) -> Net-(D11-Pad2)
- TR1 pad 8: (no net) -> Net-(C109-Pad1)
Routing:
- net Net-(C78-Pad2): track 31.5 -> 0.00 mm
- net Net-(C79-Pad1): track 0.00 -> 31.3 mm, vias 0 -> 6
- net Net-(C78-Pad1): track 25.4 -> 0.00 mm
- net Net-(C79-Pad2): track 0.00 -> 13.8 mm, vias 0 -> 6
- net Net-(C83-Pad2): track 40.1 -> 28.0 mm, vias 0 -> 3
- net Net-(C83-Pad1): track 32.5 -> 43.7 mm, vias 0 -> 3
- net /PoE Power/PGD: track 0.00 -> 6.59 mm
- net Net-(C89-Pad1): track 0.00 -> 4.53 mm
- net Net-(C104-Pad2): track 0.00 -> 2.77 mm
- net Net-(IC2-Pad31): track 0.00 -> 1.91 mm, vias 0 -> 1
- net Net-(C85-Pad2): vias 0 -> 6
- net Net-(C85-Pad1): vias 0 -> 6
- net Net-(C80-Pad2): vias 0 -> 6
- net Net-(C80-Pad1): vias 0 -> 6
- added copper zone on F.Cu, net /PoE Power/VDC
- added copper zone on B.Cu, net Net-(C78-Pad1)
- added copper zone on B.Cu, net Net-(C78-Pad2)
- added copper zone on B.Cu, net Net-(C79-Pad1)
- added copper zone on F.Cu, net Net-(C79-Pad1)
- added copper zone on B.Cu, net Net-(C79-Pad2)
- added copper zone on F.Cu, net Net-(C79-Pad2)
- added copper zone on B.Cu, net Net-(C80-Pad1)
- added copper zone on F.Cu, net Net-(C80-Pad1)
- added copper zone on B.Cu, net Net-(C80-Pad2)
- added copper zone on F.Cu, net Net-(C80-Pad2)
- added copper zone on B.Cu, net Net-(C83-Pad1)
- added copper zone on B.Cu, net Net-(C83-Pad2)
- added copper zone on B.Cu, net Net-(C85-Pad1)
- added copper zone on B.Cu, net Net-(C85-Pad2)

Commit message: Layout of PoE up to VDC - going to rework though
Parts:
- removed C103, C93: 2.2nF, Capacitor_SMD:C_1812_4532Metric
- C104, C83, C84, C87, FB3, FB4, R20, R21, R22, R23, R26: moved to B.Cu
- moved C113 203.2 mm to (73.5, 50.1)
- moved Q5 195.1 mm to (81.6, 38.3)
- moved Q1 177.3 mm to (30.1, 32.4)
- moved Q3 168.5 mm to (93.1, 37.9)
- moved Q2 168.5 mm to (85.0, 45.3)
- moved C101 157.8 mm to (25.8, 69.1), turned to 180 degrees
- moved C100 155.6 mm to (25.8, 65.7), turned to 180 degrees
- moved C86 150.3 mm to (77.2, 140.1), turned to 90 degrees
- moved Q4 147.9 mm to (28.6, 26.1), turned to 90 degrees
- moved C95 144.6 mm to (48.3, 90.1), turned to -90 degrees
- moved C82 140.4 mm to (75.9, 140.1), turned to 90 degrees
- moved C97 139.6 mm to (41.8, 92.0)
- moved C94 133.3 mm to (85.0, 90.4)
- moved C81 130.1 mm to (74.7, 140.1), turned to 90 degrees
- moved D9 126.4 mm to (-10.8, 57.8)
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Connections:
- C81 pad 1: GND -> Earth
- C82 pad 1: GND -> Earth
- C86 pad 1: GND -> Earth
- C88 pad 1: GND -> Earth
- D2 pad 1: GND -> Earth
- D3 pad 1: GND -> Earth
- D5 pad 1: GND -> Earth
- D6 pad 1: GND -> Earth
- J1 pad 21: GND -> Earth
- J1 pad 22: GND -> Earth
- R21 pad 2: GND -> Earth
Routing:
- net Net-(C90-Pad1): track 0.00 -> 25.3 mm
- net Net-(C81-Pad2): track 0.00 -> 21.4 mm
- net Net-(C82-Pad2): track 0.00 -> 18.7 mm
- net /PoE Power/VB: track 0.00 -> 17.8 mm, vias 0 -> 2
- net Net-(C88-Pad2): track 0.00 -> 12.5 mm
- net Net-(IC2-Pad9): track 0.00 -> 11.5 mm, vias 0 -> 1
- net Net-(IC2-Pad8): track 0.00 -> 10.0 mm, vias 0 -> 1
- net Net-(C86-Pad2): track 0.00 -> 9.82 mm
- net Net-(IC2-Pad7): track 0.00 -> 9.67 mm, vias 0 -> 1
- net /PoE Power/PGD: track 6.59 -> 0.00 mm
- net Net-(IC2-Pad5): track 0.00 -> 4.84 mm
- net Net-(C83-Pad1): track 43.7 -> 46.3 mm
- net Net-(IC2-Pad4): track 0.00 -> 2.62 mm
- net Net-(LED1-Pad1): track 0.00 -> 2.52 mm, vias 0 -> 1
- net Net-(LED3-Pad1): track 0.00 -> 2.52 mm, vias 0 -> 1
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- added copper zone on B.Cu, net /PoE Power/VOB
- added copper zone on F.Cu, net /PoE Power/VOB
- added copper zone on B.Cu, net Earth
- added copper zone on F.Cu, net Earth
- added copper zone on B.Cu, net GNDPWR
- added copper zone on F.Cu, net GNDPWR
- added copper zone on B.Cu, net Net-(C84-Pad1)
- added copper zone on B.Cu, net Net-(C84-Pad2)
- added copper zone on F.Cu, net Net-(D7-Pad2)

Commit message: More PoE layout
Parts:
- C104, C78, C79, C80, C83, C84, C85, C87, FB1, FB2, FB3, FB4, R19, R26: moved to F.Cu
- C106, C107, C119, C121, C96, C97, C98, D11, D12, D18, L9, R24: moved to B.Cu
- moved C126 203.7 mm to (94.0, 47.3)
- moved C120 148.9 mm to (33.3, 78.3), turned to 180 degrees
- moved C118 145.2 mm to (46.1, 84.6), turned to 180 degrees
- moved C119 130.6 mm to (32.7, 85.2), turned to -90 degrees
- moved D12 124.5 mm to (25.9, 90.5), turned to -90 degrees
- moved R50 124.1 mm to (31.6, 90.4)
- moved R35 121.4 mm to (46.1, 81.4), turned to 180 degrees
- moved R36 113.5 mm to (37.3, 86.7), turned to -90 degrees
- moved D18 109.3 mm to (46.6, 77.9)
- moved L9 108.7 mm to (24.8, 86.1), turned to -90 degrees
- moved C107 104.9 mm to (30.9, 85.2), turned to -90 degrees
- moved D13 97.0 mm to (35.3, 86.7), turned to -90 degrees
- moved R28 93.3 mm to (39.1, 78.3), turned to -90 degrees
- moved C108 93.1 mm to (41.0, 78.2), turned to 90 degrees
- moved L10 92.2 mm to (14.1, 55.9), turned to 180 degrees
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Connections:
- net Net-(C80-Pad1) renamed /PoE Power/IN_12
- net Net-(C80-Pad2) renamed /PoE Power/IN_36
- net Net-(C85-Pad1) renamed /PoE Power/IN_45
- net Net-(C85-Pad2) renamed /PoE Power/IN_78
- D8 pad 1: /PoE Power/VDC -> /PoE Power/VOB
- D8 pad 2: /PoE Power/VOB -> /PoE Power/VDC
Routing:
- net Net-(D7-Pad2): track 1.80 -> 74.3 mm, vias 0 -> 1
- net Net-(IC2-Pad7): track 9.67 -> 64.7 mm
- net Net-(IC2-Pad8): track 10.0 -> 64.5 mm
- net Net-(IC2-Pad9): track 11.5 -> 63.0 mm
- net Net-(C83-Pad1): track 46.3 -> 0.00 mm, vias 3 -> 0
- net Net-(C79-Pad1): track 29.9 -> 0.00 mm, vias 3 -> 0
- net Net-(C83-Pad2): track 27.4 -> 0.00 mm, vias 3 -> 0
- net Net-(C90-Pad1): track 25.3 -> 6.63 mm
- net Net-(C106-Pad1): track 0.00 -> 14.8 mm, vias 0 -> 1
- net Net-(C79-Pad2): track 11.9 -> 0.00 mm, vias 3 -> 0
- net Net-(C121-Pad2): track 0.00 -> 10.7 mm, vias 0 -> 1
- net Net-(C124-Pad2): track 0.00 -> 10.7 mm
- net /PoE Power/VB: track 17.8 -> 7.43 mm, vias 2 -> 0
- net GNDPWR: track 0.00 -> 9.82 mm, vias 17 -> 14
- net Net-(D13-Pad2): track 0.00 -> 6.58 mm
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- added copper zone on In3.Cu, net /PoE Power/VDC
- added copper zone on In4.Cu, net /PoE Power/VDC
- added copper zone on F.Cu, net Net-(C100-Pad1)
- added copper zone on F.Cu, net Net-(C78-Pad1)
- added copper zone on F.Cu, net Net-(C78-Pad2)
- added copper zone on F.Cu, net Net-(C84-Pad1)
- added copper zone on F.Cu, net Net-(C84-Pad2)
- added copper zone on F.Cu, net Net-(Q1-Pad1)
- removed copper zone on B.Cu, net /PoE Power/IN_12
- removed copper zone on B.Cu, net /PoE Power/IN_36
- removed copper zone on B.Cu, net /PoE Power/IN_45
- removed copper zone on B.Cu, net /PoE Power/IN_78
- removed copper zone on B.Cu, net /PoE Power/VOB
- removed copper zone on B.Cu, net Earth
- removed copper zone on F.Cu, net Earth
- removed copper zone on B.Cu, net GNDPWR
- removed copper zone on B.Cu, net Net-(C78-Pad1)
- removed copper zone on B.Cu, net Net-(C78-Pad2)
- removed copper zone on B.Cu, net Net-(C79-Pad1)
- removed copper zone on B.Cu, net Net-(C79-Pad2)
- removed copper zone on B.Cu, net Net-(C83-Pad1)
- removed copper zone on B.Cu, net Net-(C83-Pad2)
- removed copper zone on B.Cu, net Net-(C84-Pad1)
- removed copper zone on B.Cu, net Net-(C84-Pad2)
Other:
- copper layers 2 -> 6
