File: AP3000/AP3000.kicad_pcb (KiCad board)
At the start: 4 copper layers, 186 x 226 mm, 186 parts, among them IC2 TPS23751PWPR, J1 Conn_01x03, J10 Camera 1 Power, J11 Barrel_Jack, J12 Bus_PCI_Express_Mini, J2 Conn_02x07_Odd_Even, J3 Conn_01x03, J4 Camera 0, J5 Camera 0 Power, J6 Camera 1, J7 YJ-USB-AF_SMT-01, J8 THD-20-R, J9 0826-1X1T-GH-F, Q1 BSC520N15NS3 G, Q2 MMBT2907ALT1G, Q3 MMBT3906LT1G, U1 TPD4EUSB30, U10 SIR422DP-T1-GE3, U12 TCMT1107, U13 TLV431ACDBZR, U14 74LVC1G07SE-7, U16 TPS54A24RTWR, U17 TPS628640AYCGR, U2 TPD4EUSB30, U3 ATECC608A-MAHDA, U4 TPD4EUSB30, U5 74LVC1G07SE-7, U7 AP22653W6, U8 PCF85063AT/AAZ, U9 74LVC1G07SE-7, Y2 X32K768S301

Commit message: AP3000: Fixup PartsBoxID linkage and placed first order Working on a design for a 5 GHz panel antenna array for a point-to-point replacement
Parts:
- moved J8 2.85 mm to (152.3, 82.2)
Connections:
- H1 pad 1: Net-(H1-Pad1) -> GND
- H10 pad 1: Net-(H10-Pad1) -> GND
- H11 pad 1: Net-(H11-Pad1) -> GND
- H12 pad 1: Net-(H12-Pad1) -> GND
- H2 pad 1: Net-(H2-Pad1) -> GND
- H3 pad 1: Net-(H3-Pad1) -> GNDPWR
- H4 pad 1: Net-(H4-Pad1) -> GNDPWR
- H5 pad 1: Net-(H5-Pad1) -> GNDPWR
- H6 pad 1: Net-(H6-Pad1) -> GND
- H7 pad 1: Net-(H7-Pad1) -> GND
- H8 pad 1: Net-(H8-Pad1) -> GNDPWR
- H9 pad 1: Net-(H9-Pad1) -> GNDPWR
Routing:
- net /CM4_GPIO ( Ethernet, GPIO, SDCARD)/GPIO14: track 34.6 -> 59.4 mm
- net /CM4_GPIO ( Ethernet, GPIO, SDCARD)/GPIO15: track 34.7 -> 59.4 mm
- net /CM4_GPIO ( Ethernet, GPIO, SDCARD)/GPIO2: track 38.0 -> 61.6 mm
- net /CM4_GPIO ( Ethernet, GPIO, SDCARD)/GPIO18: track 35.0 -> 58.3 mm
- net /CM4_GPIO ( Ethernet, GPIO, SDCARD)/GPIO3: track 37.7 -> 60.5 mm
- net /CM4_GPIO ( Ethernet, GPIO, SDCARD)/GPIO4: track 37.7 -> 59.5 mm
- net /CM4_GPIO ( Ethernet, GPIO, SDCARD)/GPIO17: track 37.2 -> 57.2 mm
- net /ID_SC: track 113.5 -> 131.3 mm
- net /CM4_GPIO ( Ethernet, GPIO, SDCARD)/GPIO23: track 37.7 -> 54.7 mm
- net /CM4_GPIO ( Ethernet, GPIO, SDCARD)/GPIO27: track 38.7 -> 55.4 mm
- net /CM4_GPIO ( Ethernet, GPIO, SDCARD)/GPIO24: track 39.4 -> 53.6 mm
- net /CM4_GPIO ( Ethernet, GPIO, SDCARD)/GPIO22: track 40.1 -> 54.2 mm
- net /SCL0: track 118.3 -> 131.2 mm
- net /CM4_GPIO ( Ethernet, GPIO, SDCARD)/GPIO20: track 54.8 -> 66.7 mm
- net /CM4_GPIO ( Ethernet, GPIO, SDCARD)/GPIO21: track 57.4 -> 69.0 mm
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Other:
- board text added: "AP3000-CAM V4 Copyright 2020 ISis ImageStream Internet Solutions, Inc."
- board text removed: "AP3000 V3 Copyright 2020 ISis ImageStream Internet Solutions, Inc."
