File: AP3000/CM4_GPIO.kicad_sch (KiCad schematic)
At the start: 21 parts, among them J1 Conn_01x03, J2 Conn_02x07_Odd_Even, J3 Conn_01x03, J8 THD-20-R, J9 0826-1X1T-GH-F, U1 TPD4EUSB30, U2 TPD4EUSB30, U5 74LVC1G07SE-7, U9 74LVC1G07SE-7

Commit message: Route all the high speed lines and most gpio
Connections:
- no-connect marks 13 -> 15
Changed lines of the file:
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@@
   (junction (at 269.494 63.5) (diameter 1.016) (color 0 0 0 0))
   (junction (at 269.494 68.58) (diameter 1.016) (color 0 0 0 0))
+  (no_connect (at 133.985 144.78))
+  (no_connect (at 147.955 104.14))
+  (no_connect (at 208.915 111.76))
+  (no_connect (at 147.955 109.22))
+  (no_connect (at 147.955 99.06))
+  (no_connect (at 208.915 96.52))
   (no_connect (at 147.955 127))
+  (no_connect (at 147.955 124.46))
+  (no_connect (at 208.915 99.06))
   (no_connect (at 208.915 106.68))
-  (no_connect (at 208.915 99.06))
-  (no_connect (at 208.915 111.76))
-  (no_connect (at 147.955 99.06))
+  (no_connect (at 208.915 43.18))
+  (no_connect (at 208.915 104.14))
+  (no_connect (at 208.915 91.44))
   (no_connect (at 147.955 106.68))
-  (no_connect (at 147.955 109.22))
-  (no_connect (at 208.915 96.52))
-  (no_connect (at 208.915 43.18))
-  (no_connect (at 147.955 124.46))
-  (no_connect (at 208.915 104.14))
-  (no_connect (at 147.955 104.14))
-  (no_connect (at 208.915 91.44))
+  (no_connect (at 59.69 185.42))
   (wire (pts (xy 15.24 169.545) (xy 29.21 169.545))
     (stroke (width 0) (type solid) (color 0 0 0 0))

Commit message: Forgot to add PCB cutout resulting in some components being moved
Parts:
- removed R4: DNS 0, Resistor_SMD:R_0402_1005Metric, symbol Device:R
- removed R5: 0R, Resistor_SMD:R_0402_1005Metric, symbol Device:R
- removed TP3, TP5: TestPoint, TestPoint:TestPoint_Pad_2.0x2.0mm, symbol Connector:TestPoint
Connections:
- net GPIO_VREF is gone; now on net +3.3v: Module1.78 (GPIO_VREF(1.8v/3.3v_Input))
Changed lines of the file:
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@@
   (junction (at 146.685 142.24) (diameter 1.016) (color 0 0 0 0))
   (junction (at 147.955 129.54) (diameter 1.016) (color 0 0 0 0))
-  (junction (at 160.02 165.227) (diameter 1.016) (color 0 0 0 0))
   (junction (at 208.915 116.84) (diameter 1.016) (color 0 0 0 0))
   (junction (at 208.915 119.38) (diameter 1.016) (color 0 0 0 0))
@@
   (junction (at 210.185 109.22) (diameter 1.016) (color 0 0 0 0))
   (junction (at 210.185 133.35) (diameter 1.016) (color 0 0 0 0))
-  (junction (at 225.679 33.02) (diameter 1.016) (color 0 0 0 0))
   (junction (at 252.984 27.94) (diameter 1.016) (color 0 0 0 0))
   (junction (at 254.254 58.42) (diameter 1.016) (color 0 0 0 0))
   (junction (at 254.254 76.2) (diameter 1.016) (color 0 0 0 0))
   (junction (at 255.524 45.72) (diameter 1.016) (color 0 0 0 0))
-  (junction (at 263.144 95.25) (diameter 1.016) (color 0 0 0 0))
   (junction (at 269.494 27.94) (diameter 1.016) (color 0 0 0 0))
   (junction (at 269.494 43.18) (diameter 1.016) (color 0 0 0 0))
@@
   (junction (at 269.494 63.5) (diameter 1.016) (color 0 0 0 0))
   (junction (at 269.494 68.58) (diameter 1.016) (color 0 0 0 0))
+  (no_connect (at 208.915 43.18))
+  (no_connect (at 147.955 124.46))
+  (no_connect (at 208.915 111.76))
   (no_connect (at 133.985 144.78))
+  (no_connect (at 147.955 127))
+  (no_connect (at 147.955 109.22))
+  (no_connect (at 208.915 99.06))
+  (no_connect (at 59.69 185.42))
+  (no_connect (at 208.915 104.14))
   (no_connect (at 147.955 104.14))
-  (no_connect (at 208.915 111.76))
-  (no_connect (at 147.955 109.22))
+  (no_connect (at 208.915 96.52))
+  (no_connect (at 147.955 106.68))
+  (no_connect (at 208.915 106.68))
+  (no_connect (at 208.915 91.44))
   (no_connect (at 147.955 99.06))
-  (no_connect (at 208.915 96.52))
-  (no_connect (at 147.955 127))
-  (no_connect (at 147.955 124.46))
-  (no_connect (at 208.915 99.06))
-  (no_connect (at 208.915 106.68))
-  (no_connect (at 208.915 43.18))
-  (no_connect (at 208.915 104.14))
-  (no_connect (at 208.915 91.44))
-  (no_connect (at 147.955 106.68))
-  (no_connect (at 59.69 185.42))
   (wire (pts (xy 15.24 169.545) (xy 29.21 169.545))
     (stroke (width 0) (type solid) (color 0 0 0 0))
@@
     (stroke (width 0) (type solid) (color 0 0 0 0))
   )
-  (wire (pts (xy 155.0162 165.227) (xy 160.02 165.227))
-    (stroke (width 0) (type solid) (color 0 0 0 0))
-  )
   (wire (pts (xy 160.02 156.21) (xy 156.21 156.21))
     (stroke (width 0) (type solid) (color 0 0 0 0))
@@
     (stroke (width 0) (type solid) (color 0 0 0 0))
   )
-  (wire (pts (xy 160.02 165.1) (xy 160.02 165.227))
-    (stroke (width 0) (type solid) (color 0 0 0 0))
-  )
-  (wire (pts (xy 160.02 165.227) (xy 160.02 166.37))
+  (wire (pts (xy 160.02 165.1) (xy 160.02 166.37))
     (stroke (width 0) (type solid) (color 0 0 0 0))
   )
@@
     (stroke (width 0) (type solid) (color 0 0 0 0))
   )
-  (wire (pts (xy 225.679 33.02) (xy 225.679 30.48))
-    (stroke (width 0) (type solid) (color 0 0 0 0))
-  )
-  (wire (pts (xy 225.679 35.56) (xy 225.679 33.02))
+  (wire (pts (xy 225.679 30.48) (xy 225.679 35.56))
     (stroke (width 0) (type solid) (color 0 0 0 0))
   )
@@
     (stroke (width 0) (type solid) (color 0 0 0 0))
   )
-  (wire (pts (xy 232.029 33.02) (xy 225.679 33.02))
-    (stroke (width 0) (type solid) (color 0 0 0 0))
-  )
   (wire (pts (xy 244.094 30.48) (xy 255.524 30.48))
     (stroke (width 0) (type solid) (color 0 0 0 0))
@@
     (stroke (width 0) (type solid) (color 0 0 0 0))
   )
-  (wire (pts (xy 246.634 95.25) (xy 255.524 95.25))
-    (stroke (width 0) (type solid) (color 0 0 0 0))
-  )
-  (wire (pts (xy 246.634 99.06) (xy 255.524 99.06))
+  (wire (pts (xy 246.634 95.25) (xy 269.875 95.25))
     (stroke (width 0) (type solid) (color 0 0 0 0))
   )
@@
   )
   (wire (pts (xy 258.064 45.72) (xy 255.524 45.72))
-    (stroke (width 0) (type solid) (color 0 0 0 0))
-  )
-  (wire (pts (xy 263.144 95.25) (xy 263.144 99.06))
-    (stroke (width 0) (type solid) (color 0 0 0 0))
-  )
-  (wire (pts (xy 263.144 95.25) (xy 269.875 95.25))
     (stroke (width 0) (type solid) (color 0 0 0 0))
   )
@@
     (effects (font (size 1.27 1.27)) (justify right bottom))
   )
-  (label "+1.8v" (at 251.714 99.06 180)
-    (effects (font (size 1.27 1.27)) (justify right bottom))
-  )
   (label "RUN_PG" (at 256.921 134.62 180)
     (effects (font (size 1.27 1.27)) (justify right bottom))
@@
   (hierarchical_label "GLOBAL_EN" (shape input) (at 225.425 144.78 0)
     (effects (font (size 1.27 1.27)) (justify left))
-  )
-  (hierarchical_label "GPIO_VREF" (shape output) (at 269.875 95.25 0)
-    (effects (font (size 1.27 1.27)) (justify left))
-  )
-  (symbol (lib_id "Connector:TestPoint") (at 155.0162 165.227 90) (unit 1)
-    (in_bom yes) (on_board yes)
-    (property "Reference" "TP5" (id 0) (at 152.654 162.56 90)
-      (effects (font (size 1.27 1.27)) (justify left))
-    )
-    (property "Value" "TestPoint" (id 1) (at 157.734 167.64 90)
-      (effects (font (size 1.27 1.27)) (justify left))
-    )
-    (property "Footprint" "TestPoint:TestPoint_Pad_2.0x2.0mm" (id 2) (at 155.0162 160.147 0)
-      (effects (font (size 1.27 1.27)) hide)
-    )
-    (property "Datasheet" "" (id 3) (at 155.0162 160.147 0)
-      (effects (font (size 1.27 1.27)) hide)
-    )
-    (property "Field4" "nf" (id 4) (at 155.0162 165.227 0)
-      (effects (font (size 1.27 1.27)) hide)
-    )
-    (property "Field5" "nf" (id 5) (at 155.0162 165.227 0)
-      (effects (font (size 1.27 1.27)) hide)
-    )
-    (property "Field6" "nf" (id 6) (at 155.0162 165.227 0)
-      (effects (font (size 1.27 1.27)) hide)
-    )
-    (property "Field7" "nf" (id 7) (at 155.0162 165.227 0)
-      (effects (font (size 1.27 1.27)) hide)
-    )
-  )
-  (symbol (lib_id "Connector:TestPoint") (at 232.029 33.02 270) (unit 1)
-    (in_bom yes) (on_board yes)
-    (property "Reference" "TP3" (id 0) (at 233.299 36.83 90)
-      (effects (font (size 1.27 1.27)) (justify left))
-    )
-    (property "Value" "TestPoint" (id 1) (at 230.759 34.925 90)
-      (effects (font (size 1.27 1.27)) (justify left))
-    )
-    (property "Footprint" "TestPoint:TestPoint_Pad_2.0x2.0mm" (id 2) (at 232.029 38.1 0)
-      (effects (font (size 1.27 1.27)) hide)
-    )
-    (property "Datasheet" "" (id 3) (at 232.029 38.1 0)
-      (effects (font (size 1.27 1.27)) hide)
-    )
-    (property "Field4" "nf" (id 4) (at 232.029 33.02 0)
-      (effects (font (size 1.27 1.27)) hide)
-    )
-    (property "Field5" "nf" (id 5) (at 232.029 33.02 0)
-      (effects (font (size 1.27 1.27)) hide)
-    )
-    (property "Field6" "nf" (id 6) (at 232.029 33.02 0)
-      (effects (font (size 1.27 1.27)) hide)
-    )
-    (property "Field7" "nf" (id 7) (at 232.029 33.02 0)
-      (effects (font (size 1.27 1.27)) hide)
-    )
   )
   (symbol (lib_id "power:GND") (at 19.05 57.785 0) (unit 1)
@@
       (effects (font (size 1.27 1.27)) hide)
     )
-  )
-  (symbol (lib_id "Device:R") (at 259.334 95.25 90) (unit 1)
-    (in_bom yes) (on_board yes)
-    (property "Reference" "R5" (id 0) (at 258.064 92.71 90)
-      (effects (font (size 1.27 1.27)) (justify left))
-    )
-    (property "Value" "0R" (id 1) (at 263.144 92.71 90)
-      (effects (font (size 1.27 1.27)) (justify left))
-    )
-    (property "Footprint" "Resistor_SMD:R_0402_1005Metric" (id 2) (at 259.334 97.028 90)
-      (effects (font (size 1.27 1.27)) hide)
-    )
-    (property "Datasheet" "https://fscdn.rohm.com/en/products/databook/datasheet/passive/resistor/chip_resistor/mcr-e.pdf" (id 3) (at 259.334 95.25 0)
-      (effects (font (size 1.27 1.27)) hide)
-    )
-    (property "Field4" "Farnell" (id 4) (at 259.334 95.25 0)
-      (effects (font (size 1.27 1.27)) hide)
-    )
-    (property "Field5" "9233750" (id 5) (at 259.334 95.25 0)
-      (effects (font (size 1.27 1.27)) hide)
-    )
-    (property "Field7" "Rohm" (id 6) (at 259.334 95.25 0)
-      (effects (font (size 1.27 1.27)) hide)
-    )
-    (property "Field6" "MCR10EZPJ000" (id 7) (at 259.334 95.25 0)
-      (effects (font (size 1.27 1.27)) hide)
-    )
-    (property "Part Description" "Resistor 0R M2012 5% " (id 8) (at 259.334 95.25 0)
-      (effects (font (size 1.27 1.27)) hide)
-    )
-    (property "Field8" "121629591" (id 9) (at 259.334 95.25 0)
-      (effects (font (size 1.27 1.27)) hide)
-    )
-  )
-  (symbol (lib_id "Device:R") (at 259.334 99.06 90) (unit 1)
-    (in_bom yes) (on_board yes)
-    (property "Reference" "R4" (id 0) (at 258.064 101.6 90)
-      (effects (font (size 1.27 1.27)) (justify left))
-    )
-    (property "Value" "DNS 0" (id 1) (at 265.684 101.6 90)
-      (effects (font (size 1.27 1.27)) (justify left))
-    )
-    (property "Footprint" "Resistor_SMD:R_0402_1005Metric" (id 2) (at 259.334 100.838 90)
-      (effects (font (size 1.27 1.27)) hide)
-    )
-    (property "Datasheet" "https://fscdn.rohm.com/en/products/databook/datasheet/passive/resistor/chip_resistor/mcr-e.pdf" (id 3) (at 259.334 99.06 0)
-      (effects (font (size 1.27 1.27)) hide)
-    )
-    (property "Field4" "nf" (id 4) (at 259.334 99.06 0)
-      (effects (font (size 1.27 1.27)) hide)
-    )
-    (property "Field5" "nf" (id 5) (at 259.334 99.06 0)
-      (effects (font (size 1.27 1.27)) hide)
-    )
-    (property "Field6" "nf" (id 6) (at 259.334 99.06 0)
-      (effects (font (size 1.27 1.27)) hide)
-    )

Commit message: Almost done routing!
Connections:
- net CAM_GPIO: no longer names the net of Module1.97 (Camera_GPIO)
- no-connect marks 15 -> 16
Changed lines of the file:
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@@
   (junction (at 269.494 63.5) (diameter 1.016) (color 0 0 0 0))
   (junction (at 269.494 68.58) (diameter 1.016) (color 0 0 0 0))
-  (no_connect (at 208.915 106.68))
-  (no_connect (at 147.955 124.46))
   (no_connect (at 208.915 96.52))
-  (no_connect (at 208.915 104.14))
-  (no_connect (at 208.915 111.76))
-  (no_connect (at 59.69 185.42))
   (no_connect (at 147.955 106.68))
-  (no_connect (at 133.985 144.78))
-  (no_connect (at 147.955 104.14))
+  (no_connect (at 147.955 109.22))
   (no_connect (at 147.955 99.06))
   (no_connect (at 208.915 43.18))
   (no_connect (at 208.915 91.44))
+  (no_connect (at 59.69 185.42))
+  (no_connect (at 133.985 144.78))
+  (no_connect (at 208.915 111.76))
+  (no_connect (at 208.915 142.24))
+  (no_connect (at 147.955 124.46))
   (no_connect (at 208.915 99.06))
-  (no_connect (at 147.955 109.22))
   (no_connect (at 147.955 127))
+  (no_connect (at 208.915 104.14))
+  (no_connect (at 208.915 106.68))
+  (no_connect (at 147.955 104.14))
   (wire (pts (xy 15.24 169.545) (xy 29.21 169.545))
     (stroke (width 0) (type solid) (color 0 0 0 0))
@@
   )
   (wire (pts (xy 208.915 139.7) (xy 222.885 139.7))
-    (stroke (width 0) (type solid) (color 0 0 0 0))
-  )
-  (wire (pts (xy 208.915 142.24) (xy 225.425 142.24))
     (stroke (width 0) (type solid) (color 0 0 0 0))
   )
@@
     (effects (font (size 1.27 1.27)) (justify left))
   )
-  (hierarchical_label "CAM_GPIO" (shape output) (at 225.425 142.24 0)
-    (effects (font (size 1.27 1.27)) (justify left))
-  )

Commit message: Finished routing board.
Parts:
- added C45: .1uF, Capacitor_SMD:C_0402_1005Metric, symbol Device:C_Small
- added U3: ATECC608A-MAHDA, Package_DFN_QFN:DFN-8-1EP_3x2mm_P0.5mm_EP1.3x1.5mm, symbol Security:ATECC608A-MAHDA
Connections:
- net +3.3v: now also C45.1, U3.8 (VCC)
- net GND: now also C45.2, U3.4 (GND), U3.9 (EP); no longer J9.21 (SHIELD), J9.22 (SHIELD)
- net SCL0: now also U3.6 (SCL)
- net SDA0: now also U3.5 (SDA)
- new net GNDPWR: J9.21 (SHIELD), J9.22 (SHIELD)
Other:
- note added: "Crypto / Key Storage"
- note added: "Note: I2C Address: 0x60"
Changed lines of the file:
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@@
   (junction (at 19.05 57.15) (diameter 1.016) (color 0 0 0 0))
   (junction (at 84.455 39.37) (diameter 1.016) (color 0 0 0 0))
+  (junction (at 90.805 146.05) (diameter 0.9144) (color 0 0 0 0))
+  (junction (at 97.155 127.635) (diameter 0.9144) (color 0 0 0 0))
+  (junction (at 97.155 146.05) (diameter 0.9144) (color 0 0 0 0))
   (junction (at 146.685 27.94) (diameter 1.016) (color 0 0 0 0))
   (junction (at 146.685 35.56) (diameter 1.016) (color 0 0 0 0))
@@
   (junction (at 269.494 63.5) (diameter 1.016) (color 0 0 0 0))
   (junction (at 269.494 68.58) (diameter 1.016) (color 0 0 0 0))
+  (no_connect (at 147.955 127))
+  (no_connect (at 147.955 104.14))
+  (no_connect (at 208.915 111.76))
   (no_connect (at 208.915 96.52))
-  (no_connect (at 147.955 106.68))
   (no_connect (at 147.955 109.22))
+  (no_connect (at 147.955 124.46))
+  (no_connect (at 59.69 185.42))
+  (no_connect (at 133.985 144.78))
+  (no_connect (at 208.915 99.06))
+  (no_connect (at 208.915 142.24))
+  (no_connect (at 208.915 91.44))
   (no_connect (at 147.955 99.06))
   (no_connect (at 208.915 43.18))
-  (no_connect (at 208.915 91.44))
-  (no_connect (at 59.69 185.42))
-  (no_connect (at 133.985 144.78))
-  (no_connect (at 208.915 111.76))
-  (no_connect (at 208.915 142.24))
-  (no_connect (at 147.955 124.46))
-  (no_connect (at 208.915 99.06))
-  (no_connect (at 147.955 127))
+  (no_connect (at 208.915 106.68))
+  (no_connect (at 147.955 106.68))
   (no_connect (at 208.915 104.14))
-  (no_connect (at 208.915 106.68))
-  (no_connect (at 147.955 104.14))
   (wire (pts (xy 15.24 169.545) (xy 29.21 169.545))
     (stroke (width 0) (type solid) (color 0 0 0 0))
@@
     (stroke (width 0) (type solid) (color 0 0 0 0))
   )
+  (wire (pts (xy 69.85 135.255) (xy 80.645 135.255))
+    (stroke (width 0) (type solid) (color 0 0 0 0))
+  )
+  (wire (pts (xy 69.85 140.335) (xy 80.645 140.335))
+    (stroke (width 0) (type solid) (color 0 0 0 0))
+  )
   (wire (pts (xy 72.39 172.72) (xy 90.17 172.72))
     (stroke (width 0) (type solid) (color 0 0 0 0))
@@
     (stroke (width 0) (type solid) (color 0 0 0 0))
   )
+  (wire (pts (xy 88.265 127.635) (xy 88.265 130.175))
+    (stroke (width 0) (type solid) (color 0 0 0 0))
+  )
+  (wire (pts (xy 88.265 145.415) (xy 88.265 146.05))
+    (stroke (width 0) (type solid) (color 0 0 0 0))
+  )
+  (wire (pts (xy 88.265 146.05) (xy 90.805 146.05))
+    (stroke (width 0) (type solid) (color 0 0 0 0))
+  )
+  (wire (pts (xy 90.805 146.05) (xy 90.805 145.415))
+    (stroke (width 0) (type solid) (color 0 0 0 0))
+  )
   (wire (pts (xy 92.075 39.37) (xy 84.455 39.37))
     (stroke (width 0) (type solid) (color 0 0 0 0))
   )
+  (wire (pts (xy 97.155 127.635) (xy 88.265 127.635))
+    (stroke (width 0) (type solid) (color 0 0 0 0))
+  )
+  (wire (pts (xy 97.155 127.635) (xy 97.155 129.54))
+    (stroke (width 0) (type solid) (color 0 0 0 0))
+  )
+  (wire (pts (xy 97.155 134.62) (xy 97.155 146.05))
+    (stroke (width 0) (type solid) (color 0 0 0 0))
+  )
+  (wire (pts (xy 97.155 146.05) (xy 90.805 146.05))
+    (stroke (width 0) (type solid) (color 0 0 0 0))
+  )
+  (wire (pts (xy 97.155 146.05) (xy 97.155 146.685))
+    (stroke (width 0) (type solid) (color 0 0 0 0))
+  )
   (wire (pts (xy 101.6 74.295) (xy 113.03 74.295))
     (stroke (width 0) (type solid) (color 0 0 0 0))
@@
   )
   (wire (pts (xy 102.87 49.53) (xy 91.44 49.53))
+    (stroke (width 0) (type solid) (color 0 0 0 0))
+  )
+  (wire (pts (xy 104.775 127.635) (xy 97.155 127.635))
     (stroke (width 0) (type solid) (color 0 0 0 0))
   )
@@
     (effects (font (size 1.27 1.27)) (justify left bottom))
   )
+  (text "Note: I2C Address: 0x60" (at 63.5 146.685 180)
+    (effects (font (size 1.27 1.27)) (justify right bottom))
+  )
+  (text "Crypto / Key Storage" (at 101.6 125.095 180)
+    (effects (font (size 2.54 2.54)) (justify right bottom))
+  )
   (text "Force RPIBOOT = Jumper Pins 1-2 \n" (at 127.254 184.023 180)
     (effects (font (size 1.27 1.27)) (justify right bottom))
@@
     (effects (font (size 1.27 1.27)) (justify right bottom))
   )
+  (label "SDA0" (at 71.755 135.255 0)
+    (effects (font (size 1.27 1.27)) (justify left bottom))
+  )
+  (label "SCL0" (at 71.755 140.335 0)
+    (effects (font (size 1.27 1.27)) (justify left bottom))
+  )
   (label "E0_TRD1_P" (at 76.2 74.295 180)
     (effects (font (size 1.27 1.27)) (justify right bottom))
@@
     (effects (font (size 1.27 1.27)) (justify left bottom))
   )
+  (label "+3.3v" (at 104.14 127.635 180)
+    (effects (font (size 1.27 1.27)) (justify right bottom))
+  )
   (label "E0_TRD0_N" (at 112.395 74.295 180)
     (effects (font (size 1.27 1.27)) (justify right bottom))
@@
   )
   (label "GPIO2" (at 140.335 91.44 180)
+    (effects (font (size 1.27 1.27)) (justify right bottom))
+  )
+  (label "SCL0" (at 140.335 119.38 180)
+    (effects (font (size 1.27 1.27)) (justify right bottom))
+  )
+  (label "SDA0" (at 140.335 121.92 180)
     (effects (font (size 1.27 1.27)) (justify right bottom))
   )
@@
     (effects (font (size 1.27 1.27)) (justify left))
   )
+  (symbol (lib_id "power:GNDPWR") (at 83.185 57.15 0) (mirror y) (unit 1)
+    (in_bom yes) (on_board yes)
+    (property "Reference" "#PWR0108" (id 0) (at 83.185 63.5 0)
+      (effects (font (size 1.27 1.27)) hide)
+    )
+    (property "Value" "GNDPWR" (id 1) (at 83.185 60.325 0))
+    (property "Footprint" "" (id 2) (at 83.185 57.15 0)
+      (effects (font (size 1.27 1.27)) hide)
+    )
+    (property "Datasheet" "" (id 3) (at 83.185 57.15 0)
+      (effects (font (size 1.27 1.27)) hide)
+    )
+  )
   (symbol (lib_id "power:GND") (at 19.05 57.785 0) (unit 1)
     (in_bom yes) (on_board yes)
@@
     )
   )
-  (symbol (lib_id "power:GND") (at 83.185 57.15 0) (mirror y) (unit 1)
-    (in_bom yes) (on_board yes)
-    (property "Reference" "#PWR0108" (id 0) (at 83.185 63.5 0)
-      (effects (font (size 1.27 1.27)) hide)
-    )
-    (property "Value" "GND" (id 1) (at 83.058 61.5442 0))
-    (property "Footprint" "" (id 2) (at 83.185 57.15 0)
-      (effects (font (size 1.27 1.27)) hide)
-    )
-    (property "Datasheet" "" (id 3) (at 83.185 57.15 0)
-      (effects (font (size 1.27 1.27)) hide)
-    )
-  )
   (symbol (lib_id "power:GND") (at 88.9 89.535 0) (unit 1)
     (in_bom yes) (on_board yes)
@@
     )
     (property "Datasheet" "" (id 3) (at 88.9 89.535 0)
+      (effects (font (size 1.27 1.27)) hide)
+    )
+  )
+  (symbol (lib_id "power:GND") (at 97.155 146.685 0) (unit 1)
+    (in_bom yes) (on_board yes)
+    (property "Reference" "#PWR0125" (id 0) (at 97.155 153.035 0)
+      (effects (font (size 1.27 1.27)) hide)
+    )
+    (property "Value" "GND" (id 1) (at 97.282 151.0792 0))
+    (property "Footprint" "" (id 2) (at 97.155 146.685 0)
+      (effects (font (size 1.27 1.27)) hide)
+    )
+    (property "Datasheet" "" (id 3) (at 97.155 146.685 0)
       (effects (font (size 1.27 1.27)) hide)
     )
@@
     )
   )
+  (symbol (lib_id "Device:C_Small") (at 97.155 132.08 0) (mirror y) (unit 1)
+    (in_bom yes) (on_board yes)
+    (property "Reference" "C45" (id 0) (at 97.5868 130.3274 0)
+      (effects (font (size 1.27 1.27)) (justify right))
+    )
+    (property "Value" ".1uF" (id 1) (at 97.5868 134.112 0)
+      (effects (font (size 1.27 1.27)) (justify right))
+    )
+    (property "Footprint" "Capacitor_SMD:C_0402_1005Metric" (id 2) (at 97.155 132.08 0)
+      (effects (font (size 1.27 1.27)) hide)
+    )
+    (property "Datasheet" "~" (id 3) (at 97.155 132.08 0)
+      (effects (font (size 1.27 1.27)) hide)
+    )
+    (property "PartsBoxID" "0402-.1uF-X5R-25V" (id 4) (at 97.155 132.08 0)
+      (effects (font (size 1.27 1.27)) hide)
+    )
+    (property "MPN" "-" (id 5) (at 201.295 182.245 0)
+      (effects (font (size 1.27 1.27)) hide)
+    )
+    (property "SPR" "-" (id 6) (at 201.295 182.245 0)
+      (effects (font (size 1.27 1.27)) hide)
+    )
+    (property "SPN" "-" (id 7) (at 201.295 182.245 0)
+      (effects (font (size 1.27 1.27)) hide)
+    )
+    (property "SPURL" "-" (id 8) (at 201.295 182.245 0)
+      (effects (font (size 1.27 1.27)) hide)
+    )
+  )
   (symbol (lib_id "Device:LED") (at 160.02 161.29 90) (unit 1)
     (in_bom yes) (on_board yes)
@@
       (effects (font (size 1.27 1.27)) hide)
     )
+  )
+  (symbol (lib_id "Security:ATECC608A-MAHDA") (at 88.265 137.795 0) (mirror y) (unit 1)
+    (in_bom yes) (on_board yes)
+    (property "Reference" "U3" (id 0) (at 83.185 131.445 0)
+      (effects (font (size 1.27 1.27)) (justify right))
+    )
+    (property "Value" "ATECC608A-MAHDA" (id 1) (at 67.945 144.78 0)
+      (effects (font (size 1.27 1.27)) (justify right))
+    )
+    (property "Footprint" "Package_DFN_QFN:DFN-8-1EP_3x2mm_P0.5mm_EP1.3x1.5mm" (id 2) (at 88.265 137.795 0)
+      (effects (font (size 1.27 1.27)) hide)
+    )
+    (property "Datasheet" "http://ww1.microchip.com/downloads/en/DeviceDoc/ATECC608A-CryptoAuthentication-Device-Summary-Data-Sheet-DS40001977B.pdf" (id 3) (at 84.455 131.445 0)
+      (effects (font (size 1.27 1.27)) hide)
+    )
+    (property "PartsBoxID" "ATECC608A-MAHDA-T" (id 4) (at 88.265 137.795 0)
+      (effects (font (size 1.27 1.27)) hide)
+    )
