File: AP3000/CM4_GPIO.kicad_sch (KiCad schematic)
At the start: 19 parts, among them J1 Conn_01x03, J2 Conn_02x07_Odd_Even, J3 Conn_01x03, J8 THD-20-R, J9 0826-1X1T-GH-F, U1 TPD4EUSB30, U2 TPD4EUSB30, U3 ATECC608A-MAHDA, U5 74LVC1G07SE-7, U9 74LVC1G07SE-7

Commit message: AP3000: Fixup PartsBoxID linkage and placed first order Working on a design for a 5 GHz panel antenna array for a point-to-point replacement
Parts:
- C1: value 100n -> 100n 16v; PartsBoxID (none) -> 0402-100nF-X7R-16V
- D1: PartsBoxID (none) -> LTST-S270KRKT
- D2: PartsBoxID (none) -> LTST-S270KGKT
- J8: PartsBoxID (none) -> C124374
- J9: PartsBoxID (none) -> 0826-1X1T-GH-F
- Module1: PartsBoxID (none) -> DF40C-100DS-0.4V(51)
- R1, R10: value 1k -> 1K 1%; PartsBoxID (none) -> 0402-1K-1%
- R2, R3: PartsBoxID (none) -> 0402-470R-1%
- U1, U2: PartsBoxID (none) -> CDDFN10-3324P
- U5, U9: PartsBoxID (none) -> 74LVC1G07SE-7
Changed lines of the file:
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@@
   (junction (at 269.494 63.5) (diameter 1.016) (color 0 0 0 0))
   (junction (at 269.494 68.58) (diameter 1.016) (color 0 0 0 0))
-  (no_connect (at 147.955 127))
-  (no_connect (at 147.955 104.14))
+  (no_connect (at 208.915 91.44))
   (no_connect (at 208.915 111.76))
-  (no_connect (at 208.915 96.52))
-  (no_connect (at 147.955 109.22))
-  (no_connect (at 147.955 124.46))
+  (no_connect (at 208.915 99.06))
   (no_connect (at 59.69 185.42))
   (no_connect (at 133.985 144.78))
-  (no_connect (at 208.915 99.06))
   (no_connect (at 208.915 142.24))
-  (no_connect (at 208.915 91.44))
-  (no_connect (at 147.955 99.06))
-  (no_connect (at 208.915 43.18))
-  (no_connect (at 208.915 106.68))
   (no_connect (at 147.955 106.68))
   (no_connect (at 208.915 104.14))
+  (no_connect (at 147.955 109.22))
+  (no_connect (at 208.915 96.52))
+  (no_connect (at 147.955 127))
+  (no_connect (at 147.955 99.06))
+  (no_connect (at 208.915 106.68))
+  (no_connect (at 147.955 104.14))
+  (no_connect (at 208.915 43.18))
+  (no_connect (at 147.955 124.46))
   (wire (pts (xy 15.24 169.545) (xy 29.21 169.545))
     (stroke (width 0) (type solid) (color 0 0 0 0))
@@
       (effects (font (size 1.27 1.27)) hide)
     )
+    (property "PartsBoxID" "0402-470R-1%" (id 4) (at 87.63 41.91 0)
+      (effects (font (size 1.27 1.27)) hide)
+    )
   )
   (symbol (lib_id "Device:R") (at 87.63 49.53 90) (mirror x) (unit 1)
@@
       (effects (font (size 1.27 1.27)) hide)
     )
+    (property "PartsBoxID" "0402-470R-1%" (id 4) (at 87.63 49.53 0)
+      (effects (font (size 1.27 1.27)) hide)
+    )
   )
   (symbol (lib_id "Device:R") (at 160.02 170.18 0) (unit 1)
@@
       (effects (font (size 1.27 1.27)) (justify left))
     )
-    (property "Value" "1k" (id 1) (at 161.798 171.323 0)
+    (property "Value" "1K 1%" (id 1) (at 161.798 171.323 0)
       (effects (font (size 1.27 1.27)) (justify left))
     )
@@
     )
     (property "Field8" "125049511" (id 9) (at 160.02 170.18 0)
+      (effects (font (size 1.27 1.27)) hide)
+    )
+    (property "PartsBoxID" "0402-1K-1%" (id 4) (at 160.02 170.18 0)
       (effects (font (size 1.27 1.27)) hide)
     )
@@
       (effects (font (size 1.27 1.27)) (justify left))
     )
-    (property "Value" "1k" (id 1) (at 227.457 40.513 0)
+    (property "Value" "1K 1%" (id 1) (at 227.457 40.513 0)
       (effects (font (size 1.27 1.27)) (justify left))
     )
@@
     )
     (property "Field8" "125049511" (id 9) (at 225.679 39.37 0)
+      (effects (font (size 1.27 1.27)) hide)
+    )
+    (property "PartsBoxID" "0402-1K-1%" (id 4) (at 225.679 39.37 0)
       (effects (font (size 1.27 1.27)) hide)
     )
@@
       (effects (font (size 1.27 1.27)) hide)
     )
+    (property "PartsBoxID" "LTST-S270KRKT" (id 4) (at 160.02 161.29 0)
+      (effects (font (size 1.27 1.27)) hide)
+    )
   )
   (symbol (lib_id "Device:LED") (at 225.679 26.67 90) (unit 1)
@@
       (effects (font (size 1.27 1.27)) hide)
     )
+    (property "PartsBoxID" "LTST-S270KGKT" (id 4) (at 225.679 26.67 0)
+      (effects (font (size 1.27 1.27)) hide)
+    )
   )
   (symbol (lib_id "Device:C") (at 19.05 52.07 0) (unit 1)
@@
       (effects (font (size 1.27 1.27)) (justify left))
     )
-    (property "Value" "100n" (id 1) (at 19.431 54.483 0)
+    (property "Value" "100n 16v" (id 1) (at 19.431 54.483 0)
       (effects (font (size 1.27 1.27)) (justify left))
     )
@@
     )
     (property "Field8" "110091611" (id 9) (at 19.05 52.07 0)
+      (effects (font (size 1.27 1.27)) hide)
+    )
+    (property "PartsBoxID" "0402-100nF-X7R-16V" (id 4) (at 19.05 52.07 0)
       (effects (font (size 1.27 1.27)) hide)
     )
@@
       (effects (font (size 1.27 1.27)) hide)
     )
+    (property "PartsBoxID" "74LVC1G07SE-7" (id 4) (at 29.21 177.165 0)
+      (effects (font (size 1.27 1.27)) hide)
+    )
   )
   (symbol (lib_id "AP3000:74LVC1G07_copy") (at 152.4 180.34 0) (unit 1)
@@
     )
     (property "Part Description" "Buffer, Non-Inverting 1 Element 1 Bit per Element Open Drain Output SOT-353" (id 8) (at 152.4 180.34 0)
+      (effects (font (size 1.27 1.27)) hide)
+    )
+    (property "PartsBoxID" "74LVC1G07SE-7" (id 4) (at 152.4 180.34 0)
       (effects (font (size 1.27 1.27)) hide)
     )
@@
       (effects (font (size 1.27 1.27)) hide)
     )
+    (property "PartsBoxID" "CDDFN10-3324P" (id 4) (at 40.64 76.835 0)
+      (effects (font (size 1.27 1.27)) hide)
+    )
   )
   (symbol (lib_id "AP3000:TPD4EUSB30") (at 88.9 76.835 0) (unit 1)
@@
       (effects (font (size 1.27 1.27)) hide)
     )
+    (property "PartsBoxID" "CDDFN10-3324P" (id 4) (at 88.9 76.835 0)
+      (effects (font (size 1.27 1.27)) hide)
+    )
   )
   (symbol (lib_id "Connector_Generic:Conn_02x20_Odd_Even") (at 260.604 50.8 0) (unit 1)
@@
     )
     (property "Part Description" "PinHeader_2x20_P2.54mm_Vertical" (id 9) (at 260.604 50.8 0)
+      (effects (font (size 1.27 1.27)) hide)
+    )
+    (property "PartsBoxID" "C124374" (id 4) (at 260.604 50.8 0)
       (effects (font (size 1.27 1.27)) hide)
     )
@@
       (effects (font (size 1.27 1.27)) (justify left bottom) hide)
     )
+    (property "PartsBoxID" "0826-1X1T-GH-F" (id 4) (at 65.405 41.91 0)
+      (effects (font (size 1.27 1.27)) hide)
+    )
   )
   (symbol (lib_id "AP3000:ComputeModule4-CM4") (at 180.975 76.2 0) (unit 1)
@@
       (effects (font (size 1.27 1.27)) hide)
     )
+    (property "PartsBoxID" "\nDF40C-100DS-0.4V(51)" (id 4) (at 180.975 76.2 0)
+      (effects (font (size 1.27 1.27)) hide)
+    )

Commit message: Rework AP3000 PoE section, power section and change solder paste to -10% overall, -15% for small chips / mpcie and -20% for the raspi connector
Parts:
- C1: footprint Capacitor_SMD:C_0402_1005Metric -> Capacitor_SMD:C_0603_1608Metric; PartsBoxID 0402-100nF-X7R-16V -> 0603-100nF-X7R-16V
- C45: footprint Capacitor_SMD:C_0402_1005Metric -> Capacitor_SMD:C_0603_1608Metric; PartsBoxID 0402-.1uF-X5R-25V -> 0603-.1uF-X5R-25V
- R1, R10: footprint Resistor_SMD:R_0402_1005Metric -> Resistor_SMD:R_0603_1608Metric; PartsBoxID 0402-1K-1% -> 0603-1K-1%
- R2, R3: footprint Resistor_SMD:R_0402_1005Metric -> Resistor_SMD:R_0603_1608Metric; PartsBoxID 0402-470R-1% -> 0603-470R-1%
- U1, U2: footprint Package_SON:USON-10_2.5x1.0mm_P0.5mm -> Scott:USON-10_2.51x1.0mm_P0.5mm
Changed lines of the file:
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@@
 (kicad_sch (version 20201015) (generator eeschema)
-  (page 1 8)
   (paper "A4")
   (title_block
@@
   (junction (at 269.494 63.5) (diameter 1.016) (color 0 0 0 0))
   (junction (at 269.494 68.58) (diameter 1.016) (color 0 0 0 0))
+  (no_connect (at 208.915 142.24))
+  (no_connect (at 133.985 144.78))
+  (no_connect (at 208.915 111.76))
+  (no_connect (at 147.955 124.46))
+  (no_connect (at 147.955 104.14))
   (no_connect (at 208.915 91.44))
-  (no_connect (at 208.915 111.76))
   (no_connect (at 208.915 99.06))
   (no_connect (at 59.69 185.42))
-  (no_connect (at 133.985 144.78))
-  (no_connect (at 208.915 142.24))
+  (no_connect (at 147.955 109.22))
+  (no_connect (at 208.915 104.14))
+  (no_connect (at 208.915 96.52))
   (no_connect (at 147.955 106.68))
-  (no_connect (at 208.915 104.14))
-  (no_connect (at 147.955 109.22))
-  (no_connect (at 208.915 96.52))
   (no_connect (at 147.955 127))
   (no_connect (at 147.955 99.06))
   (no_connect (at 208.915 106.68))
-  (no_connect (at 147.955 104.14))
   (no_connect (at 208.915 43.18))
-  (no_connect (at 147.955 124.46))
   (wire (pts (xy 15.24 169.545) (xy 29.21 169.545))
     (stroke (width 0) (type solid) (color 0 0 0 0))
@@
     (property "Reference" "R2" (id 0) (at 88.265 44.2722 90))
     (property "Value" "470R" (id 1) (at 88.265 46.5836 90))
-    (property "Footprint" "Resistor_SMD:R_0402_1005Metric" (id 2) (at 87.63 40.132 90)
+    (property "Footprint" "Resistor_SMD:R_0603_1608Metric" (id 2) (at 87.63 40.132 90)
       (effects (font (size 1.27 1.27)) hide)
     )
@@
       (effects (font (size 1.27 1.27)) hide)
     )
-    (property "PartsBoxID" "0402-470R-1%" (id 4) (at 87.63 41.91 0)
+    (property "PartsBoxID" "0603-470R-1%" (id 4) (at 87.63 41.91 0)
       (effects (font (size 1.27 1.27)) hide)
     )
@@
     (property "Reference" "R3" (id 0) (at 87.63 54.61 90))
     (property "Value" "470R" (id 1) (at 87.63 52.07 90))
-    (property "Footprint" "Resistor_SMD:R_0402_1005Metric" (id 2) (at 87.63 47.752 90)
+    (property "Footprint" "Resistor_SMD:R_0603_1608Metric" (id 2) (at 87.63 47.752 90)
       (effects (font (size 1.27 1.27)) hide)
     )
@@
       (effects (font (size 1.27 1.27)) hide)
     )
-    (property "PartsBoxID" "0402-470R-1%" (id 4) (at 87.63 49.53 0)
+    (property "PartsBoxID" "0603-470R-1%" (id 4) (at 87.63 49.53 0)
       (effects (font (size 1.27 1.27)) hide)
     )
@@
       (effects (font (size 1.27 1.27)) (justify left))
     )
-    (property "Footprint" "Resistor_SMD:R_0402_1005Metric" (id 2) (at 158.242 170.18 90)
+    (property "Footprint" "Resistor_SMD:R_0603_1608Metric" (id 2) (at 158.242 170.18 90)
       (effects (font (size 1.27 1.27)) hide)
     )
@@
       (effects (font (size 1.27 1.27)) hide)
     )
-    (property "PartsBoxID" "0402-1K-1%" (id 4) (at 160.02 170.18 0)
+    (property "PartsBoxID" "0603-1K-1%" (id 4) (at 160.02 170.18 0)
       (effects (font (size 1.27 1.27)) hide)
     )
@@
       (effects (font (size 1.27 1.27)) (justify left))
     )
-    (property "Footprint" "Resistor_SMD:R_0402_1005Metric" (id 2) (at 223.901 39.37 90)
+    (property "Footprint" "Resistor_SMD:R_0603_1608Metric" (id 2) (at 223.901 39.37 90)
       (effects (font (size 1.27 1.27)) hide)
     )
@@
       (effects (font (size 1.27 1.27)) hide)
     )
-    (property "PartsBoxID" "0402-1K-1%" (id 4) (at 225.679 39.37 0)
+    (property "PartsBoxID" "0603-1K-1%" (id 4) (at 225.679 39.37 0)
       (effects (font (size 1.27 1.27)) hide)
     )
@@
       (effects (font (size 1.27 1.27)) (justify right))
     )
-    (property "Footprint" "Capacitor_SMD:C_0402_1005Metric" (id 2) (at 97.155 132.08 0)
+    (property "Footprint" "Capacitor_SMD:C_0603_1608Metric" (id 2) (at 97.155 132.08 0)
       (effects (font (size 1.27 1.27)) hide)
     )
@@
       (effects (font (size 1.27 1.27)) hide)
     )
-    (property "PartsBoxID" "0402-.1uF-X5R-25V" (id 4) (at 97.155 132.08 0)
+    (property "PartsBoxID" "0603-.1uF-X5R-25V" (id 4) (at 97.155 132.08 0)
       (effects (font (size 1.27 1.27)) hide)
     )
@@
       (effects (font (size 1.27 1.27)) (justify left))
     )
-    (property "Footprint" "Capacitor_SMD:C_0402_1005Metric" (id 2) (at 20.0152 55.88 0)
+    (property "Footprint" "Capacitor_SMD:C_0603_1608Metric" (id 2) (at 20.0152 55.88 0)
       (effects (font (size 1.27 1.27)) hide)
     )
@@
       (effects (font (size 1.27 1.27)) hide)
     )
-    (property "PartsBoxID" "0402-100nF-X7R-16V" (id 4) (at 19.05 52.07 0)
+    (property "PartsBoxID" "0603-100nF-X7R-16V" (id 4) (at 19.05 52.07 0)
       (effects (font (size 1.27 1.27)) hide)
     )
@@
     (property "Reference" "U1" (id 0) (at 40.64 64.9732 0))
     (property "Value" "TPD4EUSB30" (id 1) (at 40.64 67.2846 0))
-    (property "Footprint" "Package_SON:USON-10_2.5x1.0mm_P0.5mm" (id 2) (at 16.51 86.995 0)
+    (property "Footprint" "Scott:USON-10_2.51x1.0mm_P0.5mm" (id 2) (at 16.51 86.995 0)
       (effects (font (size 1.27 1.27)) hide)
     )
@@
     (property "Reference" "U2" (id 0) (at 88.9 64.9732 0))
     (property "Value" "TPD4EUSB30" (id 1) (at 88.9 67.2846 0))
-    (property "Footprint" "Package_SON:USON-10_2.5x1.0mm_P0.5mm" (id 2) (at 64.77 86.995 0)
-      (effects (font (size 1.27 1.27)) hide)
-    )
+    (property "Footprint" "Scott:USON-10_2.51x1.0mm_P0.5mm" (id 2) (at 64.77 86.995 0)
+      (effects (font (size 1.27 1.27)) hide)
+    )

Commit message: Ordered AP3000 PCBs Ordered FlatAntPanel4x4 PCBs Ordered FlatAntPanel4x4_Reflector PCBs
Parts:
- C45: PartsBoxID 0603-.1uF-X5R-25V -> 0603-100nF-X7R-25V
Changed lines of the file:
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@@
   (junction (at 269.494 63.5) (diameter 1.016) (color 0 0 0 0))
   (junction (at 269.494 68.58) (diameter 1.016) (color 0 0 0 0))
-  (no_connect (at 208.915 142.24))
-  (no_connect (at 133.985 144.78))
-  (no_connect (at 208.915 111.76))
-  (no_connect (at 147.955 124.46))
-  (no_connect (at 147.955 104.14))
-  (no_connect (at 208.915 91.44))
-  (no_connect (at 208.915 99.06))
-  (no_connect (at 59.69 185.42))
-  (no_connect (at 147.955 109.22))
-  (no_connect (at 208.915 104.14))
   (no_connect (at 208.915 96.52))
-  (no_connect (at 147.955 106.68))
+  (no_connect (at 208.915 106.68))
   (no_connect (at 147.955 127))
   (no_connect (at 147.955 99.06))
-  (no_connect (at 208.915 106.68))
+  (no_connect (at 208.915 99.06))
+  (no_connect (at 147.955 109.22))
+  (no_connect (at 208.915 111.76))
+  (no_connect (at 208.915 91.44))
+  (no_connect (at 133.985 144.78))
+  (no_connect (at 147.955 106.68))
+  (no_connect (at 59.69 185.42))
   (no_connect (at 208.915 43.18))
+  (no_connect (at 147.955 104.14))
+  (no_connect (at 147.955 124.46))
+  (no_connect (at 208.915 142.24))
+  (no_connect (at 208.915 104.14))
   (wire (pts (xy 15.24 169.545) (xy 29.21 169.545))
     (stroke (width 0) (type solid) (color 0 0 0 0))
@@
       (effects (font (size 1.27 1.27)) hide)
     )
-    (property "PartsBoxID" "0603-.1uF-X5R-25V" (id 4) (at 97.155 132.08 0)
-      (effects (font (size 1.27 1.27)) hide)
-    )
+    (property "PartsBoxID" "0603-100nF-X7R-25V" (id 4) (at 97.155 132.08 0)
+      (effects (font (size 1.27 1.27)) hide)
+    )
