File: AP3000/CM4_HighSpeed.kicad_sch (KiCad schematic)
At the start: 6 parts, among them J4 Conn_01x22_Female, J5 Conn_01x22_Female, J6 THD-02-R

Commit message: Forgot to add PCB cutout resulting in some components being moved
Parts:
- removed J6: THD-02-R, Connector_PinHeader_2.54mm:PinHeader_2x02_P2.54mm_Vertical, symbol Connector_Generic:Conn_02x02_Odd_Even
Connections:
- net GPIO_VREF is gone; now on net +3.3v: R6.1, R7.1
- net SCL1 is gone; now on net ID_SC: J4.20 (Pin_20), R7.2
- net SDA1 is gone; now on net ID_SD: J4.21 (Pin_21), R6.2
Changed lines of the file:
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@@
   (junction (at 157.48 133.35) (diameter 1.016) (color 0 0 0 0))
   (junction (at 157.48 140.97) (diameter 1.016) (color 0 0 0 0))
+  (no_connect (at 102.87 100.33))
+  (no_connect (at 102.87 39.37))
+  (no_connect (at 41.91 92.71))
+  (no_connect (at 41.91 128.27))
+  (no_connect (at 41.91 82.55))
+  (no_connect (at 160.02 55.88))
+  (no_connect (at 102.87 82.55))
+  (no_connect (at 102.87 120.65))
+  (no_connect (at 41.91 135.89))
+  (no_connect (at 41.91 97.79))
+  (no_connect (at 41.91 146.05))
+  (no_connect (at 160.02 53.34))
+  (no_connect (at 41.91 29.21))
+  (no_connect (at 160.02 71.12))
+  (no_connect (at 102.87 113.03))
+  (no_connect (at 102.87 130.81))
+  (no_connect (at 102.87 97.79))
+  (no_connect (at 102.87 80.01))
+  (no_connect (at 102.87 26.67))
+  (no_connect (at 160.02 138.43))
+  (no_connect (at 102.87 135.89))
+  (no_connect (at 102.87 105.41))
+  (no_connect (at 160.02 63.5))
   (no_connect (at 41.91 138.43))
-  (no_connect (at 102.87 105.41))
+  (no_connect (at 41.91 90.17))
   (no_connect (at 102.87 107.95))
-  (no_connect (at 160.02 53.34))
-  (no_connect (at 41.91 107.95))
-  (no_connect (at 41.91 146.05))
+  (no_connect (at 41.91 100.33))
+  (no_connect (at 102.87 146.05))
+  (no_connect (at 41.91 105.41))
+  (no_connect (at 41.91 115.57))
+  (no_connect (at 41.91 85.09))
+  (no_connect (at 41.91 123.19))
+  (no_connect (at 41.91 151.13))
+  (no_connect (at 102.87 123.19))
+  (no_connect (at 41.91 143.51))
+  (no_connect (at 102.87 92.71))
+  (no_connect (at 102.87 90.17))
   (no_connect (at 160.02 60.96))
-  (no_connect (at 41.91 100.33))
-  (no_connect (at 102.87 97.79))
-  (no_connect (at 102.87 85.09))
-  (no_connect (at 41.91 82.55))
-  (no_connect (at 41.91 85.09))
-  (no_connect (at 102.87 123.19))
-  (no_connect (at 41.91 31.75))
-  (no_connect (at 102.87 138.43))
-  (no_connect (at 41.91 92.71))
-  (no_connect (at 41.91 90.17))
   (no_connect (at 102.87 128.27))
   (no_connect (at 102.87 151.13))
-  (no_connect (at 102.87 100.33))
-  (no_connect (at 41.91 151.13))
-  (no_connect (at 41.91 97.79))
+  (no_connect (at 102.87 138.43))
+  (no_connect (at 102.87 85.09))
   (no_connect (at 102.87 87.63))
-  (no_connect (at 102.87 92.71))
-  (no_connect (at 102.87 146.05))
-  (no_connect (at 102.87 82.55))
-  (no_connect (at 102.87 90.17))
-  (no_connect (at 160.02 55.88))
-  (no_connect (at 102.87 39.37))
+  (no_connect (at 41.91 107.95))
+  (no_connect (at 41.91 31.75))
+  (no_connect (at 41.91 120.65))
+  (no_connect (at 102.87 143.51))
+  (no_connect (at 41.91 130.81))
   (no_connect (at 102.87 115.57))
-  (no_connect (at 102.87 120.65))
-  (no_connect (at 41.91 130.81))
-  (no_connect (at 41.91 29.21))
-  (no_connect (at 102.87 26.67))
-  (no_connect (at 41.91 123.19))
-  (no_connect (at 41.91 143.51))
   (no_connect (at 41.91 113.03))
-  (no_connect (at 41.91 105.41))
-  (no_connect (at 102.87 143.51))
-  (no_connect (at 102.87 130.81))
-  (no_connect (at 160.02 71.12))
-  (no_connect (at 102.87 135.89))
-  (no_connect (at 41.91 135.89))
-  (no_connect (at 41.91 120.65))
-  (no_connect (at 160.02 63.5))
-  (no_connect (at 160.02 138.43))
-  (no_connect (at 102.87 80.01))
-  (no_connect (at 102.87 113.03))
-  (no_connect (at 41.91 128.27))
-  (no_connect (at 41.91 115.57))
   (wire (pts (xy 25.4 74.93) (xy 41.91 74.93))
     (stroke (width 0) (type solid) (color 0 0 0 0))
@@
     (stroke (width 0) (type solid) (color 0 0 0 0))
   )
-  (wire (pts (xy 35.052 184.912) (xy 41.402 184.912))
-    (stroke (width 0) (type solid) (color 0 0 0 0))
-  )
-  (wire (pts (xy 35.052 187.452) (xy 41.402 187.452))
+  (wire (pts (xy 35.052 184.912) (xy 64.262 184.912))
+    (stroke (width 0) (type solid) (color 0 0 0 0))
+  )
+  (wire (pts (xy 35.052 187.452) (xy 56.642 187.452))
     (stroke (width 0) (type solid) (color 0 0 0 0))
   )
@@
   )
   (wire (pts (xy 46.99 170.561) (xy 56.642 170.561))
-    (stroke (width 0) (type solid) (color 0 0 0 0))
-  )
-  (wire (pts (xy 54.102 184.912) (xy 64.262 184.912))
-    (stroke (width 0) (type solid) (color 0 0 0 0))
-  )
-  (wire (pts (xy 54.102 187.452) (xy 56.642 187.452))
     (stroke (width 0) (type solid) (color 0 0 0 0))
   )
@@
     (effects (font (size 1.27 1.27)) (justify right bottom))
   )
-  (label "ID_SC" (at 40.64 184.912 180)
-    (effects (font (size 1.27 1.27)) (justify right bottom))
-  )
-  (label "ID_SD" (at 40.64 187.452 180)
-    (effects (font (size 1.27 1.27)) (justify right bottom))
-  )
-  (label "GPIO_VREF" (at 46.99 170.561 0)
-    (effects (font (size 1.27 1.27)) (justify left bottom))
-  )
   (label "SCL1" (at 77.47 184.912 180)
     (effects (font (size 1.27 1.27)) (justify right bottom))
@@
     (effects (font (size 1.27 1.27)) (justify right))
   )
-  (hierarchical_label "GPIO_VREF" (shape input) (at 46.99 170.561 180)
+  (hierarchical_label "+3.3v" (shape input) (at 46.99 170.561 180)
     (effects (font (size 1.27 1.27)) (justify right))
   )
@@
       (effects (font (size 1.27 1.27)) hide)
     )
-  )
-  (symbol (lib_id "Connector_Generic:Conn_02x02_Odd_Even") (at 46.482 184.912 0) (unit 1)
-    (in_bom yes) (on_board yes)
-    (property "Reference" "J6" (id 0) (at 43.815 179.705 0))
-    (property "Value" "THD-02-R" (id 1) (at 47.752 181.7116 0))
-    (property "Footprint" "Connector_PinHeader_2.54mm:PinHeader_2x02_P2.54mm_Vertical" (id 2) (at 46.482 184.912 0)
-      (effects (font (size 1.27 1.27)) hide)
-    )
-    (property "Datasheet" "https://www.toby.co.uk/uploads/publications/1673.pdf" (id 3) (at 46.482 184.912 0)
-      (effects (font (size 1.27 1.27)) hide)
-    )
-    (property "Field4" "Toby" (id 4) (at 46.482 184.912 0)
-      (effects (font (size 1.27 1.27)) hide)
-    )
-    (property "Field5" "THD-02-R" (id 5) (at 46.482 184.912 0)
-      (effects (font (size 1.27 1.27)) hide)
-    )
-    (property "Field6" "151-604-425-761" (id 6) (at 46.482 184.912 0)
-      (effects (font (size 1.27 1.27)) hide)
-    )
-    (property "Field7" "EDAC" (id 7) (at 46.482 184.912 0)
-      (effects (font (size 1.27 1.27)) hide)
-    )
-    (property "Field8" "UCON00791" (id 8) (at 46.482 184.912 0)
-      (effects (font (size 1.27 1.27)) hide)
-    )
-    (property "Part Description" "PinHeader_2x02_P2.54mm_Vertical" (id 9) (at 46.482 184.912 0)
-      (effects (font (size 1.27 1.27)) hide)
-    )

Commit message: Route more
Parts:
- removed J4, J5: Conn_01x22_Female, Connector_FFC-FPC:Hirose_FH12-22S-0.5SH_1x22-1MP_P0.50mm_Horizontal, symbol Connector:Conn_01x22_Female
- added J4: Camera 0, AP3000:EDAC 690-019-298-412, symbol AP3000:HDMI_A_1.4
- added J5: Camera 1, AP3000:EDAC 690-019-298-412, symbol AP3000:HDMI_A_1.4
Connections:
- net +3.3v: now also J4.18 (+5V), J5.18 (+5V)
- net CAM0_C_N: now also J4.12 (CK-)
- net CAM0_C_P: now also J4.10 (CK+)
- net CAM0_D0_N: now also J4.9 (D0-)
- net CAM0_D0_P: now also J4.7 (D0+)
- net CAM0_D1_N: now also J4.6 (D1-)
- net CAM0_D1_P: now also J4.4 (D1+)
- net CAM1_C_N: now also J5.12 (CK-)
- net CAM1_C_P: now also J5.10 (CK+)
- net CAM1_D0_N: now also J5.9 (D0-)
- net CAM1_D0_P: now also J5.7 (D0+)
- net CAM1_D1_N: now also J5.6 (D1-)
- net CAM1_D1_P: now also J5.4 (D1+)
- net CAM1_D2_N: now also J5.3 (D2-)
- net CAM1_D2_P: now also J5.1 (D2+)
- net CAM1_D3_N: now also J5.19 (HPD/HEAC-)
- net CAM1_D3_P: now also J5.14 (UTILITY/HEAC+)
- net CAM_GPIO: now also J4.13 (CEC), J5.13 (CEC)
- net GND: now also J4.11 (CKS), J4.17 (GND), J4.2 (D2S), J4.5 (D1S), J4.8 (D0S), J4.SH1 (SH), J4.SH2 (SH), J4.SH3 (SH), J4.SH4 (SH), J5.11 (CKS), J5.17 (GND), J5.2 (D2S), J5.5 (D1S), J5.8 (D0S), J5.SH1 (SH), J5.SH2 (SH), J5.SH3 (SH), J5.SH4 (SH)
- net ID_SC: now also J4.15 (SCL)
- net ID_SD: now also J4.16 (SDA)
- net SCL0: now also J5.15 (SCL)
- net SDA0: now also J5.16 (SDA)
- no-connect marks 50 -> 48

Commit message: Almost done routing!
Parts:
- removed J4: Camera 0, AP3000:EDAC 690-019-298-412, symbol AP3000:HDMI_A_1.4
- removed J5: Camera 1, AP3000:EDAC 690-019-298-412, symbol AP3000:HDMI_A_1.4
- added J10: Camera 1 Power, Connectors:SCREWTERMINAL-5MM-2, symbol Connector:Screw_Terminal_01x02
- added J4: Camera 0, Connector_RJ:RJ45_Amphenol_54602-x08_Horizontal, symbol Connector:RJ45
- added J5: Camera 0 Power, Connectors:SCREWTERMINAL-5MM-2, symbol Connector:Screw_Terminal_01x02
- added J6: Camera 1, Connector_RJ:RJ45_Amphenol_54602-x08_Horizontal, symbol Connector:RJ45
Connections:
- net +3.3v: now also J10.1 (Pin_1), J5.1 (Pin_1)
- net CAM0_C_N: now also J4.6
- net CAM0_C_P: now also J4.5
- net CAM0_D0_N: now also J4.2
- net CAM0_D0_P: now also J4.1
- net CAM0_D1_N: now also J4.4
- net CAM0_D1_P: now also J4.3
- net CAM1_C_N: now also J6.6
- net CAM1_C_P: now also J6.5
- net CAM1_D0_N: now also J6.2
- net CAM1_D0_P: now also J6.1
- net CAM1_D1_N: now also J6.4
- net CAM1_D1_P: now also J6.3
- net GND: now also J10.2 (Pin_2), J5.2 (Pin_2)
- net ID_SC: now also J4.7
- net ID_SD: now also J4.8
- net SCL0: now also J6.7
- net SDA0: now also J6.8
- net CAM1_D2_N: no longer names the net of Module1.133 (CAM1_D2_N)
- net CAM1_D2_P: no longer names the net of Module1.135 (CAM1_D2_P)
- net CAM1_D3_N: no longer names the net of Module1.139 (CAM1_D3_N)
- net CAM1_D3_P: no longer names the net of Module1.141 (CAM1_D3_P)

Commit message: AP3000: Fixup PartsBoxID linkage and placed first order Working on a design for a 5 GHz panel antenna array for a point-to-point replacement
Parts:
- Module1: PartsBoxID (none) -> DF40C-100DS-0.4V(51)
- R6, R7: PartsBoxID (none) -> 0402-2.2K-1%
Changed lines of the file:
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@@
   (junction (at 105.41 140.97) (diameter 1.016) (color 0 0 0 0))
   (junction (at 105.41 148.59) (diameter 1.016) (color 0 0 0 0))
+  (no_connect (at 102.87 85.09))
+  (no_connect (at 102.87 135.89))
+  (no_connect (at 41.91 135.89))
+  (no_connect (at 41.91 82.55))
+  (no_connect (at 102.87 67.31))
+  (no_connect (at 41.91 115.57))
+  (no_connect (at 41.91 151.13))
+  (no_connect (at 41.91 85.09))
+  (no_connect (at 41.91 123.19))
+  (no_connect (at 102.87 77.47))
+  (no_connect (at 41.91 92.71))
+  (no_connect (at 41.91 128.27))
+  (no_connect (at 102.87 143.51))
+  (no_connect (at 102.87 26.67))
+  (no_connect (at 41.91 31.75))
+  (no_connect (at 102.87 97.79))
+  (no_connect (at 102.87 120.65))
+  (no_connect (at 41.91 29.21))
+  (no_connect (at 102.87 82.55))
+  (no_connect (at 102.87 113.03))
   (no_connect (at 102.87 92.71))
-  (no_connect (at 102.87 120.65))
-  (no_connect (at 102.87 146.05))
-  (no_connect (at 41.91 85.09))
-  (no_connect (at 102.87 77.47))
-  (no_connect (at 41.91 100.33))
-  (no_connect (at 41.91 128.27))
-  (no_connect (at 41.91 143.51))
-  (no_connect (at 41.91 92.71))
-  (no_connect (at 102.87 115.57))
-  (no_connect (at 102.87 90.17))
+  (no_connect (at 102.87 128.27))
+  (no_connect (at 102.87 39.37))
+  (no_connect (at 41.91 130.81))
+  (no_connect (at 102.87 138.43))
+  (no_connect (at 41.91 146.05))
+  (no_connect (at 41.91 90.17))
+  (no_connect (at 102.87 74.93))
+  (no_connect (at 41.91 138.43))
   (no_connect (at 102.87 87.63))
   (no_connect (at 41.91 120.65))
-  (no_connect (at 102.87 113.03))
-  (no_connect (at 41.91 82.55))
+  (no_connect (at 41.91 105.41))
+  (no_connect (at 102.87 107.95))
   (no_connect (at 41.91 113.03))
+  (no_connect (at 102.87 105.41))
+  (no_connect (at 102.87 130.81))
+  (no_connect (at 41.91 143.51))
+  (no_connect (at 41.91 107.95))
   (no_connect (at 102.87 123.19))
-  (no_connect (at 41.91 138.43))
-  (no_connect (at 41.91 123.19))
+  (no_connect (at 102.87 69.85))
+  (no_connect (at 102.87 80.01))
+  (no_connect (at 102.87 115.57))
+  (no_connect (at 102.87 146.05))
+  (no_connect (at 102.87 100.33))
+  (no_connect (at 41.91 97.79))
+  (no_connect (at 41.91 100.33))
   (no_connect (at 102.87 151.13))
-  (no_connect (at 102.87 85.09))
-  (no_connect (at 102.87 138.43))
-  (no_connect (at 41.91 107.95))
-  (no_connect (at 41.91 135.89))
-  (no_connect (at 102.87 26.67))
-  (no_connect (at 41.91 146.05))
-  (no_connect (at 102.87 100.33))
-  (no_connect (at 102.87 105.41))
-  (no_connect (at 102.87 135.89))
-  (no_connect (at 102.87 128.27))
-  (no_connect (at 102.87 67.31))
-  (no_connect (at 102.87 39.37))
-  (no_connect (at 102.87 97.79))
-  (no_connect (at 41.91 151.13))
-  (no_connect (at 102.87 82.55))
-  (no_connect (at 41.91 29.21))
-  (no_connect (at 102.87 80.01))
-  (no_connect (at 41.91 115.57))
-  (no_connect (at 102.87 69.85))
-  (no_connect (at 102.87 130.81))
-  (no_connect (at 102.87 74.93))
-  (no_connect (at 41.91 90.17))
-  (no_connect (at 102.87 107.95))
-  (no_connect (at 41.91 130.81))
-  (no_connect (at 41.91 97.79))
-  (no_connect (at 41.91 31.75))
-  (no_connect (at 102.87 143.51))
-  (no_connect (at 41.91 105.41))
+  (no_connect (at 102.87 90.17))
   (wire (pts (xy 25.4 74.93) (xy 41.91 74.93))
     (stroke (width 0) (type solid) (color 0 0 0 0))
@@
       (effects (font (size 1.27 1.27)) hide)
     )
+    (property "PartsBoxID" "0402-2.2K-1%" (id 4) (at 56.642 175.895 0)
+      (effects (font (size 1.27 1.27)) hide)
+    )
   )
   (symbol (lib_id "Device:R") (at 64.262 175.895 0) (unit 1)
@@
     )
     (property "Field8" "120889581" (id 9) (at 64.262 175.895 0)
+      (effects (font (size 1.27 1.27)) hide)
+    )
+    (property "PartsBoxID" "0402-2.2K-1%" (id 4) (at 64.262 175.895 0)
       (effects (font (size 1.27 1.27)) hide)
     )
@@
       (effects (font (size 1.27 1.27)) hide)
     )
+    (property "PartsBoxID" "\nDF40C-100DS-0.4V(51)" (id 4) (at -67.31 87.63 0)
+      (effects (font (size 1.27 1.27)) hide)
+    )

Commit message: Rework AP3000 PoE section, power section and change solder paste to -10% overall, -15% for small chips / mpcie and -20% for the raspi connector
Parts:
- Module1: PartsBoxID DF40C-100DS-0.4V(51) -> DF40C-100DS-0.4V(51)
- R6, R7: footprint Resistor_SMD:R_0402_1005Metric -> Resistor_SMD:R_0603_1608Metric; PartsBoxID 0402-2.2K-1% -> 0603-2.2K-1%
Changed lines of the file:
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@@
 (kicad_sch (version 20201015) (generator eeschema)
-  (page 1 8)
   (paper "A4")
   (title_block
@@
   (junction (at 105.41 140.97) (diameter 1.016) (color 0 0 0 0))
   (junction (at 105.41 148.59) (diameter 1.016) (color 0 0 0 0))
-  (no_connect (at 102.87 85.09))
-  (no_connect (at 102.87 135.89))
-  (no_connect (at 41.91 135.89))
+  (no_connect (at 41.91 105.41))
+  (no_connect (at 102.87 128.27))
+  (no_connect (at 102.87 120.65))
+  (no_connect (at 41.91 138.43))
+  (no_connect (at 102.87 130.81))
+  (no_connect (at 41.91 128.27))
   (no_connect (at 41.91 82.55))
-  (no_connect (at 102.87 67.31))
   (no_connect (at 41.91 115.57))
+  (no_connect (at 41.91 113.03))
+  (no_connect (at 41.91 31.75))
   (no_connect (at 41.91 151.13))
-  (no_connect (at 41.91 85.09))
-  (no_connect (at 41.91 123.19))
   (no_connect (at 102.87 77.47))
-  (no_connect (at 41.91 92.71))
-  (no_connect (at 41.91 128.27))
-  (no_connect (at 102.87 143.51))
-  (no_connect (at 102.87 26.67))
-  (no_connect (at 41.91 31.75))
-  (no_connect (at 102.87 97.79))
-  (no_connect (at 102.87 120.65))
-  (no_connect (at 41.91 29.21))
-  (no_connect (at 102.87 82.55))
-  (no_connect (at 102.87 113.03))
-  (no_connect (at 102.87 92.71))
-  (no_connect (at 102.87 128.27))
   (no_connect (at 102.87 39.37))
   (no_connect (at 41.91 130.81))
+  (no_connect (at 102.87 143.51))
+  (no_connect (at 41.91 123.19))
+  (no_connect (at 102.87 146.05))
+  (no_connect (at 41.91 135.89))
+  (no_connect (at 41.91 85.09))
+  (no_connect (at 102.87 80.01))
+  (no_connect (at 41.91 92.71))
   (no_connect (at 102.87 138.43))
+  (no_connect (at 41.91 120.65))
+  (no_connect (at 41.91 29.21))
+  (no_connect (at 102.87 135.89))
+  (no_connect (at 102.87 107.95))
+  (no_connect (at 102.87 92.71))
+  (no_connect (at 102.87 113.03))
+  (no_connect (at 102.87 74.93))
+  (no_connect (at 41.91 100.33))
+  (no_connect (at 102.87 87.63))
+  (no_connect (at 102.87 105.41))
+  (no_connect (at 41.91 97.79))
+  (no_connect (at 102.87 69.85))
+  (no_connect (at 102.87 151.13))
+  (no_connect (at 41.91 90.17))
+  (no_connect (at 102.87 26.67))
+  (no_connect (at 102.87 82.55))
+  (no_connect (at 102.87 90.17))
+  (no_connect (at 102.87 67.31))
+  (no_connect (at 102.87 123.19))
+  (no_connect (at 102.87 100.33))
+  (no_connect (at 102.87 97.79))
+  (no_connect (at 102.87 85.09))
+  (no_connect (at 41.91 107.95))
+  (no_connect (at 41.91 143.51))
+  (no_connect (at 102.87 115.57))
   (no_connect (at 41.91 146.05))
-  (no_connect (at 41.91 90.17))
-  (no_connect (at 102.87 74.93))
-  (no_connect (at 41.91 138.43))
-  (no_connect (at 102.87 87.63))
-  (no_connect (at 41.91 120.65))
-  (no_connect (at 41.91 105.41))
-  (no_connect (at 102.87 107.95))
-  (no_connect (at 41.91 113.03))
-  (no_connect (at 102.87 105.41))
-  (no_connect (at 102.87 130.81))
-  (no_connect (at 41.91 143.51))
-  (no_connect (at 41.91 107.95))
-  (no_connect (at 102.87 123.19))
-  (no_connect (at 102.87 69.85))
-  (no_connect (at 102.87 80.01))
-  (no_connect (at 102.87 115.57))
-  (no_connect (at 102.87 146.05))
-  (no_connect (at 102.87 100.33))
-  (no_connect (at 41.91 97.79))
-  (no_connect (at 41.91 100.33))
-  (no_connect (at 102.87 151.13))
-  (no_connect (at 102.87 90.17))
   (wire (pts (xy 25.4 74.93) (xy 41.91 74.93))
     (stroke (width 0) (type solid) (color 0 0 0 0))
@@
       (effects (font (size 1.27 1.27)) (justify left))
     )
-    (property "Footprint" "Resistor_SMD:R_0402_1005Metric" (id 2) (at 54.864 175.895 90)
+    (property "Footprint" "Resistor_SMD:R_0603_1608Metric" (id 2) (at 54.864 175.895 90)
       (effects (font (size 1.27 1.27)) hide)
     )
@@
       (effects (font (size 1.27 1.27)) hide)
     )
-    (property "PartsBoxID" "0402-2.2K-1%" (id 4) (at 56.642 175.895 0)
+    (property "PartsBoxID" "0603-2.2K-1%" (id 4) (at 56.642 175.895 0)
       (effects (font (size 1.27 1.27)) hide)
     )
@@
       (effects (font (size 1.27 1.27)) (justify left))
     )
-    (property "Footprint" "Resistor_SMD:R_0402_1005Metric" (id 2) (at 62.484 175.895 90)
+    (property "Footprint" "Resistor_SMD:R_0603_1608Metric" (id 2) (at 62.484 175.895 90)
       (effects (font (size 1.27 1.27)) hide)
     )
@@
       (effects (font (size 1.27 1.27)) hide)
     )
-    (property "PartsBoxID" "0402-2.2K-1%" (id 4) (at 64.262 175.895 0)
+    (property "PartsBoxID" "0603-2.2K-1%" (id 4) (at 64.262 175.895 0)
       (effects (font (size 1.27 1.27)) hide)
     )
@@
       (effects (font (size 1.27 1.27)) hide)
     )
-    (property "PartsBoxID" "\nDF40C-100DS-0.4V(51)" (id 4) (at -67.31 87.63 0)
-      (effects (font (size 1.27 1.27)) hide)
-    )
+    (property "PartsBoxID" "DF40C-100DS-0.4V(51)" (id 4) (at -67.31 87.63 0)
+      (effects (font (size 1.27 1.27)) hide)
+    )
