File: AP3000/USB2-HUB.kicad_sch (KiCad schematic)
At the start: 10 parts, among them J7 YJ-USB-AF_SMT-01, U4 TPD4EUSB30, U7 AP22653W6

Commit message: Route all the high speed lines and most gpio
Connections:
- no-connect marks 3 -> 1
Changed lines of the file:
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@@
   (junction (at 224.155 70.485) (diameter 1.016) (color 0 0 0 0))
   (junction (at 234.315 70.485) (diameter 1.016) (color 0 0 0 0))
-  (no_connect (at 73.66 54.61))
-  (no_connect (at 73.66 59.69))
   (no_connect (at 180.975 75.565))
   (wire (pts (xy 84.455 106.045) (xy 86.995 106.045))

Commit message: AP3000: Fixup PartsBoxID linkage and placed first order Working on a design for a 5 GHz panel antenna array for a point-to-point replacement
Parts:
- C16: PartsBoxID (none) -> EEF-CX0J101R
- C17, C19, C2, C20, C21: value 10u -> 10u 10v; PartsBoxID (none) -> 0805-10uF-X7R-10V
- J7: PartsBoxID (none) -> YJ-USB-AF_SMT-01
- R36: PartsBoxID (none) -> 0402-15K-1%
- U4: PartsBoxID (none) -> CDDFN10-3324P
- U7: PartsBoxID (none) -> AP22653W6-7
Changed lines of the file:
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@@
+      (effects (font (size 1.27 1.27)) hide)
+    )
+    (property "PartsBoxID" "0402-15K-1%" (id 4) (at 192.405 73.025 0)
       (effects (font (size 1.27 1.27)) hide)
     )
@@
       (effects (font (size 1.27 1.27)) (justify left))
     )
-    (property "Value" "10u" (id 1) (at 145.796 76.708 0)
+    (property "Value" "10u 10v" (id 1) (at 145.796 76.708 0)
       (effects (font (size 1.27 1.27)) (justify left))
     )
@@
       (effects (font (size 1.27 1.27)) hide)
     )
+    (property "PartsBoxID" "0805-10uF-X7R-10V" (id 4) (at 142.875 75.565 0)
+      (effects (font (size 1.27 1.27)) hide)
+    )
   )
   (symbol (lib_id "Device:CP") (at 200.533 76.835 0) (unit 1)
@@
       (effects (font (size 1.27 1.27)) hide)
     )
+    (property "PartsBoxID" "EEF-CX0J101R" (id 4) (at 200.533 76.835 0)
+      (effects (font (size 1.27 1.27)) hide)
+    )
   )
   (symbol (lib_id "Device:C") (at 213.995 76.835 0) (unit 1)
@@
       (effects (font (size 1.27 1.27)) (justify left))
     )
-    (property "Value" "10u" (id 1) (at 216.916 77.978 0)
+    (property "Value" "10u 10v" (id 1) (at 216.916 77.978 0)
       (effects (font (size 1.27 1.27)) (justify left))
     )
@@
       (effects (font (size 1.27 1.27)) hide)
     )
+    (property "PartsBoxID" "0805-10uF-X7R-10V" (id 4) (at 213.995 76.835 0)
+      (effects (font (size 1.27 1.27)) hide)
+    )
   )
   (symbol (lib_id "Device:C") (at 224.155 76.835 0) (unit 1)
@@
       (effects (font (size 1.27 1.27)) (justify left))
     )
-    (property "Value" "10u" (id 1) (at 227.076 77.978 0)
+    (property "Value" "10u 10v" (id 1) (at 227.076 77.978 0)
       (effects (font (size 1.27 1.27)) (justify left))
     )
@@
       (effects (font (size 1.27 1.27)) hide)
     )
+    (property "PartsBoxID" "0805-10uF-X7R-10V" (id 4) (at 224.155 76.835 0)
+      (effects (font (size 1.27 1.27)) hide)
+    )
   )
   (symbol (lib_id "Device:C") (at 234.315 76.835 0) (unit 1)
@@
       (effects (font (size 1.27 1.27)) (justify left))
     )
-    (property "Value" "10u" (id 1) (at 237.236 77.978 0)
+    (property "Value" "10u 10v" (id 1) (at 237.236 77.978 0)
       (effects (font (size 1.27 1.27)) (justify left))
     )
@@
       (effects (font (size 1.27 1.27)) hide)
     )
+    (property "PartsBoxID" "0805-10uF-X7R-10V" (id 4) (at 234.315 76.835 0)
+      (effects (font (size 1.27 1.27)) hide)
+    )
   )
   (symbol (lib_id "Device:C") (at 244.475 76.835 0) (unit 1)
@@
       (effects (font (size 1.27 1.27)) (justify left))
     )
-    (property "Value" "10u" (id 1) (at 247.396 77.978 0)
+    (property "Value" "10u 10v" (id 1) (at 247.396 77.978 0)
       (effects (font (size 1.27 1.27)) (justify left))
     )
@@
     )
     (property "Field8" "111893011" (id 9) (at 244.475 76.835 0)
+      (effects (font (size 1.27 1.27)) hide)
+    )
+    (property "PartsBoxID" "0805-10uF-X7R-10V" (id 4) (at 244.475 76.835 0)
       (effects (font (size 1.27 1.27)) hide)
     )
@@
       (effects (font (size 1.27 1.27)) hide)
     )
+    (property "PartsBoxID" "AP22653W6-7" (id 4) (at 173.355 73.025 0)
+      (effects (font (size 1.27 1.27)) hide)
+    )
   )
   (symbol (lib_id "Scott:YJ-USB-AF_SMT-01") (at 86.995 95.885 0) (unit 1)
@@
     )
     (property "Datasheet" "" (id 3) (at 86.995 95.885 0)
+      (effects (font (size 1.27 1.27)) hide)
+    )
+    (property "PartsBoxID" "YJ-USB-AF_SMT-01" (id 4) (at 86.995 95.885 0)
       (effects (font (size 1.27 1.27)) hide)
     )
@@
       (effects (font (size 1.27 1.27)) hide)
     )
+    (property "PartsBoxID" "CDDFN10-3324P" (id 4) (at 86.36 57.15 0)
+      (effects (font (size 1.27 1.27)) hide)
+    )

Commit message: Rework AP3000 PoE section, power section and change solder paste to -10% overall, -15% for small chips / mpcie and -20% for the raspi connector
Parts:
- R36: footprint Resistor_SMD:R_0402_1005Metric -> Resistor_SMD:R_0603_1608Metric; PartsBoxID 0402-15K-1% -> 0603-15K-1%
- U4: footprint Package_SON:USON-10_2.5x1.0mm_P0.5mm -> Scott:USON-10_2.51x1.0mm_P0.5mm
Changed lines of the file:
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@@
 (kicad_sch (version 20201015) (generator eeschema)
-  (page 1 8)
   (paper "A4")
   (title_block
@@
       (effects (font (size 1.27 1.27)) (justify left))
     )
-    (property "Footprint" "Resistor_SMD:R_0402_1005Metric" (id 2) (at 192.405 74.803 90)
+    (property "Footprint" "Resistor_SMD:R_0603_1608Metric" (id 2) (at 192.405 74.803 90)
       (effects (font (size 1.27 1.27)) hide)
     )
@@
       (effects (font (size 1.27 1.27)) hide)
     )
-    (property "PartsBoxID" "0402-15K-1%" (id 4) (at 192.405 73.025 0)
+    (property "PartsBoxID" "0603-15K-1%" (id 4) (at 192.405 73.025 0)
       (effects (font (size 1.27 1.27)) hide)
     )
@@
     (property "Reference" "U4" (id 0) (at 86.36 45.2882 0))
     (property "Value" "TPD4EUSB30" (id 1) (at 86.36 47.5996 0))
-    (property "Footprint" "Package_SON:USON-10_2.5x1.0mm_P0.5mm" (id 2) (at 62.23 67.31 0)
-      (effects (font (size 1.27 1.27)) hide)
-    )
+    (property "Footprint" "Scott:USON-10_2.51x1.0mm_P0.5mm" (id 2) (at 62.23 67.31 0)
+      (effects (font (size 1.27 1.27)) hide)
+    )
