File: AP3000/poe.kicad_sch (KiCad schematic)
At the start: 72 parts, among them IC2 TPS23751PWPR, J11 Barrel_Jack, Q1 FDS86242, U12 HMHA2801AR2, U6 TL431AIDBVR

Commit message: Rework AP3000 board - ground planes instead of power planes internal
Parts:
- C28: footprint Capacitor_SMD:C_1812_4532Metric -> Capacitor_SMD:C_1210_3225Metric; PartsBoxID 1812-2.2nF-X7R-2KV -> 1210-2.2nF-X7R-2KV
Changed lines of the file:
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@@
       (effects (font (size 1.27 1.27)) (justify left))
     )
-    (property "Footprint" "Capacitor_SMD:C_1812_4532Metric" (id 2) (at 186.055 100.33 0)
+    (property "Footprint" "Capacitor_SMD:C_1210_3225Metric" (id 2) (at 186.055 100.33 0)
       (effects (font (size 1.27 1.27)) hide)
     )
@@
       (effects (font (size 1.27 1.27)) hide)
     )
-    (property "PartsBoxID" "1812-2.2nF-X7R-2KV" (id 4) (at 186.055 100.33 0)
+    (property "PartsBoxID" "1210-2.2nF-X7R-2KV" (id 4) (at 186.055 100.33 0)
       (effects (font (size 1.27 1.27)) hide)
     )
