File: AP3000/PSUs.kicad_sch (KiCad schematic)
At the start: 37 parts, among them U10 TPS563249DDCR, U11 TPS563249DDCR, U13 TPS563249DDCR

Commit message: Update JLCPCB components for AP3000
Parts:
- C30, C49, C56: LCSC (none) -> C14663; Part Description (none) -> 100nF 10% or 20% 50V Ceramic Capacitor X7R 0603
- C31, C35, C50, C51, C52, C57, C58, C59: LCSC (none) -> C90146
- C37, C47, C53, C54, C60, C61: LCSC (none) -> C15850
- C48, C55, C62: LCSC (none) -> C14663
- R28: LCSC (none) -> C14890
- R30, R33, R38: LCSC (none) -> C25804
- R32: LCSC (none) -> C23058
- R37: LCSC (none) -> C22809
