File: FlatAntPanel4x4_dual/FlatAntPanel4x4_dual.kicad_pcb (KiCad board)
At the start: 4 copper layers, 186 x 226 mm, 124 parts

Commit message: Rework AP3000 PoE section, power section and change solder paste to -10% overall, -15% for small chips / mpcie and -20% for the raspi connector
Parts:
- added NT1: NetTie_3_Tee, Scott-RF-JLCPCB-1.2mm7628-4layer:RF-T-50ohm, F.Cu at (-40.9, 78.3)
- added NT1: NetTie_3_Tee, Scott-RF-JLCPCB-1.2mm7628-4layer:RF-T-50ohm, F.Cu at (13.6, 78.3)
- added NT1: NetTie_3_Tee, Scott-RF-JLCPCB-1.2mm7628-4layer:RF-T-50ohm, F.Cu at (13.6, 22.3)
- added NT1: NetTie_3_Tee, Scott-RF-JLCPCB-1.2mm7628-4layer:RF-T-50ohm, F.Cu at (-40.9, 22.3)
- added REF**: RF-Angle-100ohm, Scott-RF-JLCPCB-1.2mm7628-4layer:RF-Angle-100ohm, F.Cu at (17.5, 35.9)
- added REF**: RF-Transformer-70.71ohm-Right, Scott-RF-JLCPCB-1.2mm7628-4layer:RF-Transformer-70.71ohm-Right, F.Cu at (-11.2, 69.6)
- added REF**: Patch_5.5_Linear_DualPol_420R, Scott-RF-JLCPCB-1.2mm7628-4layer:Patch_5.5_Linear_DualPol_420R, F.Cu at (-54.5, 83.3)
- added REF**: RF-Transformer-70.71ohm, Scott-RF-JLCPCB-1.2mm7628-4layer:RF-Transformer-70.71ohm, F.Cu at (38.5, 13.6)
- added REF**: Patch_5.5_Linear_DualPol_420R, Scott-RF-JLCPCB-1.2mm7628-4layer:Patch_5.5_Linear_DualPol_420R, F.Cu at (27.2, 56.0)
- added REF**: RF-Transformer-70.71ohm, Scott-RF-JLCPCB-1.2mm7628-4layer:RF-Transformer-70.71ohm, F.Cu at (-54.5, 91.9)
- added REF**: RF-Transformer-70.71ohm, Scott-RF-JLCPCB-1.2mm7628-4layer:RF-Transformer-70.71ohm, F.Cu at (-63.2, 0.00)
- added REF**: RF-Transformer-70.71ohm, Scott-RF-JLCPCB-1.2mm7628-4layer:RF-Transformer-70.71ohm, F.Cu at (13.6, -10.9)
- added REF**: RF-Angle-100ohm, Scott-RF-JLCPCB-1.2mm7628-4layer:RF-Angle-100ohm, F.Cu at (17.4, 64.6)
- added REF**: RF-Transformer-70.71ohm, Scott-RF-JLCPCB-1.2mm7628-4layer:RF-Transformer-70.71ohm, F.Cu at (0.00, 8.64)
- added REF**: RF-Angle-100ohm, Scott-RF-JLCPCB-1.2mm7628-4layer:RF-Angle-100ohm, F.Cu at (9.81, 8.64)
- added REF**: RF-Transformer-70.71ohm-Right, Scott-RF-JLCPCB-1.2mm7628-4layer:RF-Transformer-70.71ohm-Right, F.Cu at (35.9, 56.0)
- added REF**: RF-Transformer-70.71ohm-Right, Scott-RF-JLCPCB-1.2mm7628-4layer:RF-Transformer-70.71ohm-Right, F.Cu at (27.2, 64.6)
- added REF**: RF-Transformer-70.71ohm-Right, Scott-RF-JLCPCB-1.2mm7628-4layer:RF-Transformer-70.71ohm-Right, F.Cu at (27.3, 8.64)
- added REF**: RF-Angle-100ohm, Scott-RF-JLCPCB-1.2mm7628-4layer:RF-Angle-100ohm, F.Cu at (-37.1, 8.64)
- added REF**: RF-Angle-100ohm, Scott-RF-JLCPCB-1.2mm7628-4layer:RF-Angle-100ohm, F.Cu at (-65.7, -8.40)
- added REF**: RF-Angle-100ohm, Scott-RF-JLCPCB-1.2mm7628-4layer:RF-Angle-100ohm, F.Cu at (-16.1, 47.6)
- added REF**: Patch_5.5_Linear_DualPol_420R, Scott-RF-JLCPCB-1.2mm7628-4layer:Patch_5.5_Linear_DualPol_420R, F.Cu at (-54.5, 0.00)
- added REF**: Patch_5.5_Linear_DualPol_420R, Scott-RF-JLCPCB-1.2mm7628-4layer:Patch_5.5_Linear_DualPol_420R, F.Cu at (0.00, 27.3)
- added REF**: Flat_Ant_Hole, Scott:Flat_Ant_Hole, F.Cu at (41.4, 14.5)
- added REF**: RF-Angle-100ohm, Scott-RF-JLCPCB-1.2mm7628-4layer:RF-Angle-100ohm, F.Cu at (-68.7, 96.5)
- added REF**: RF-Transformer-70.71ohm-Right, Scott-RF-JLCPCB-1.2mm7628-4layer:RF-Transformer-70.71ohm-Right, F.Cu at (-63.2, 27.3)
- added REF**: RF-Transformer-70.71ohm-Right, Scott-RF-JLCPCB-1.2mm7628-4layer:RF-Transformer-70.71ohm-Right, F.Cu at (-13.6, 40.5)
- added REF**: RF-Angle-100ohm, Scott-RF-JLCPCB-1.2mm7628-4layer:RF-Angle-100ohm, F.Cu at (17.4, 91.9)
- added REF**: RF-Angle-100ohm, Scott-RF-JLCPCB-1.2mm7628-4layer:RF-Angle-100ohm, F.Cu at (-68.7, 40.5)
- added REF**: Patch_5.5_Linear_DualPol_420R, Scott-RF-JLCPCB-1.2mm7628-4layer:Patch_5.5_Linear_DualPol_420R, F.Cu at (-27.3, 56.0)
- added REF**: RF-Transformer-70.71ohm, Scott-RF-JLCPCB-1.2mm7628-4layer:RF-Transformer-70.71ohm, F.Cu at (-0.01, 91.9)
- added REF**: RF-Angle-100ohm, Scott-RF-JLCPCB-1.2mm7628-4layer:RF-Angle-100ohm, F.Cu at (9.80, 91.9)
- added REF**: RF-Transformer-70.71ohm-Right, Scott-RF-JLCPCB-1.2mm7628-4layer:RF-Transformer-70.71ohm-Right, F.Cu at (-13.6, 96.5)
- added REF**: RF-Angle-100ohm, Scott-RF-JLCPCB-1.2mm7628-4layer:RF-Angle-100ohm, F.Cu at (41.4, -13.5)
- added REF**: Patch_5.5_Linear_DualPol_420R, Scott-RF-JLCPCB-1.2mm7628-4layer:Patch_5.5_Linear_DualPol_420R, F.Cu at (27.3, 0.00)
- added REF**: Patch_5.5_Linear_DualPol_420R, Scott-RF-JLCPCB-1.2mm7628-4layer:Patch_5.5_Linear_DualPol_420R, F.Cu at (-27.3, 0.00)
- added REF**: RF-Angle-100ohm, Scott-RF-JLCPCB-1.2mm7628-4layer:RF-Angle-100ohm, F.Cu at (-37.1, 64.6)
- added REF**: RF-Transformer-70.71ohm-Right, Scott-RF-JLCPCB-1.2mm7628-4layer:RF-Transformer-70.71ohm-Right, F.Cu at (-8.65, 83.3)
- added REF**: RF-Transformer-70.71ohm, Scott-RF-JLCPCB-1.2mm7628-4layer:RF-Transformer-70.71ohm, F.Cu at (-18.6, 83.3)
- added REF**: Patch_5.5_Linear_DualPol_420R, Scott-RF-JLCPCB-1.2mm7628-4layer:Patch_5.5_Linear_DualPol_420R, F.Cu at (-54.5, 27.3)
- added REF**: Patch_5.5_Linear_DualPol_420R, Scott-RF-JLCPCB-1.2mm7628-4layer:Patch_5.5_Linear_DualPol_420R, F.Cu at (27.3, 27.3)
- added REF**: RF-Transformer-70.71ohm-Right, Scott-RF-JLCPCB-1.2mm7628-4layer:RF-Transformer-70.71ohm-Right, F.Cu at (-18.6, 56.0)
- added REF**: RF-Angle-100ohm, Scott-RF-JLCPCB-1.2mm7628-4layer:RF-Angle-100ohm, F.Cu at (13.6, 93.9)
- added REF**: RF-Angle-100ohm, Scott-RF-JLCPCB-1.2mm7628-4layer:RF-Angle-100ohm, F.Cu at (38.5, -8.40)
- added REF**: Flat_Ant_Hole, Scott:Flat_Ant_Hole, F.Cu at (-68.7, 68.5)
- added REF**: RF-Transformer-70.71ohm, Scott-RF-JLCPCB-1.2mm7628-4layer:RF-Transformer-70.71ohm, F.Cu at (35.9, 83.3)
- added REF**: RF-Transformer-70.71ohm-Right, Scott-RF-JLCPCB-1.2mm7628-4layer:RF-Transformer-70.71ohm-Right, F.Cu at (27.3, 35.9)
- added REF**: RF-Angle-100ohm, Scott-RF-JLCPCB-1.2mm7628-4layer:RF-Angle-100ohm, F.Cu at (38.4, 47.6)
- added REF**: Patch_5.5_Linear_DualPol_420R, Scott-RF-JLCPCB-1.2mm7628-4layer:Patch_5.5_Linear_DualPol_420R, F.Cu at (-54.5, 56.0)
- added REF**: RF-Transformer-70.71ohm, Scott-RF-JLCPCB-1.2mm7628-4layer:RF-Transformer-70.71ohm, F.Cu at (-18.6, 27.3)
- added REF**: RF-Angle-100ohm, Scott-RF-JLCPCB-1.2mm7628-4layer:RF-Angle-100ohm, F.Cu at (-37.1, 35.9)
- added REF**: RF-Transformer-70.71ohm-Right, Scott-RF-JLCPCB-1.2mm7628-4layer:RF-Transformer-70.71ohm-Right, F.Cu at (-27.3, 8.64)
- added REF**: RF-Transformer-70.71ohm, Scott-RF-JLCPCB-1.2mm7628-4layer:RF-Transformer-70.71ohm, F.Cu at (35.9, 27.3)
- added REF**: RF-Transformer-70.71ohm-Right, Scott-RF-JLCPCB-1.2mm7628-4layer:RF-Transformer-70.71ohm-Right, F.Cu at (-13.6, 42.5)
- added REF**: RF-Transformer-70.71ohm-Right, Scott-RF-JLCPCB-1.2mm7628-4layer:RF-Transformer-70.71ohm-Right, F.Cu at (-40.9, -10.9)
- added REF**: RF-Angle-100ohm, Scott-RF-JLCPCB-1.2mm7628-4layer:RF-Angle-100ohm, F.Cu at (17.5, 8.64)
- added REF**: RF-Transformer-70.71ohm-Right, Scott-RF-JLCPCB-1.2mm7628-4layer:RF-Transformer-70.71ohm-Right, F.Cu at (-65.7, 13.6)
- added REF**: RF-Transformer-70.71ohm-Right, Scott-RF-JLCPCB-1.2mm7628-4layer:RF-Transformer-70.71ohm-Right, F.Cu at (-18.6, 0.00)
- added REF**: RF-Transformer-70.71ohm-Right, Scott-RF-JLCPCB-1.2mm7628-4layer:RF-Transformer-70.71ohm-Right, F.Cu at (-8.64, 27.3)
- added REF**: Patch_5.5_Linear_DualPol_420R, Scott-RF-JLCPCB-1.2mm7628-4layer:Patch_5.5_Linear_DualPol_420R, F.Cu at (0.00, 0.00)
- added REF**: Patch_5.5_Linear_DualPol_420R, Scott-RF-JLCPCB-1.2mm7628-4layer:Patch_5.5_Linear_DualPol_420R, F.Cu at (-27.3, 27.3)
- added REF**: RF-Transformer-70.71ohm, Scott-RF-JLCPCB-1.2mm7628-4layer:RF-Transformer-70.71ohm, F.Cu at (0.00, 35.9)
- added REF**: RF-Angle-100ohm, Scott-RF-JLCPCB-1.2mm7628-4layer:RF-Angle-100ohm, F.Cu at (-40.9, 93.9)
- added REF**: RF-Angle-100ohm, Scott-RF-JLCPCB-1.2mm7628-4layer:RF-Angle-100ohm, F.Cu at (13.6, 37.9)
- added REF**: RF-Transformer-70.71ohm-Right, Scott-RF-JLCPCB-1.2mm7628-4layer:RF-Transformer-70.71ohm-Right, F.Cu at (-27.3, 64.6)
- added REF**: RF-Transformer-70.71ohm-Right, Scott-RF-JLCPCB-1.2mm7628-4layer:RF-Transformer-70.71ohm-Right, F.Cu at (-65.7, 69.6)
- added REF**: RF-Transformer-70.71ohm, Scott-RF-JLCPCB-1.2mm7628-4layer:RF-Transformer-70.71ohm, F.Cu at (-63.2, 56.0)
- added REF**: Patch_5.5_Linear_DualPol_420R, Scott-RF-JLCPCB-1.2mm7628-4layer:Patch_5.5_Linear_DualPol_420R, F.Cu at (-0.01, 56.0)
- added REF**: RF-Transformer-70.71ohm, Scott-RF-JLCPCB-1.2mm7628-4layer:RF-Transformer-70.71ohm, F.Cu at (-54.5, 8.64)
- added REF**: RF-Angle-100ohm, Scott-RF-JLCPCB-1.2mm7628-4layer:RF-Angle-100ohm, F.Cu at (-11.2, -8.40)
- added REF**: RF-Transformer-70.71ohm-Right, Scott-RF-JLCPCB-1.2mm7628-4layer:RF-Transformer-70.71ohm-Right, F.Cu at (-40.9, 45.0)
- added REF**: RF-Transformer-70.71ohm, Scott-RF-JLCPCB-1.2mm7628-4layer:RF-Transformer-70.71ohm, F.Cu at (-54.5, 64.6)
- added REF**: RF-Transformer-70.71ohm, Scott-RF-JLCPCB-1.2mm7628-4layer:RF-Transformer-70.71ohm, F.Cu at (-0.01, 64.6)
- added REF**: RF-Transformer-70.71ohm, Scott-RF-JLCPCB-1.2mm7628-4layer:RF-Transformer-70.71ohm, F.Cu at (38.4, 69.6)
- added REF**: RF-Transformer-70.71ohm, Scott-RF-JLCPCB-1.2mm7628-4layer:RF-Transformer-70.71ohm, F.Cu at (-54.5, 35.9)
- added REF**: RF-Transformer-70.71ohm, Scott-RF-JLCPCB-1.2mm7628-4layer:RF-Transformer-70.71ohm, F.Cu at (-16.1, 69.6)
- added REF**: RF-Angle-100ohm, Scott-RF-JLCPCB-1.2mm7628-4layer:RF-Angle-100ohm, F.Cu at (-11.2, 47.6)
- added REF**: RF-Transformer-70.71ohm-Right, Scott-RF-JLCPCB-1.2mm7628-4layer:RF-Transformer-70.71ohm-Right, F.Cu at (-27.3, 91.9)
- added REF**: RF-Angle-100ohm, Scott-RF-JLCPCB-1.2mm7628-4layer:RF-Angle-100ohm, F.Cu at (-44.7, 91.9)
- added REF**: RF-Transformer-70.71ohm-Right, Scott-RF-JLCPCB-1.2mm7628-4layer:RF-Transformer-70.71ohm-Right, F.Cu at (35.9, 0.00)
- added REF**: RF-Transformer-70.71ohm, Scott-RF-JLCPCB-1.2mm7628-4layer:RF-Transformer-70.71ohm, F.Cu at (-16.1, 13.6)
- added REF**: RF-Angle-100ohm, Scott-RF-JLCPCB-1.2mm7628-4layer:RF-Angle-100ohm, F.Cu at (-16.1, -8.40)
- added REF**: RF-Angle-100ohm, Scott-RF-JLCPCB-1.2mm7628-4layer:RF-Angle-100ohm, F.Cu at (-44.7, 8.64)
- added REF**: Patch_5.5_Linear_DualPol_420R, Scott-RF-JLCPCB-1.2mm7628-4layer:Patch_5.5_Linear_DualPol_420R, F.Cu at (27.2, 83.3)
- added REF**: RF-Angle-100ohm, Scott-RF-JLCPCB-1.2mm7628-4layer:RF-Angle-100ohm, F.Cu at (-37.1, 91.9)
- added REF**: RF-Transformer-70.71ohm-Right, Scott-RF-JLCPCB-1.2mm7628-4layer:RF-Transformer-70.71ohm-Right, F.Cu at (-13.6, -13.5)
- added REF**: RF-Angle-100ohm, Scott-RF-JLCPCB-1.2mm7628-4layer:RF-Angle-100ohm, F.Cu at (-40.9, 37.9)
- added REF**: RF-Angle-100ohm, Scott-RF-JLCPCB-1.2mm7628-4layer:RF-Angle-100ohm, F.Cu at (9.81, 35.9)
- added REF**: RF-Angle-100ohm, Scott-RF-JLCPCB-1.2mm7628-4layer:RF-Angle-100ohm, F.Cu at (-44.7, 35.9)
- added REF**: RF-Angle-100ohm, Scott-RF-JLCPCB-1.2mm7628-4layer:RF-Angle-100ohm, F.Cu at (-44.7, 64.6)
- added REF**: RF-Transformer-70.71ohm-Right, Scott-RF-JLCPCB-1.2mm7628-4layer:RF-Transformer-70.71ohm-Right, F.Cu at (-11.2, 13.6)
- added REF**: RF-Angle-100ohm, Scott-RF-JLCPCB-1.2mm7628-4layer:RF-Angle-100ohm, F.Cu at (41.4, 42.5)
- added REF**: RF-Angle-100ohm, Scott-RF-JLCPCB-1.2mm7628-4layer:RF-Angle-100ohm, F.Cu at (9.80, 64.6)
- added REF**: RF-Transformer-70.71ohm, Scott-RF-JLCPCB-1.2mm7628-4layer:RF-Transformer-70.71ohm, F.Cu at (-8.65, 56.0)
- added REF**: RF-Transformer-70.71ohm-Right, Scott-RF-JLCPCB-1.2mm7628-4layer:RF-Transformer-70.71ohm-Right, F.Cu at (-27.3, 35.9)
- added REF**: RF-Transformer-70.71ohm, Scott-RF-JLCPCB-1.2mm7628-4layer:RF-Transformer-70.71ohm, F.Cu at (-8.64, 0.00)
- added REF**: RF-Transformer-70.71ohm, Scott-RF-JLCPCB-1.2mm7628-4layer:RF-Transformer-70.71ohm, F.Cu at (13.6, 45.0)
- added REF**: RF-Transformer-70.71ohm-Right, Scott-RF-JLCPCB-1.2mm7628-4layer:RF-Transformer-70.71ohm-Right, F.Cu at (-63.2, 83.3)
- added REF**: RF-Transformer-70.71ohm-Right, Scott-RF-JLCPCB-1.2mm7628-4layer:RF-Transformer-70.71ohm-Right, F.Cu at (27.2, 91.9)
- added REF**: Patch_5.5_Linear_DualPol_420R, Scott-RF-JLCPCB-1.2mm7628-4layer:Patch_5.5_Linear_DualPol_420R, F.Cu at (-27.3, 83.3)
- added REF**: RF-Angle-100ohm, Scott-RF-JLCPCB-1.2mm7628-4layer:RF-Angle-100ohm, F.Cu at (-65.7, 47.6)
- added REF**: Patch_5.5_Linear_DualPol_420R, Scott-RF-JLCPCB-1.2mm7628-4layer:Patch_5.5_Linear_DualPol_420R, F.Cu at (-0.01, 83.3)
- moved Feed1 260.7 mm to (336.3, 37.7)
- moved REF** 260.7 mm to (395.2, 135.9)
- moved REF** 260.7 mm to (336.3, 10.4)
- moved REF** 260.7 mm to (336.3, 64.9)
- moved REF** 260.7 mm to (395.2, 108.6)
- moved REF** 260.7 mm to (395.2, 190.4)
- moved REF** 260.7 mm to (395.2, 163.1)
- moved AA10 260.7 mm to (404.6, 17.7)
- moved AA10 260.7 mm to (318.3, 111.5)
- moved AA10 260.7 mm to (404.6, 99.4)
- moved AA10 260.7 mm to (404.6, 44.9)
- moved AA10 260.7 mm to (318.3, 166.0)
- moved AA10 260.7 mm to (318.3, 138.7)
- moved AA10 260.7 mm to (318.3, 193.2)
- moved AA10 260.7 mm to (404.6, 72.2)
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Routing:
- net (no net): track 0.00 -> 1265.8 mm
