File: FlatAntPanel4x4_dual/FlatAntPanel4x4_dual.kicad_sch (KiCad schematic)
At the start: 27 parts

Commit message: Rework AP3000 PoE section, power section and change solder paste to -10% overall, -15% for small chips / mpcie and -20% for the raspi connector
Parts:
- removed AA1, AA10, AA11, AA12, AA13, AA14, AA15, AA16, AA2, AA3, AA4, AA5, AA6, AA7, AA8, AA9: RFAngle, Scott-RF-JLCPCB-1.2mm7628-4layer:RF-Angle-100ohm, symbol Scott:RFAngle
- removed AE1, AE2, AE3, AE4, AE5, AE6, AE7, AE8: Antenna, Scott-RF-JLCPCB-1.2mm7628-4layer:Patch_Inset_5.5_Linear_7.1dBi_100R, symbol Device:Antenna
- removed Feed1: Feed1, Scott:Flat_Ant_Hole, symbol Device:Antenna_Shield
- removed NT1, NT2: NetTie_3_Tee, Scott-RF-JLCPCB-1.2mm7628-4layer:RF-T-50ohm, symbol Device:NetTie_3_Tee
