File: Taylor's Water Layout/Taylor's Water Layout.kicad_pcb (KiCad board)
At the start: 2 copper layers, 0 parts

Commit message: More work on Antennas - laying out the new panel as a 2x2 aperture coupled patch
Other:
- board text added: "10 ft"
- board text added: "12.5 ft"
- board text removed: "18 ft"
Changed lines of the file:
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@@
-(kicad_pcb (version 20201220) (generator pcbnew)
+(kicad_pcb (version 20210126) (generator pcbnew)
   (general
     (thickness 1.6)
@@
       (hpglpenspeed 20)
       (hpglpendiameter 15.000000)
+      (dxfpolygonmode true)
+      (dxfimperialunits true)
+      (dxfusepcbnewfont true)
       (psnegative false)
       (psa4output false)
@@
   (gr_rect (start 266.7 -63.5) (end 241.3 63.5) (layer "F.Cu") (width 0.2) (fill none))
   (gr_circle (center 406.4 139.7) (end 508 139.7) (layer "B.Cu") (width 0.2) (fill none))
-  (gr_circle (center 609.6 0) (end 711.2 0) (layer "B.Cu") (width 0.2) (fill none))
   (gr_circle (center 406.4 -139.7) (end 508 -139.7) (layer "B.Cu") (width 0.2) (fill none))
   (gr_line (start 266.7 0) (end 292.1 0) (layer "B.Adhes") (width 2.74))
@@
   (gr_line (start 0 152.4) (end 266.7 152.4) (layer "Eco1.User") (width 2.74))
   (gr_line (start 266.7 63.5) (end 266.7 152.4) (layer "Eco1.User") (width 2.74))
-  (gr_rect (start 279.4 -266.7) (end 736.6 266.7) (layer "B.CrtYd") (width 0.2) (fill none))
+  (gr_rect (start 279.4 -266.7) (end 533.4 266.7) (layer "B.CrtYd") (width 0.2) (fill none))
   (gr_text "S" (at 787.4 -368.3 180) (layer "F.Cu")
     (effects (font (size 6.58 6.58) (thickness 0.3)))
@@
     (effects (font (size 4.04 4.04) (thickness 0.3)))
   )
+  (gr_text "5 ft" (at 254 -330.2 90) (layer "F.SilkS")
+    (effects (font (size 4.04 4.04) (thickness 0.3)))
+  )
   (gr_text "6 ft" (at 127 0 90) (layer "F.SilkS")
     (effects (font (size 4.04 4.04) (thickness 0.3)))
@@
     (effects (font (size 6.58 6.58) (thickness 0.3)))
   )
+  (gr_text "5 ft" (at 254 330.2 90) (layer "F.SilkS")
+    (effects (font (size 4.04 4.04) (thickness 0.3)))
+  )
   (gr_text "5 ft" (at 215.9 101.6) (layer "F.SilkS")
     (effects (font (size 4.04 4.04) (thickness 0.3)))
   )
+  (gr_text "12.5 ft" (at 127 -228.6 90) (layer "F.SilkS")
+    (effects (font (size 4.04 4.04) (thickness 0.3)))
+  )
   (gr_text "3/4\" PVC to house" (at 190.5 127) (layer "F.SilkS")
     (effects (font (size 4.04 4.04) (thickness 0.3)))
@@
     (effects (font (size 4.04 4.04) (thickness 0.3)))
   )
-  (gr_text "21 ft" (at 762 0 270) (layer "F.SilkS")
+  (gr_text "21 ft" (at 558.8 0 270) (layer "F.SilkS")
     (effects (font (size 4.04 4.04) (thickness 0.3)))
   )
@@
     (effects (font (size 4.04 4.04) (thickness 0.3)))
   )
-  (gr_text "18 ft" (at 508 -292.1) (layer "F.SilkS")
-    (effects (font (size 4.04 4.04) (thickness 0.3)))
-  )
-  (gr_text "Pump house\nshed\n6'x5'" (at 215.9 0) (layer "B.Fab")
+  (gr_text "10 ft" (at 406.4 -292.1) (layer "F.SilkS")
+    (effects (font (size 4.04 4.04) (thickness 0.3)))
+  )
+  (gr_text "Pump house\nshed\n6'x5'" (at 203.2 0) (layer "B.Fab")
     (effects (font (size 6.58 6.58) (thickness 0.3)))
   )
   (gr_text "Norwesco 3450\nGallon Tank\n96\" diameter" (at 406.4 -139.7) (layer "F.Fab")
-    (effects (font (size 6.58 6.58) (thickness 0.3)))
-  )
-  (gr_text "Norwesco 3450\nGallon Tank\n96\" diameter" (at 609.6 0) (layer "F.Fab")
     (effects (font (size 6.58 6.58) (thickness 0.3)))
   )
@@
     (style (thickness 0.2) (arrow_length 1.27) (text_position_mode 0) (extension_height 0.58642) (extension_offset 0.5) keep_text_aligned)
   )
-  (dimension (type aligned) (layer "F.Paste")
-    (pts (xy 508 0) (xy 406.4 0))
-    (height 0)
-    (gr_text "48 in" (at 457.2 -4.34) (layer "F.Paste")
-      (effects (font (size 4.04 4.04) (thickness 0.3)))
-    )
-    (format (units 3) (units_format 1) (precision 4) (override_value "48"))
+  (dimension (type aligned) (layer "F.SilkS")
+    (pts (xy 279.4 -266.7) (xy 533.4 -266.7))
+    (height -12.7)
+    (gr_text "120 in" (at 406.4 -283.74) (layer "F.SilkS")
+      (effects (font (size 4.04 4.04) (thickness 0.3)))
+    )
+    (format (units 3) (units_format 1) (precision 4) (override_value "120"))
     (style (thickness 0.2) (arrow_length 1.27) (text_position_mode 0) (extension_height 0.58642) (extension_offset 0.5) keep_text_aligned)
   )
   (dimension (type aligned) (layer "F.SilkS")
-    (pts (xy 279.4 -266.7) (xy 736.6 -266.7))
-    (height -12.7)
-    (gr_text "216 in" (at 508 -283.74) (layer "F.SilkS")
-      (effects (font (size 4.04 4.04) (thickness 0.3)))
-    )
-    (format (units 3) (units_format 1) (precision 4) (override_value "216"))
-    (style (thickness 0.2) (arrow_length 1.27) (text_position_mode 0) (extension_height 0.58642) (extension_offset 0.5) keep_text_aligned)
+    (pts (xy 279.4 -266.7) (xy 279.4 -393.7))
+    (height -12.7)
+    (gr_text "60 in" (at 262.36 -330.2 90) (layer "F.SilkS")
+      (effects (font (size 4.04 4.04) (thickness 0.3)))
+    )
+    (format (units 3) (units_format 1) (precision 4) (override_value "60"))
+    (style (thickness 0.2) (arrow_length 1.27) (text_position_mode 0) (extension_height 0.58642) (extension_offset 0.5))
+  )
+  (dimension (type aligned) (layer "F.SilkS")
+    (pts (xy 279.4 393.7) (xy 279.4 266.7))
+    (height -12.7)
+    (gr_text "60 in" (at 262.36 330.2 90) (layer "F.SilkS")
+      (effects (font (size 4.04 4.04) (thickness 0.3)))
+    )
+    (format (units 3) (units_format 1) (precision 4) (override_value "60"))
+    (style (thickness 0.2) (arrow_length 1.27) (text_position_mode 0) (extension_height 0.58642) (extension_offset 0.5))
   )
   (dimension (type aligned) (layer "F.SilkS")
@@
   )
   (dimension (type aligned) (layer "F.SilkS")
-    (pts (xy 736.6 -266.7) (xy 736.6 266.7))
-    (height -12.7)
-    (gr_text "252 in" (at 753.64 0 270) (layer "F.SilkS")
+    (pts (xy 533.4 -266.7) (xy 533.4 266.7))
+    (height -12.7)
+    (gr_text "252 in" (at 550.44 0 270) (layer "F.SilkS")
       (effects (font (size 4.04 4.04) (thickness 0.3)))
     )
@@
     (style (thickness 0.2) (arrow_length 1.27) (text_position_mode 0) (extension_height 0.58642) (extension_offset 0.5))
   )
+  (dimension (type aligned) (layer "F.SilkS")
+    (pts (xy 152.4 -76.2) (xy 152.4 -393.7))
+    (height -12.7)
+    (gr_text "150 in" (at 135.36 -234.95 90) (layer "F.SilkS")
+      (effects (font (size 4.04 4.04) (thickness 0.3)))
+    )
+    (format (units 3) (units_format 1) (precision 4) (override_value "150"))
+    (style (thickness 0.2) (arrow_length 1.27) (text_position_mode 0) (extension_height 0.58642) (extension_offset 0.5))
+  )
