File: Antennas/Panel_4x4_5GHz_Dual_XPol_1/Feeds/Feeds.kicad_pcb (KiCad board)
At the start: 2 copper layers, 186 x 226 mm, 76 parts

Commit message: Placed an order with JLCPCB for the Tighter 4pol version and the "Dual XPol" which actually was aperture coupled.
Parts:
- added H12: Mounting Hole, MountingHole:MountingHole_2.5mm_Pad_TopBottom, F.Cu at (93.0, 113.0)
- moved REF** 121.2 mm to (164.0, 170.9), turned to 0 degrees
- moved REF** 118.1 mm to (157.6, 176.4), turned to -135 degrees
- moved AE5 117.1 mm to (147.0, 187.0), turned to -135 degrees
- moved REF** 114.4 mm to (166.5, 154.9), turned to 90 degrees
- moved REF** 112.6 mm to (54.5, 135.3), turned to 180 degrees
- moved REF** 109.7 mm to (52.0, 138.9), turned to 90 degrees
- moved REF** 108.3 mm to (45.6, 144.4), turned to -135 degrees
- moved REF** 107.6 mm to (166.5, 135.3), turned to 90 degrees
- moved AE5 107.1 mm to (35.0, 155.0), turned to -135 degrees
- moved REF** 104.9 mm to (164.0, 138.9), turned to 90 degrees
- moved Feed4 104.2 mm to (70.5, 135.3), turned to 0 degrees
- moved REF** 100.2 mm to (86.5, 135.3), turned to 90 degrees
- moved REF** 97.7 mm to (157.6, 144.4), turned to -135 degrees
- moved REF** 95.4 mm to (84.0, 138.9), turned to 90 degrees
- moved AE5 92.7 mm to (115.0, 187.0), turned to -135 degrees
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Other:
- outline, holes or cut-outs redrawn
- board text added: "Panel Antenna 4x4 rev3 Copyright 2021 ISis ImageStream Internet Solutions, Inc."
- board text removed: "Panel Antenna 4x4 rev2 Copyright 2020 ISis ImageStream Internet Solutions, Inc."

Commit message: Fix antenna hole (again?) so that the feed isn't shorted to ground
Other:
- board text added: "Panel Antenna 4x4 rev4 Copyright 2021 ISis ImageStream Internet Solutions, Inc."
- board text removed: "Panel Antenna 4x4 rev3 Copyright 2021 ISis ImageStream Internet Solutions, Inc."
Changed lines of the file:
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@@
-(kicad_pcb (version 20210126) (generator pcbnew)
+(kicad_pcb (version 20210228) (generator pcbnew)
   (general
     (thickness 0.8)
@@
       (dielectric_constraints yes)
     )
+    (pad_to_mask_clearance 0)
     (pcbplotparams
       (layerselection 0x00010fc_ffffffff)
@@
       (effects (font (size 1 1) (thickness 0.15)) (justify mirror))
     )
+    (fp_text user "${REF}" (at 0 -2.5 unlocked) (layer "B.Fab")
+      (effects (font (size 1 1) (thickness 0.15)) (justify mirror))
+    )
     (fp_poly (pts (xy 0.997704 0.78249)
       (xy 0.997704 -0.781621)
@@
       (xy -1.001585 0.78249)) (layer "B.Mask") (width 0.0001) (fill solid))
     (fp_arc (start 0.0091 -0.004623) (end 1.095 3.734) (angle -147.1780634) (layer "F.Mask") (width 2.2))
-    (fp_poly (pts (xy 2.982 0.486)
-      (xy 0.0034 0.5594)
-      (xy 0.003 4.996)
-      (xy 1.284 4.81)) (layer "F.Mask") (width 0.0001) (fill solid))
+    (fp_poly (pts (xy 0.3284 4.99115)
+      (xy 0.526 4.971)
+      (xy 0.68 4.948)
+      (xy 0.908 4.913)
+      (xy 1.271 4.826)
+      (xy 1.783 4.657)
+      (xy 0.0034 4.6624)
+      (xy 0.0034 5.0124)
+      (xy 0.142 5.004)) (layer "F.Mask") (width 0.0001) (fill solid))
     (fp_poly (pts (xy 1.2624 -4.8386)
       (xy 1.0924 -4.8786)
@@
       (xy 0.0024 -4.9986)
       (xy 1.4724 -4.7786)) (layer "F.Mask") (width 0.0001) (fill solid))
+    (fp_poly (pts (xy 2.982 0.486)
+      (xy 0.0034 0.5594)
+      (xy 0.003 4.996)
+      (xy 1.284 4.81)) (layer "F.Mask") (width 0.0001) (fill solid))
     (fp_poly (pts (xy 1.467943 -4.784133)
       (xy -0.002057 -5.004133)
@@
       (xy 0.1134 0.5594)
       (xy 0.6134 0.5594)) (layer "F.Mask") (width 0.0001) (fill solid))
-    (fp_poly (pts (xy 0.3284 4.99115)
-      (xy 0.526 4.971)
-      (xy 0.68 4.948)
-      (xy 0.908 4.913)
-      (xy 1.271 4.826)
-      (xy 1.783 4.657)
-      (xy 0.0034 4.6624)
-      (xy 0.0034 5.0124)
-      (xy 0.142 5.004)) (layer "F.Mask") (width 0.0001) (fill solid))
-    (pad "" np_thru_hole circle (at 0 0) (locked) (size 1.565 1.565) (drill 0.8) (layers "B.Cu" "B.Mask")
+    (pad "" np_thru_hole circle (at 0 0) (locked) (size 1.565 1.565) (drill 1) (layers "B.Cu" "B.Mask")
       (net 4 "/A1P1"))
     (pad "1" smd custom (at 0 0) (locked) (size 1.524 1.524) (layers "B.Cu")
@@
         )         (width 0.0001)         (fill yes)        )
       ))
-    (pad "2" smd circle (at 0 0) (locked) (size 10 10) (layers "F.Cu")
+    (pad "2" smd circle (at 4 0) (locked) (size 1 1) (layers "F.Cu")
       (net 1 "GND") (pinfunction "Shield"))
   )
@@
       (xy 0.0034 5.0124)
       (xy 0.142 5.004)) (layer "F.Mask") (width 0.0001) (fill solid))
+    (fp_poly (pts (xy 1.467943 -4.784133)
+      (xy -0.002057 -5.004133)
+      (xy -0.005279 -0.559875)
+      (xy 0.616 -0.555)
+      (xy 0.597 0.567)
+      (xy 3.24 0.486)) (layer "F.Mask") (width 0.0001) (fill solid))
     (fp_poly (pts (xy 0.6134 -0.5606)
       (xy 0.0234 -0.5606)
@@
       (xy 0.003 4.996)
       (xy 1.284 4.81)) (layer "F.Mask") (width 0.0001) (fill solid))
-    (fp_poly (pts (xy 1.467943 -4.784133)
-      (xy -0.002057 -5.004133)
-      (xy -0.005279 -0.559875)
-      (xy 0.616 -0.555)
-      (xy 0.597 0.567)
-      (xy 3.24 0.486)) (layer "F.Mask") (width 0.0001) (fill solid))
-    (pad "" np_thru_hole circle (at 0 0) (locked) (size 1.565 1.565) (drill 0.8) (layers "B.Cu" "B.Mask")
+    (pad "" np_thru_hole circle (at 0 0) (locked) (size 1.565 1.565) (drill 1) (layers "B.Cu" "B.Mask")
       (net 4 "/A1P1"))
     (pad "1" smd custom (at 0 0) (locked) (size 1.524 1.524) (layers "B.Cu")
@@
         )         (width 0.0001)         (fill yes)        )
       ))
-    (pad "2" smd circle (at 0 0) (locked) (size 10 10) (layers "F.Cu")
+    (pad "2" smd circle (at 4 0) (locked) (size 1 1) (layers "F.Cu")
       (net 1 "GND") (pinfunction "Shield"))
   )
@@
       (effects (font (size 1 1) (thickness 0.15)) (justify mirror))
     )
+    (fp_text user "${REF}" (at 0 -2.5 180 unlocked) (layer "B.Fab")
+      (effects (font (size 1 1) (thickness 0.15)) (justify mirror))
+    )
     (fp_poly (pts (xy 0.997704 0.78249)
       (xy 0.997704 -0.781621)
@@
       (xy 0.597 0.567)
       (xy 3.24 0.486)) (layer "F.Mask") (width 0.0001) (fill solid))
+    (fp_poly (pts (xy 2.982 0.486)
+      (xy 0.0034 0.5594)
+      (xy 0.003 4.996)
+      (xy 1.284 4.81)) (layer "F.Mask") (width 0.0001) (fill solid))
     (fp_poly (pts (xy 1.2624 -4.8386)
       (xy 1.0924 -4.8786)
@@
       (xy 0.0024 -4.9986)
       (xy 1.4724 -4.7786)) (layer "F.Mask") (width 0.0001) (fill solid))
-    (fp_poly (pts (xy 2.982 0.486)
-      (xy 0.0034 0.5594)
-      (xy 0.003 4.996)
-      (xy 1.284 4.81)) (layer "F.Mask") (width 0.0001) (fill solid))
     (fp_poly (pts (xy 0.3284 4.99115)
       (xy 0.526 4.971)
@@
       (xy 0.1134 0.5594)
       (xy 0.6134 0.5594)) (layer "F.Mask") (width 0.0001) (fill solid))
-    (pad "" np_thru_hole circle (at 0 0 180) (locked) (size 1.565 1.565) (drill 0.8) (layers "B.Cu" "B.Mask")
+    (pad "" np_thru_hole circle (at 0 0 180) (locked) (size 1.565 1.565) (drill 1) (layers "B.Cu" "B.Mask")
       (net 4 "/A1P1"))
     (pad "1" smd custom (at 0 0 180) (locked) (size 1.524 1.524) (layers "B.Cu")
@@
         )         (width 0.0001)         (fill yes)        )
       ))
-    (pad "2" smd circle (at 0 0 180) (locked) (size 10 10) (layers "F.Cu")
+    (pad "2" smd circle (at 4 0 180) (locked) (size 1 1) (layers "F.Cu")
       (net 1 "GND") (pinfunction "Shield"))
   )
@@
       (xy -1.001585 0.78249)) (layer "B.Mask") (width 0.0001) (fill solid))
     (fp_arc (start 0.0091 -0.004623) (end 1.095 3.734) (angle -147.1780634) (layer "F.Mask") (width 2.2))
-    (fp_poly (pts (xy 1.467943 -4.784133)
-      (xy -0.002057 -5.004133)
-      (xy -0.005279 -0.559875)
-      (xy 0.616 -0.555)
-      (xy 0.597 0.567)
-      (xy 3.24 0.486)) (layer "F.Mask") (width 0.0001) (fill solid))
     (fp_poly (pts (xy 2.982 0.486)
       (xy 0.0034 0.5594)
@@
       (xy 0.0034 5.0124)
       (xy 0.142 5.004)) (layer "F.Mask") (width 0.0001) (fill solid))
-    (fp_poly (pts (xy 1.2624 -4.8386)
-      (xy 1.0924 -4.8786)
-      (xy 0.8924 -4.9186)
-      (xy 0.6424 -4.9586)
-      (xy 0.4524 -4.9786)
-      (xy 0.3024 -4.9886)
-      (xy 0.0924 -4.9986)
-      (xy 0.0024 -4.9986)
-      (xy 1.4724 -4.7786)) (layer "F.Mask") (width 0.0001) (fill solid))
+    (fp_poly (pts (xy 1.467943 -4.784133)
+      (xy -0.002057 -5.004133)
+      (xy -0.005279 -0.559875)
+      (xy 0.616 -0.555)
+      (xy 0.597 0.567)
+      (xy 3.24 0.486)) (layer "F.Mask") (width 0.0001) (fill solid))
     (fp_poly (pts (xy 0.6134 -0.5606)
       (xy 0.0234 -0.5606)
@@
       (xy 0.1134 0.5594)
       (xy 0.6134 0.5594)) (layer "F.Mask") (width 0.0001) (fill solid))
-    (pad "" np_thru_hole circle (at 0 0 180) (locked) (size 1.565 1.565) (drill 0.8) (layers "B.Cu" "B.Mask")
+    (fp_poly (pts (xy 1.2624 -4.8386)
+      (xy 1.0924 -4.8786)
+      (xy 0.8924 -4.9186)
+      (xy 0.6424 -4.9586)
+      (xy 0.4524 -4.9786)
+      (xy 0.3024 -4.9886)
+      (xy 0.0924 -4.9986)
+      (xy 0.0024 -4.9986)
+      (xy 1.4724 -4.7786)) (layer "F.Mask") (width 0.0001) (fill solid))
+    (pad "" np_thru_hole circle (at 0 0 180) (locked) (size 1.565 1.565) (drill 1) (layers "B.Cu" "B.Mask")
       (net 4 "/A1P1"))
     (pad "1" smd custom (at 0 0 180) (locked) (size 1.524 1.524) (layers "B.Cu")
@@
         )         (width 0.0001)         (fill yes)        )
       ))
-    (pad "2" smd circle (at 0 0 180) (locked) (size 10 10) (layers "F.Cu")
+    (pad "2" smd circle (at 4 0 180) (locked) (size 1 1) (layers "F.Cu")
       (net 1 "GND") (pinfunction "Shield"))
   )
@@
   (gr_line (start 6 108) (end 0 108) (layer "Edge.Cuts") (width 0.1))
   (gr_line (start 186 0) (end 186 108) (layer "Edge.Cuts") (width 0.1))
-  (gr_text "Panel Antenna 4x4 rev3\nCopyright 2021 ISis ImageStream Internet Solutions, Inc." (at 179.9844 137.3632 90) (layer "B.SilkS")
+  (gr_text "Panel Antenna 4x4 rev4\nCopyright 2021 ISis ImageStream Internet Solutions, Inc." (at 179.9844 137.3632 90) (layer "B.SilkS")
     (effects (font (size 1.5 1.5) (thickness 0.3)) (justify left mirror))
   )
