File: AP3500/AP3500.kicad_sch (KiCad schematic)
At the start: 4 parts

Commit message: Almost done with new smaller AP3500 board
Connections:
- net GNDPWR is gone; now on net GND: H3.1, H4.1
Other:
- moved on the sheet: H3, H4
Changed lines of the file:
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@@
     (comment 1 "www.imagestream.com")
   )
-  (junction (at 208.915 109.22) (diameter 1.016) (color 0 0 0 0))
+  (junction (at 222.25 109.22) (diameter 1.016) (color 0 0 0 0))
+  (junction (at 229.87 109.22) (diameter 1.016) (color 0 0 0 0))
   (junction (at 240.03 109.22) (diameter 1.016) (color 0 0 0 0))
   (wire (pts (xy 120.015 35.56) (xy 141.605 35.56))
@@
     (stroke (width 0) (type solid) (color 0 0 0 0))
   )
-  (wire (pts (xy 199.39 107.95) (xy 199.39 109.22))
+  (wire (pts (xy 212.725 107.95) (xy 212.725 109.22))
     (stroke (width 0) (type solid) (color 0 0 0 0))
   )
-  (wire (pts (xy 199.39 109.22) (xy 208.915 109.22))
+  (wire (pts (xy 212.725 109.22) (xy 222.25 109.22))
     (stroke (width 0) (type solid) (color 0 0 0 0))
   )
-  (wire (pts (xy 208.915 107.95) (xy 208.915 109.22))
+  (wire (pts (xy 222.25 107.95) (xy 222.25 109.22))
+    (stroke (width 0) (type solid) (color 0 0 0 0))
+  )
+  (wire (pts (xy 222.25 109.22) (xy 229.87 109.22))
     (stroke (width 0) (type solid) (color 0 0 0 0))
   )
@@
     (effects (font (size 1.27 1.27)) (justify left bottom))
   )
-  (symbol (lib_id "power:GNDPWR") (at 208.915 109.22 0) (mirror y) (unit 1)
-    (in_bom yes) (on_board yes)
-    (property "Reference" "#PWR0133" (id 0) (at 208.915 115.57 0)
-      (effects (font (size 1.27 1.27)) hide)
-    )
-    (property "Value" "GNDPWR" (id 1) (at 208.915 112.395 0))
-    (property "Footprint" "" (id 2) (at 208.915 109.22 0)
-      (effects (font (size 1.27 1.27)) hide)
-    )
-    (property "Datasheet" "" (id 3) (at 208.915 109.22 0)
-      (effects (font (size 1.27 1.27)) hide)
-    )
-  )
   (symbol (lib_id "power:GND") (at 248.285 109.22 0) (unit 1)
     (in_bom yes) (on_board yes)
@@
     )
   )
-  (symbol (lib_id "Mechanical:MountingHole_Pad") (at 199.39 105.41 0) (unit 1)
+  (symbol (lib_id "Mechanical:MountingHole_Pad") (at 212.725 105.41 0) (unit 1)
     (in_bom yes) (on_board yes)
-    (property "Reference" "H3" (id 0) (at 200.025 100.965 0)
+    (property "Reference" "H3" (id 0) (at 213.36 100.965 0)
       (effects (font (size 1.27 1.27)) (justify left))
     )
-    (property "Value" "Mounting Hole" (id 1) (at 200.025 107.315 0)
+    (property "Value" "Mounting Hole" (id 1) (at 213.36 107.315 0)
       (effects (font (size 1.27 1.27)) (justify left) hide)
     )
-    (property "Footprint" "MountingHole:MountingHole_3.7mm_Pad_TopBottom" (id 2) (at 199.39 105.41 0)
+    (property "Footprint" "MountingHole:MountingHole_3.7mm_Pad_TopBottom" (id 2) (at 212.725 105.41 0)
       (effects (font (size 1.27 1.27)) hide)
     )
-    (property "Datasheet" "~" (id 3) (at 199.39 105.41 0)
+    (property "Datasheet" "~" (id 3) (at 212.725 105.41 0)
       (effects (font (size 1.27 1.27)) hide)
     )
   )
-  (symbol (lib_id "Mechanical:MountingHole_Pad") (at 208.915 105.41 0) (unit 1)
+  (symbol (lib_id "Mechanical:MountingHole_Pad") (at 222.25 105.41 0) (unit 1)
     (in_bom yes) (on_board yes)
-    (property "Reference" "H4" (id 0) (at 209.55 100.965 0)
+    (property "Reference" "H4" (id 0) (at 222.885 100.965 0)
       (effects (font (size 1.27 1.27)) (justify left))
     )
-    (property "Value" "Mounting Hole" (id 1) (at 209.55 107.315 0)
+    (property "Value" "Mounting Hole" (id 1) (at 222.885 107.315 0)
       (effects (font (size 1.27 1.27)) (justify left) hide)
     )
-    (property "Footprint" "MountingHole:MountingHole_3.7mm_Pad_TopBottom" (id 2) (at 208.915 105.41 0)
+    (property "Footprint" "MountingHole:MountingHole_3.7mm_Pad_TopBottom" (id 2) (at 222.25 105.41 0)
       (effects (font (size 1.27 1.27)) hide)
     )
-    (property "Datasheet" "~" (id 3) (at 208.915 105.41 0)
+    (property "Datasheet" "~" (id 3) (at 222.25 105.41 0)
       (effects (font (size 1.27 1.27)) hide)
     )
@@
   )
   (symbol_instances
-    (path "/68723c10-ac8d-4552-b88f-1e57e225da4a"
-      (reference "#PWR0133") (unit 1) (value "GNDPWR") (footprint "")
-    )
     (path "/f741eefe-9395-49f1-bf5f-759153dc687d"
       (reference "#PWR0134") (unit 1) (value "GND") (footprint "")

Commit message: Add new single polarity aperture coupled 4x4 antenna. RasPiCNM4Connector test Gerbers for PCBWay Cleanups and optimixations for AP3500
Parts:
- added J2, J4: Conn_Coaxial, Connector_Coaxial:U.FL_Hirose_U.FL-R-SMT-1_Vertical, symbol Connector:Conn_Coaxial
- added J3, J5: Conn_Coaxial, Connector_Coaxial:MMCX_Molex_73415-1471_Vertical, symbol Connector:Conn_Coaxial
Connections:
- new net RF_GND1: J2.2 (Ext), J3.2 (Ext)
- new net RF_GND2: J4.2 (Ext), J5.2 (Ext)
- new net RF_SIG1: J2.1 (In), J3.1 (In)
- new net RF_SIG2: J4.1 (In), J5.1 (In)
