File: AP3500/PSUs.kicad_sch (KiCad schematic)
At the start: 37 parts, among them U10 TPS563249DDCR, U11 TPS563249DDCR, U13 TPS563249DDCR

Commit message: Finalize AP3500 board
Parts:
- removed TP1, TP4, TP5, TP6, TP7: TestPoint, TestPoint:TestPoint_Keystone_5000-5004_Miniature, symbol Connector:TestPoint
Changed lines of the file:
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@@
     (effects (font (size 2.007 2.007)) (justify left))
-  )
-  (symbol (lib_id "Connector:TestPoint") (at 147.32 35.56 0) (unit 1)
-    (in_bom yes) (on_board yes)
-    (property "Reference" "TP1" (id 0) (at 148.7932 32.5628 0)
-      (effects (font (size 1.27 1.27)) (justify left))
-    )
-    (property "Value" "TestPoint" (id 1) (at 148.7932 34.8742 0)
-      (effects (font (size 1.27 1.27)) (justify left))
-    )
-    (property "Footprint" "TestPoint:TestPoint_Keystone_5000-5004_Miniature" (id 2) (at 152.4 35.56 0)
-      (effects (font (size 1.27 1.27)) hide)
-    )
-    (property "Datasheet" "" (id 3) (at 152.4 35.56 0)
-      (effects (font (size 1.27 1.27)) hide)
-    )
-    (property "Field4" "nf" (id 4) (at 147.32 35.56 0)
-      (effects (font (size 1.27 1.27)) hide)
-    )
-    (property "Field5" "nf" (id 5) (at 147.32 35.56 0)
-      (effects (font (size 1.27 1.27)) hide)
-    )
-    (property "Field6" "nf" (id 6) (at 147.32 35.56 0)
-      (effects (font (size 1.27 1.27)) hide)
-    )
-    (property "Field7" "nf" (id 7) (at 147.32 35.56 0)
-      (effects (font (size 1.27 1.27)) hide)
-    )
-    (property "PartsBoxID" "5001" (id 4) (at 147.32 35.56 0)
-      (effects (font (size 1.27 1.27)) hide)
-    )
-  )
-  (symbol (lib_id "Connector:TestPoint") (at 147.32 95.25 0) (unit 1)
-    (in_bom yes) (on_board yes)
-    (property "Reference" "TP4" (id 0) (at 148.7932 92.2528 0)
-      (effects (font (size 1.27 1.27)) (justify left))
-    )
-    (property "Value" "TestPoint" (id 1) (at 148.7932 94.5642 0)
-      (effects (font (size 1.27 1.27)) (justify left))
-    )
-    (property "Footprint" "TestPoint:TestPoint_Keystone_5000-5004_Miniature" (id 2) (at 152.4 95.25 0)
-      (effects (font (size 1.27 1.27)) hide)
-    )
-    (property "Datasheet" "" (id 3) (at 152.4 95.25 0)
-      (effects (font (size 1.27 1.27)) hide)
-    )
-    (property "Field4" "nf" (id 4) (at 147.32 95.25 0)
-      (effects (font (size 1.27 1.27)) hide)
-    )
-    (property "Field5" "nf" (id 5) (at 147.32 95.25 0)
-      (effects (font (size 1.27 1.27)) hide)
-    )
-    (property "Field6" "nf" (id 6) (at 147.32 95.25 0)
-      (effects (font (size 1.27 1.27)) hide)
-    )
-    (property "Field7" "nf" (id 7) (at 147.32 95.25 0)
-      (effects (font (size 1.27 1.27)) hide)
-    )
-    (property "PartsBoxID" "5001" (id 4) (at 147.32 95.25 0)
-      (effects (font (size 1.27 1.27)) hide)
-    )
-  )
-  (symbol (lib_id "Connector:TestPoint") (at 147.32 121.92 180) (unit 1)
-    (in_bom yes) (on_board yes)
-    (property "Reference" "TP5" (id 0) (at 145.8468 124.9172 0)
-      (effects (font (size 1.27 1.27)) (justify left))
-    )
-    (property "Value" "TestPoint" (id 1) (at 145.8468 122.6058 0)
-      (effects (font (size 1.27 1.27)) (justify left))
-    )
-    (property "Footprint" "TestPoint:TestPoint_Keystone_5000-5004_Miniature" (id 2) (at 142.24 121.92 0)
-      (effects (font (size 1.27 1.27)) hide)
-    )
-    (property "Datasheet" "" (id 3) (at 142.24 121.92 0)
-      (effects (font (size 1.27 1.27)) hide)
-    )
-    (property "Field4" "nf" (id 4) (at 147.32 121.92 0)
-      (effects (font (size 1.27 1.27)) hide)
-    )
-    (property "Field5" "nf" (id 5) (at 147.32 121.92 0)
-      (effects (font (size 1.27 1.27)) hide)
-    )
-    (property "Field6" "nf" (id 6) (at 147.32 121.92 0)
-      (effects (font (size 1.27 1.27)) hide)
-    )
-    (property "Field7" "nf" (id 7) (at 147.32 121.92 0)
-      (effects (font (size 1.27 1.27)) hide)
-    )
-    (property "PartsBoxID" "5001" (id 4) (at 147.32 121.92 0)
-      (effects (font (size 1.27 1.27)) hide)
-    )
-  )
-  (symbol (lib_id "Connector:TestPoint") (at 147.955 151.13 0) (unit 1)
-    (in_bom yes) (on_board yes)
-    (property "Reference" "TP6" (id 0) (at 149.4282 148.1328 0)
-      (effects (font (size 1.27 1.27)) (justify left))
-    )
-    (property "Value" "TestPoint" (id 1) (at 149.4282 150.4442 0)
-      (effects (font (size 1.27 1.27)) (justify left))
-    )
-    (property "Footprint" "TestPoint:TestPoint_Keystone_5000-5004_Miniature" (id 2) (at 153.035 151.13 0)
-      (effects (font (size 1.27 1.27)) hide)
-    )
-    (property "Datasheet" "" (id 3) (at 153.035 151.13 0)
-      (effects (font (size 1.27 1.27)) hide)
-    )
-    (property "Field4" "nf" (id 4) (at 147.955 151.13 0)
-      (effects (font (size 1.27 1.27)) hide)
-    )
-    (property "Field5" "nf" (id 5) (at 147.955 151.13 0)
-      (effects (font (size 1.27 1.27)) hide)
-    )
-    (property "Field6" "nf" (id 6) (at 147.955 151.13 0)
-      (effects (font (size 1.27 1.27)) hide)
-    )
-    (property "Field7" "nf" (id 7) (at 147.955 151.13 0)
-      (effects (font (size 1.27 1.27)) hide)
-    )
-    (property "PartsBoxID" "5001" (id 4) (at 147.955 151.13 0)
-      (effects (font (size 1.27 1.27)) hide)
-    )
-  )
-  (symbol (lib_id "Connector:TestPoint") (at 147.955 177.8 180) (unit 1)
-    (in_bom yes) (on_board yes)
-    (property "Reference" "TP7" (id 0) (at 146.4818 180.7972 0)
-      (effects (font (size 1.27 1.27)) (justify left))
-    )
-    (property "Value" "TestPoint" (id 1) (at 146.4818 178.4858 0)
-      (effects (font (size 1.27 1.27)) (justify left))
-    )
-    (property "Footprint" "TestPoint:TestPoint_Keystone_5000-5004_Miniature" (id 2) (at 142.875 177.8 0)
-      (effects (font (size 1.27 1.27)) hide)
-    )
-    (property "Datasheet" "" (id 3) (at 142.875 177.8 0)
-      (effects (font (size 1.27 1.27)) hide)
-    )
-    (property "Field4" "nf" (id 4) (at 147.955 177.8 0)
-      (effects (font (size 1.27 1.27)) hide)
-    )
-    (property "Field5" "nf" (id 5) (at 147.955 177.8 0)
-      (effects (font (size 1.27 1.27)) hide)
-    )
-    (property "Field6" "nf" (id 6) (at 147.955 177.8 0)
-      (effects (font (size 1.27 1.27)) hide)
-    )
-    (property "Field7" "nf" (id 7) (at 147.955 177.8 0)
-      (effects (font (size 1.27 1.27)) hide)
-    )
-    (property "PartsBoxID" "5001" (id 4) (at 147.955 177.8 0)
-      (effects (font (size 1.27 1.27)) hide)
-    )
   )
   (symbol (lib_id "power:GND") (at 85.09 62.23 0) (unit 1)

Commit message: More work on Antennas - laying out the new panel as a 2x2 aperture coupled patch
Parts:
- C30, C48, C49, C55, C56, C62: LCSC (none) -> C14663
- C31, C35, C50, C51, C52, C57, C58, C59: footprint Capacitor_SMD:C_1210_3225Metric -> Capacitor_SMD:C_1206_3216Metric; LCSC (none) -> C90146; PartsBoxID 1210-22uF-X7R-16V -> 1206-22uF-X7R-16V
- C37, C47, C53, C54, C60, C61: LCSC (none) -> C15850
- R28: LCSC (none) -> C14890
- R30, R33, R38: LCSC (none) -> C25804
- R32: LCSC (none) -> C23058
- R37: LCSC (none) -> C22809

Commit message: Add new single polarity aperture coupled 4x4 antenna. RasPiCNM4Connector test Gerbers for PCBWay Cleanups and optimixations for AP3500
Parts:
- C30, C48, C49, C55, C56, C62: PartsBoxID 0603-100nF-X7R-50V -> (none)
- C31, C35, C50, C51, C52, C57, C58, C59: PartsBoxID 1206-22uF-X7R-16V -> (none)
- C37, C47, C53, C54, C60, C61: PartsBoxID 0805-10uF-X7R-25V -> (none)
- R28: PartsBoxID CRCW060373K2FKEA -> (none)
- R30, R33, R38: PartsBoxID 0603-10K-1% -> (none)
- R32: PartsBoxID CRCW060345K3FKEA -> (none)
- R37: PartsBoxID 0603-15K-1% -> (none)
